Commit message: Tune Pod1 model
Remeasured side width and bin heights
Add front flap
Make recipe a parameter to the pod macro
Adjust frame geometry to better match real frame
Make pod selectable via launch arg in view_models

Co-authored-by: Collin Dang <collindang88@gmail.com>

File: tahoma_description/robots/pod1.xacro (robot description, xacro)
@@ -2,4 +2,4 @@
 <robot xmlns:xacro="http://www.ros.org/wiki/xacro" name="tahoma">
   <xacro:include filename="$(find tahoma_description)/urdf/pod.xacro"/>
-  <xacro:pod prefix="pod_"/>
+  <xacro:pod prefix="pod_" recipe_a="${[8.75,5.5,7.5,6,4.5,8.75,5,6,5,8.75,5,6,11]}"/>
 </robot>

File: tahoma_description/urdf/pod.xacro (robot description, xacro)
@@ -1,12 +1,12 @@
 <?xml version="1.0"?>
 <robot xmlns:xacro="http://www.ros.org/wiki/xacro" name="pod">
-  <xacro:macro name="pod" params="prefix">
+  <xacro:macro name="pod" params="prefix recipe_a">
     <xacro:arg name="prefix" default="pod_"/>
+    <xacro:arg name="recipe_a" default="[]"/>     <!-- bin heights in inches -->
     <xacro:property name="M_PI" value="3.1415926535897931"/>
     <xacro:property name="M_PI_2" value="1.57079632679489661923"/>
-    <xacro:property name="SIDE" value=".9398"/>     <!-- 37 in -->
+    <xacro:property name="SIDE" value="0.9144"/>     <!-- 36 in -->
     <xacro:property name="IN_TO_M" value="0.0254"/>
-    <!-- bin heights in inches -->
-    <xacro:property name="front_recipe" value="${[9,5.5,8,6,5,9,5,6,5,9,5,5.5,10.5]}"/>
+    <xacro:property name="FLAP_HEIGHT" value="${1 * IN_TO_M}"/> <!-- 1 inch -->
     <xacro:property name="alphabet" value="abcdefghijklmnopqrstuvwxyz"/>
     <material name="yellow_fabric">
@@ -17,8 +17,8 @@
     </material>
     <link name="${prefix}base_link">
-              <inertial>
-            <mass value="30.0" />
-            <inertia ixx="0.0002835" ixy="0.0" ixz="0.0" iyy="0.0002835" iyz="0.0" izz="0.000324"/>
-        </inertial>
+      <inertial>
+        <mass value="30.0"/>
+        <inertia ixx="0.0002835" ixy="0.0" ixz="0.0" iyy="0.0002835" iyz="0.0" izz="0.000324"/>
+      </inertial>
       <visual>
         <origin rpy="0 0 0" xyz=".4699 .4699 1.303"/>
@@ -41,7 +41,7 @@
       <child link="${prefix}brace"/>
     </joint>
-      <link name="${prefix}fabric_base"/>
+    <link name="${prefix}fabric_base"/>
     <joint name="${prefix}brace_${prefix}fabric_base" type="fixed">
-      <origin xyz="0 0 .065"/>
+      <origin xyz="0.01 0.01 .045"/>
       <parent link="${prefix}brace"/>
       <child link="${prefix}fabric_base"/>
@@ -50,6 +50,6 @@
       <link name="${name}">
         <inertial>
-            <mass value="0.01" />
-            <inertia ixx="0.0002835" ixy="0.0" ixz="0.0" iyy="0.0002835" iyz="0.0" izz="0.000324"/>
+          <mass value="0.01"/>
+          <inertia ixx="0.0002835" ixy="0.0" ixz="0.0" iyy="0.0002835" iyz="0.0" izz="0.000324"/>
         </inertial>
         <visual>
@@ -77,4 +77,5 @@
       <xacro:shifted_box name="${bin_name}_top" width="${width}" height="${depth}" length="${thickness}"/>
       <xacro:shifted_box name="${bin_name}_back" width="${width}" height="${height}" length="${thickness}"/>
+      <xacro:shifted_box name="${bin_name}_flap" width="${width}" height="${FLAP_HEIGHT}" length="${thickness}"/>
       <joint name="${bin_name}_${bin_name}_bottom" type="fixed">
         <parent link="${bin_name}"/>
@@ -100,4 +101,9 @@
         <parent link="${bin_name}"/>
         <child link="${bin_name}_back"/>
+      </joint>
+      <joint name="${bin_name}_${bin_name}_flap" type="fixed">
+        <origin xyz="0 0 0" rpy="${M_PI_2} 0 0"/>
+        <parent link="${bin_name}"/>
+        <child link="${bin_name}_flap"/>
       </joint>
     </xacro:macro>
@@ -138,5 +144,5 @@
       </xacro:if>
     </xacro:macro>
-    <xacro:shelf_stack prefix="${prefix}" parent="${prefix}fabric_base" recipe="${front_recipe}" width="${SIDE}"
+    <xacro:shelf_stack prefix="${prefix}" parent="${prefix}fabric_base" recipe="${recipe_a}" width="${SIDE}"
                        depth=".1524"/>
     <!-- Front left corner -->

Commit message: Tweak pod xacro
Remove some hardcoded constants
Fix robot name

File: tahoma_description/robots/pod1.xacro (robot description, xacro)
@@ -1,4 +1,4 @@
 <?xml version="1.0"?>
-<robot xmlns:xacro="http://www.ros.org/wiki/xacro" name="tahoma">
+<robot xmlns:xacro="http://www.ros.org/wiki/xacro" name="pod1">
   <xacro:include filename="$(find tahoma_description)/urdf/pod.xacro"/>
   <xacro:pod prefix="pod_" recipe_a="${[8.75,5.5,7.5,6,4.5,8.75,5,6,5,8.75,5,6,11]}"/>

File: tahoma_description/urdf/pod.xacro (robot description, xacro)
@@ -4,6 +4,4 @@
     <xacro:arg name="prefix" default="pod_"/>
     <xacro:arg name="recipe_a" default="[]"/>     <!-- bin heights in inches -->
-    <xacro:property name="M_PI" value="3.1415926535897931"/>
-    <xacro:property name="M_PI_2" value="1.57079632679489661923"/>
     <xacro:property name="SIDE" value="0.9144"/>     <!-- 36 in -->
     <xacro:property name="IN_TO_M" value="0.0254"/>
@@ -83,10 +81,10 @@
       </joint>
       <joint name="${bin_name}_${bin_name}_left" type="fixed">
-        <origin xyz="0 0 0" rpy="${M_PI_2} 0 ${M_PI_2} "/>
+        <origin xyz="0 0 0" rpy="${pi / 2} 0 ${pi / 2} "/>
         <parent link="${bin_name}"/>
         <child link="${bin_name}_left"/>
       </joint>
       <joint name="${bin_name}_${bin_name}_right" type="fixed">
-        <origin xyz="${width} 0 0" rpy="${M_PI_2} 0 ${M_PI_2} "/>
+        <origin xyz="${width} 0 0" rpy="${pi / 2} 0 ${pi / 2} "/>
         <parent link="${bin_name}"/>
         <child link="${bin_name}_right"/>
@@ -98,10 +96,10 @@
       </joint>
       <joint name="${bin_name}_${bin_name}_back" type="fixed">
-        <origin xyz="0 ${depth} 0" rpy="${M_PI_2} 0 0"/>
+        <origin xyz="0 ${depth} 0" rpy="${pi / 2} 0 0"/>
         <parent link="${bin_name}"/>
         <child link="${bin_name}_back"/>
       </joint>
       <joint name="${bin_name}_${bin_name}_flap" type="fixed">
-        <origin xyz="0 0 0" rpy="${M_PI_2} 0 0"/>
+        <origin xyz="0 0 0" rpy="${pi / 2} 0 0"/>
         <parent link="${bin_name}"/>
         <child link="${bin_name}_flap"/>
