Commit message: Improve stand model
Use vention-derived meshes
Add basic color-matched materials
Stand is broken into a few chunks to make it easier to calibrate or modify the assembly in the future
Model is now correctly oriented

File: tahoma_description/robots/tahoma.xacro (robot description, xacro)
@@ -3,26 +3,26 @@
   <xacro:include filename="$(find ur_description)/urdf/inc/ur16e_macro.xacro"/>
   <xacro:include filename="$(find tahoma_description)/urdf/stand.xacro"/>
-  <xacro:include filename="$(find robotiq_2f_85_gripper_visualization)/urdf/robotiq_arg2f_85_macro.xacro" />
+  <xacro:include filename="$(find robotiq_2f_85_gripper_visualization)/urdf/robotiq_arg2f_85_macro.xacro"/>
   <!-- parameters -->
   <xacro:arg name="transmission_hw_interface" default="hardware_interface/EffortJointInterface"/>
-  <xacro:stand />
-  <xacro:ur16e_robot prefix="arm_" />
+  <xacro:stand/>
+  <xacro:ur16e_robot prefix="arm_"/>
   <xacro:robotiq_arg2f_85
-    prefix="gripper_"
-    transmission_hw_interface="$(arg transmission_hw_interface)"/>
+          prefix="gripper_"
+          transmission_hw_interface="$(arg transmission_hw_interface)"/>
   <link name="base_link"/>
   <joint name="base_joint" type="fixed">
-    <origin rpy="0 0 0" xyz="0 0 0"/>
+    <origin rpy="0 0 0" xyz="0 0 0.15"/>
     <parent link="base_link"/>
     <child link="stand"/>
   </joint>
-  <joint name="stand-tahoma_base_link_joint" type="fixed">
-    <parent link="stand"/>
+  <joint name="robot_plate_arm_base_link_joint" type="fixed">
+    <parent link="robot_plate"/>
     <child link="arm_base_link"/>
-    <origin rpy="1.56 1.56 0" xyz="0 -0.01 0"/>
+    <origin rpy="0 3.14 3.14" xyz="0 -0.01 0"/>
   </joint>
   <joint name="arm_tool0-gripper_robotiq_arg2f_base_link" type="fixed">
-    <parent link="arm_tool0" />
-    <child link="gripper_base_link" />
+    <parent link="arm_tool0"/>
+    <child link="gripper_base_link"/>
   </joint>
 </robot>

File: tahoma_description/urdf/stand.xacro (robot description, xacro)
@@ -1,19 +1,161 @@
 <?xml version="1.0"?>
 <robot xmlns:xacro="http://www.ros.org/wiki/xacro" name="stand">
+  <xacro:include filename="$(find tahoma_description)/urdf/caster.xacro"/>
+  <xacro:include filename="$(find tahoma_description)/urdf/light_panel.xacro"/>
   <xacro:macro name="stand">
+    <material name="aluminum">
+      <color rgba=".27 .45 .68 1"/>
+    </material>
     <link name="stand">
       <visual>
-        <origin rpy="0 0 -1.57079632679" xyz="0 1.0668 0.313537"/>
+        <origin rpy="0 0 0" xyz="0 0 0"/>
         <geometry>
-          <mesh filename="package://tahoma_description/meshes/stand/visual/stand.dae"/>
+          <mesh filename="package://tahoma_description/meshes/stand/visual/stand_base.stl"/>
         </geometry>
+        <material name="aluminum"/>
       </visual>
       <collision>
-        <origin rpy="0 0 -1.57079632679" xyz="0 1.0668 0.313537"/>
+        <origin rpy="0 0 0" xyz="0 0 0"/>
         <geometry>
-          <mesh filename="package://tahoma_description/meshes/stand/collision/stand.stl"/>
+          <mesh filename="package://tahoma_description/meshes/stand/visual/stand_base.stl"/>
         </geometry>
       </collision>
     </link>
+    <link name="stand_upright">
+      <visual>
+        <origin rpy="0 0 0" xyz="0 0 0"/>
+        <geometry>
+          <mesh filename="package://tahoma_description/meshes/stand/visual/stand_upright.stl"/>
+        </geometry>
+        <material name="aluminum"/>
+      </visual>
+      <collision>
+        <origin rpy="0 0 0" xyz="0 0 0"/>
+        <geometry>
+          <mesh filename="package://tahoma_description/meshes/stand/visual/stand_upright.stl"/>
+        </geometry>
+      </collision>
+    </link>
+    <link name="stand_brace">
+      <visual>
+        <origin rpy="0 0 0" xyz="0 0 0"/>
+        <geometry>
+          <mesh filename="package://tahoma_description/meshes/stand/visual/stand_brace.stl"/>
+        </geometry>
+        <material name="aluminum"/>
+      </visual>
+      <collision>
+        <origin rpy="0 0 0" xyz="0 0 0"/>
+        <geometry>
+          <mesh filename="package://tahoma_description/meshes/stand/visual/stand_brace.stl"/>
+        </geometry>
+      </collision>
+    </link>
+    <link name="robot_beam">
+      <visual>
+        <origin rpy="0 0 0" xyz="0 0 0"/>
+        <geometry>
+          <mesh filename="package://tahoma_description/meshes/stand/visual/robot_beam.stl"/>
+        </geometry>
+        <material name="aluminum"/>
+      </visual>
+      <collision>
+        <origin rpy="0 0 0" xyz="0 0 0"/>
+        <geometry>
+          <mesh filename="package://tahoma_description/meshes/stand/visual/robot_beam.stl"/>
+        </geometry>
+      </collision>
+    </link>
+    <link name="control_box_mount">
+      <visual>
+        <origin rpy="0 0 0" xyz="0 0 0"/>
+        <geometry>
+          <mesh filename="package://tahoma_description/meshes/stand/visual/control_box_mount.stl"/>
+        </geometry>
+        <material name="aluminum"/>
+      </visual>
+      <collision>
+        <origin rpy="0 0 0" xyz="0 0 0"/>
+        <geometry>
+          <mesh filename="package://tahoma_description/meshes/stand/visual/control_box_mount.stl"/>
+        </geometry>
+      </collision>
+    </link>
+    <link name="robot_plate">
+      <visual>
+        <origin rpy="0 0 0" xyz="0 0 0"/>
+        <geometry>
+          <mesh filename="package://tahoma_description/meshes/stand/visual/robot_plate.stl"/>
+        </geometry>
+        <material name="aluminum"/>
+      </visual>
+      <collision>
+        <origin rpy="0 0 0" xyz="0 0 0"/>
+        <geometry>
+          <mesh filename="package://tahoma_description/meshes/stand/visual/robot_plate.stl"/>
+        </geometry>
+      </collision>
+    </link>
+    <xacro:caster prefix="front_right_"/>
+    <xacro:caster prefix="front_left_"/>
+    <xacro:caster prefix="back_left_"/>
+    <xacro:caster prefix="back_right_"/>
+    <xacro:light_panel prefix="left_"/>
+    <xacro:light_panel prefix="right_"/>
+    <joint name="stand_stand_upright_joint" type="fixed">
+      <parent link="stand"/>
+      <child link="stand_upright"/>
+      <origin rpy="0 0 0" xyz="-.12 0 .95"/>
+    </joint>
+    <joint name="stand_upright_stand_brace_joint" type="fixed">
+      <parent link="stand_upright"/>
+      <child link="stand_brace"/>
+      <origin rpy="0 0 0" xyz="-.24 0 -.59"/>
+    </joint>
+    <joint name="stand_upright_robot_control_box_mount_joint" type="fixed">
+      <parent link="stand_upright"/>
+      <child link="control_box_mount"/>
+      <origin rpy="0 0 0" xyz="-.1725 .7475 0"/>
+    </joint>
+    <joint name="stand_robot_beam_joint" type="fixed">
+      <parent link="stand_upright"/>
+      <child link="robot_beam"/>
+      <origin rpy="0 0 0" xyz=".0775 0  0.9475"/>
+    </joint>
+    <joint name="robot_beam_robot_plate_joint" type="fixed">
+      <parent link="robot_beam"/>
+      <child link="robot_plate"/>
+      <origin rpy="0 0 0" xyz="0.2 0 0"/>
+    </joint>
+    <joint name="stand_front_right_caster_joint" type="fixed">
+      <parent link="stand"/>
+      <child link="front_right_caster"/>
+      <origin rpy="0 0 0" xyz=".405 -.7375 -0.1"/>
+    </joint>
+    <joint name="stand_front_left_caster_joint" type="fixed">
+      <parent link="stand"/>
+      <child link="front_left_caster"/>
+      <origin rpy="0 0 0" xyz=".405 .7025 -0.1"/>
+    </joint>
+    <joint name="stand_back_right_caster_joint" type="fixed">
+      <parent link="stand"/>
+      <child link="back_right_caster"/>
+      <origin rpy="0 0 0" xyz="-.405 -.7375 -0.1"/>
+    </joint>
+    <joint name="stand_back_left_caster_joint" type="fixed">
+      <parent link="stand"/>
+      <child link="back_left_caster"/>
+      <origin rpy="0 0 0" xyz="-.405 .7025 -0.1"/>
+    </joint>
+    <joint name="stand_left_light_panel_joint" type="fixed">
+      <parent link="stand_upright"/>
+      <child link="left_light_panel"/>
+      <origin rpy="0 1.56 0" xyz="-.26 .35 .25"/>
+    </joint>
+    <joint name="stand_left_right_panel_joint" type="fixed">
+      <parent link="stand_upright"/>
+      <child link="right_light_panel"/>
+      <origin rpy="0 1.56 0" xyz="-.26 -.35 .25"/>
+    </joint>
   </xacro:macro>
 </robot>

Commit message: Improve description
Track kinematics parameters extracted from the robot
Add helper launch file to load the model into the parameter server

File: tahoma_description/robots/tahoma.xacro (robot description, xacro)
@@ -20,5 +20,5 @@
     <parent link="stand"/>
     <child link="arm_base_link"/>
-    <origin rpy="1.57079632679 0 0" xyz="0 1.017975 0.5602"/>
+    <origin rpy="1.56 1.56 0" xyz="0 -0.01 0"/>
   </joint>
   <joint name="arm_tool0-gripper_robotiq_arg2f_base_link" type="fixed">

Commit message: Add stand-mounted RealSense D415
Fix some rotations

File: tahoma_description/robots/tahoma.xacro (robot description, xacro)
@@ -4,6 +4,8 @@
   <xacro:include filename="$(find tahoma_description)/urdf/stand.xacro"/>
   <xacro:include filename="$(find robotiq_2f_85_gripper_visualization)/urdf/robotiq_arg2f_85_macro.xacro"/>
-  <!-- parameters -->
+  <xacro:include filename="$(find realsense2_description)/urdf/_d415.urdf.xacro"/>
+  <xacro:arg name="realsense" default="true" />
   <xacro:arg name="transmission_hw_interface" default="hardware_interface/EffortJointInterface"/>
+  <xacro:property name="M_PI" value="3.1415926535897931"/>
   <xacro:stand/>
   <xacro:ur16e_robot prefix="arm_"/>
@@ -20,5 +22,5 @@
     <parent link="robot_plate"/>
     <child link="arm_base_link"/>
-    <origin rpy="0 3.14 3.14" xyz="0 -0.01 0"/>
+    <origin rpy="0 ${M_PI} ${M_PI}" xyz="0 -0.01 0"/>
   </joint>
   <joint name="arm_tool0-gripper_robotiq_arg2f_base_link" type="fixed">
@@ -26,3 +28,12 @@
     <child link="gripper_base_link"/>
   </joint>
+  <link name="mid_camera_mount"/>
+  <joint name="stand_upright_mid_camera_mount_joint" type="fixed">
+      <parent link="stand_upright"/>
+      <child link="mid_camera_mount"/>
+      <origin rpy="0 0 0" xyz="-.2 0 0"/>
+  </joint>
+  <xacro:sensor_d415 name="mid_camera" parent="mid_camera_mount" use_nominal_extrinsics="true">
+      <origin xyz="0.025 -0.025 0.003" rpy="0 0 0"/>
+  </xacro:sensor_d415>
 </robot>

File: tahoma_description/urdf/stand.xacro (robot description, xacro)
@@ -4,5 +4,7 @@
   <xacro:include filename="$(find tahoma_description)/urdf/light_panel.xacro"/>
   <xacro:macro name="stand">
-    <material name="aluminum">
+  <xacro:property name="M_PI" value="3.1415926535897931"/>
+  <xacro:property name="M_PI_2" value="1.57079632679489661923"/>
+    <material name="blue_aluminum">
       <color rgba=".27 .45 .68 1"/>
     </material>
@@ -13,5 +15,5 @@
           <mesh filename="package://tahoma_description/meshes/stand/visual/stand_base.stl"/>
         </geometry>
-        <material name="aluminum"/>
+        <material name="blue_aluminum"/>
       </visual>
       <collision>
@@ -28,5 +30,5 @@
           <mesh filename="package://tahoma_description/meshes/stand/visual/stand_upright.stl"/>
         </geometry>
-        <material name="aluminum"/>
+        <material name="blue_aluminum"/>
       </visual>
       <collision>
@@ -43,5 +45,5 @@
           <mesh filename="package://tahoma_description/meshes/stand/visual/stand_brace.stl"/>
         </geometry>
-        <material name="aluminum"/>
+        <material name="blue_aluminum"/>
       </visual>
       <collision>
@@ -58,5 +60,5 @@
           <mesh filename="package://tahoma_description/meshes/stand/visual/robot_beam.stl"/>
         </geometry>
-        <material name="aluminum"/>
+        <material name="blue_aluminum"/>
       </visual>
       <collision>
@@ -73,5 +75,5 @@
           <mesh filename="package://tahoma_description/meshes/stand/visual/control_box_mount.stl"/>
         </geometry>
-        <material name="aluminum"/>
+        <material name="blue_aluminum"/>
       </visual>
       <collision>
@@ -88,5 +90,5 @@
           <mesh filename="package://tahoma_description/meshes/stand/visual/robot_plate.stl"/>
         </geometry>
-        <material name="aluminum"/>
+        <material name="blue_aluminum"/>
       </visual>
       <collision>
@@ -126,5 +128,5 @@
       <parent link="robot_beam"/>
       <child link="robot_plate"/>
-      <origin rpy="0 0 0" xyz="0.2 0 0"/>
+      <origin rpy="0 0 0" xyz="0.2 0 -.015"/>
     </joint>
     <joint name="stand_front_right_caster_joint" type="fixed">
@@ -151,10 +153,10 @@
       <parent link="stand_upright"/>
       <child link="left_light_panel"/>
-      <origin rpy="0 1.56 0" xyz="-.26 .35 .25"/>
+      <origin rpy="0 ${M_PI_2} 0" xyz="-.2625 .35 .25"/>
     </joint>
     <joint name="stand_left_right_panel_joint" type="fixed">
       <parent link="stand_upright"/>
       <child link="right_light_panel"/>
-      <origin rpy="0 1.56 0" xyz="-.26 -.35 .25"/>
+      <origin rpy="0 ${M_PI_2} 0" xyz="-.2625 -.35 .25"/>
     </joint>
   </xacro:macro>
