Commit message: Improve stand model
Add rough (wrong) inertias to stand model to make Gazebo happy
Add boxes for collision geometry
Add emitter region to light panels to better match physical appearance
Add control box
Rename robot_beam to cantilever
Tweak blue aluminum color to a darker, better match
Adjust robot plate position to better match real robot

File: tahoma_description/robots/tahoma.xacro (robot description, xacro)
@@ -4,5 +4,5 @@
   <xacro:include filename="$(find tahoma_description)/urdf/stand.xacro"/>
   <xacro:include filename="$(find robotiq_2f_85_gripper_visualization)/urdf/robotiq_arg2f_85_macro.xacro"/>
-  <xacro:include filename="$(find realsense2_description)/urdf/_d415.urdf.xacro"/>
+  <xacro:include filename="$(find realsense2_description)/urdf/_l515.urdf.xacro"/>
   <xacro:arg name="realsense" default="true" />
   <xacro:arg name="transmission_hw_interface" default="hardware_interface/EffortJointInterface"/>
@@ -34,6 +34,6 @@
       <origin rpy="0 0 0" xyz="-.2 0 0"/>
   </joint>
-  <xacro:sensor_d415 name="mid_camera" parent="mid_camera_mount" use_nominal_extrinsics="true">
+  <xacro:sensor_l515 name="stand_camera" parent="mid_camera_mount" use_nominal_extrinsics="true">
       <origin xyz="0.025 -0.025 0.003" rpy="0 0 0"/>
-  </xacro:sensor_d415>
+  </xacro:sensor_l515>
 </robot>

File: tahoma_description/urdf/caster.xacro (robot description, xacro)
@@ -7,8 +7,13 @@
     </material-->
     <link name="${prefix}caster">
+      <inertial>
+        <!-- Roughly caster, plate and bolts -->
+        <mass value="1.0"/>
+        <inertia ixx="0.0002835" ixy="0.0" ixz="0.0" iyy="0.0002835" iyz="0.0" izz="0.0002835"/>
+      </inertial>
       <visual>
         <origin rpy="1.56 0 0" xyz="0 0 0"/>
         <geometry>
-          <mesh filename="package://tahoma_description/meshes/stand/visual/caster.stl"/>
+          <mesh filename="package://tahoma_description/meshes/stand/caster.stl"/>
         </geometry>
         <material name="wheel">
@@ -19,5 +24,5 @@
         <origin rpy="1.56 0 0" xyz="0 0 0"/>
         <geometry>
-          <mesh filename="package://tahoma_description/meshes/stand/visual/caster.stl"/>
+          <box size="0.09 0.1040 0.1225"/>
         </geometry>
       </collision>

File: tahoma_description/urdf/light_panel.xacro (robot description, xacro)
@@ -5,4 +5,8 @@
     <xacro:arg name="prefix" default=""/>
     <link name="${prefix}light_panel">
+      <inertial>
+        <mass value="1.0"/>
+        <inertia ixx="0.0002835" ixy="0.0" ixz="0.0" iyy="0.0002835" iyz="0.0" izz="0.0002835"/>
+      </inertial>
       <visual>
         <origin rpy="0 0 0" xyz="0 0 0"/>
@@ -10,7 +14,7 @@
           <box size="1.21 .602 .01"/>
         </geometry>
-         <material name="white">
-           <color rgba=".9 .9 .9 1"/>
-         </material>
+        <material name="gray">
+          <color rgba=".3 .3 .3 1"/>
+        </material>
       </visual>
       <collision>
@@ -21,4 +25,25 @@
       </collision>
     </link>
+    <link name="${prefix}light_panel_emitter">
+      <visual>
+        <origin rpy="0 0 0" xyz="0 0 .005"/>
+        <geometry>
+          <box size="1.17 .562 .00251"/>
+        </geometry>
+        <material name="white">
+          <color rgba=".9 .9 .9 1"/>
+        </material>
+      </visual>
+      <collision>
+        <origin rpy="0 0 0" xyz="0 0 0"/>
+        <geometry>
+          <box size="1.17 .562 .00251"/>
+        </geometry>
+      </collision>
+    </link>
+    <joint name="${prefix}light_panel_${prefix}light_panel_emitter_joint" type="fixed">
+      <parent link="${prefix}light_panel"/>
+      <child link="${prefix}light_panel_emitter"/>
+    </joint>
   </xacro:macro>
 </robot>

File: tahoma_description/urdf/stand.xacro (robot description, xacro)
@@ -4,96 +4,172 @@
   <xacro:include filename="$(find tahoma_description)/urdf/light_panel.xacro"/>
   <xacro:macro name="stand">
-  <xacro:property name="M_PI" value="3.1415926535897931"/>
-  <xacro:property name="M_PI_2" value="1.57079632679489661923"/>
+    <xacro:property name="M_PI" value="3.1415926535897931"/>
+    <xacro:property name="M_PI_2" value="1.57079632679489661923"/>
     <material name="blue_aluminum">
-      <color rgba=".27 .45 .68 1"/>
+      <!-- more accurate but less pretty :) -->
+      <!--color rgba=".14 .24 .31 1"/>
+      <color rgba=".26 .44 .545 1"/-->
+      <color rgba=".23 .42 .64 1"/>
     </material>
     <link name="stand">
-      <visual>
-        <origin rpy="0 0 0" xyz="0 0 0"/>
-        <geometry>
-          <mesh filename="package://tahoma_description/meshes/stand/visual/stand_base.stl"/>
-        </geometry>
-        <material name="blue_aluminum"/>
-      </visual>
-      <collision>
-        <origin rpy="0 0 0" xyz="0 0 0"/>
-        <geometry>
-          <mesh filename="package://tahoma_description/meshes/stand/visual/stand_base.stl"/>
+      <inertial>
+        <mass value="10.0"/>
+        <inertia ixx="0.0002835" ixy="0.0" ixz="0.0" iyy="0.0002835" iyz="0.0" izz="0.000324"/>
+      </inertial>
+      <visual>
+        <origin rpy="0 0 0" xyz="0 0 0"/>
+        <geometry>
+          <mesh filename="package://tahoma_description/meshes/stand/stand_base.stl"/>
+        </geometry>
+        <material name="blue_aluminum"/>
+      </visual>
+      <collision>
+        <!-- across -->
+        <origin rpy="0 0 0" xyz=".4050 0 .0281"/>
+        <geometry>
+          <box size=".09 1.53 .045"/>
+        </geometry>
+      </collision>
+      <collision>
+        <!-- right -->
+        <origin rpy="0 0 0" xyz="0 -.72 -.0225"/>
+        <geometry>
+          <box size=".9 .09 .0562"/>
+        </geometry>
+      </collision>
+      <collision>
+        <!-- left -->
+        <origin rpy="0 0 0" xyz="0 .72 -.0225"/>
+        <geometry>
+          <box size=".9 .09 .0562"/>
         </geometry>
       </collision>
     </link>
     <link name="stand_upright">
-      <visual>
-        <origin rpy="0 0 0" xyz="0 0 0"/>
-        <geometry>
-          <mesh filename="package://tahoma_description/meshes/stand/visual/stand_upright.stl"/>
-        </geometry>
-        <material name="blue_aluminum"/>
-      </visual>
-      <collision>
-        <origin rpy="0 0 0" xyz="0 0 0"/>
-        <geometry>
-          <mesh filename="package://tahoma_description/meshes/stand/visual/stand_upright.stl"/>
+      <inertial>
+        <mass value="34"/>
+        <inertia ixx="0.0002835" ixy="0.0" ixz="0.0" iyy="0.0002835" iyz="0.0" izz="0.000324"/>
+      </inertial>
+      <visual>
+        <origin rpy="0 0 0" xyz="0 0 0"/>
+        <geometry>
+          <mesh filename="package://tahoma_description/meshes/stand/stand_upright.stl"/>
+        </geometry>
+        <material name="blue_aluminum"/>
+      </visual>
+      <collision>
+        <!-- right upright -->
+        <origin rpy="0 0 0" xyz="-.1709 0.6975 0"/>
+        <geometry>
+          <box size=".2298 .0450 1.89"/>
+        </geometry>
+      </collision>
+      <collision>
+        <!-- left upright -->
+        <origin rpy="0 0 0" xyz="-.1709 -0.6975 0"/>
+        <geometry>
+          <box size=".2298 .0450 1.89"/>
+        </geometry>
+      </collision>
+      <collision>
+        <!-- top beam -->
+        <origin rpy="0 0 0" xyz="-.1733 0 .9012"/>
+        <geometry>
+          <box size=".2370 1.44 .0960"/>
         </geometry>
       </collision>
     </link>
     <link name="stand_brace">
-      <visual>
-        <origin rpy="0 0 0" xyz="0 0 0"/>
-        <geometry>
-          <mesh filename="package://tahoma_description/meshes/stand/visual/stand_brace.stl"/>
-        </geometry>
-        <material name="blue_aluminum"/>
-      </visual>
-      <collision>
-        <origin rpy="0 0 0" xyz="0 0 0"/>
-        <geometry>
-          <mesh filename="package://tahoma_description/meshes/stand/visual/stand_brace.stl"/>
-        </geometry>
-      </collision>
-    </link>
-    <link name="robot_beam">
-      <visual>
-        <origin rpy="0 0 0" xyz="0 0 0"/>
-        <geometry>
-          <mesh filename="package://tahoma_description/meshes/stand/visual/robot_beam.stl"/>
-        </geometry>
-        <material name="blue_aluminum"/>
-      </visual>
-      <collision>
-        <origin rpy="0 0 0" xyz="0 0 0"/>
-        <geometry>
-          <mesh filename="package://tahoma_description/meshes/stand/visual/robot_beam.stl"/>
+      <inertial>
+        <mass value="5"/>
+        <inertia ixx="0.0002835" ixy="0.0" ixz="0.0" iyy="0.0002835" iyz="0.0" izz="0.000324"/>
+      </inertial>
+      <visual>
+        <origin rpy="0 0 0" xyz="0 0 0"/>
+        <geometry>
+          <mesh filename="package://tahoma_description/meshes/stand/stand_brace.stl"/>
+        </geometry>
+        <material name="blue_aluminum"/>
+      </visual>
+      <collision>
+        <origin rpy="0 0 0" xyz="0 0 0"/>
+        <geometry>
+          <box size=".102 1.4390 .4934"/>
+        </geometry>
+      </collision>
+    </link>
+    <link name="cantilever">
+      <inertial>
+        <mass value="8"/>
+        <inertia ixx="0.0002835" ixy="0.0" ixz="0.0" iyy="0.0002835" iyz="0.0" izz="0.000324"/>
+      </inertial>
+      <visual>
+        <origin rpy="0 0 0" xyz="0 0 0"/>
+        <geometry>
+          <mesh filename="package://tahoma_description/meshes/stand/cantilever.stl"/>
+        </geometry>
+        <material name="blue_aluminum"/>
+      </visual>
+      <collision>
+        <origin xyz="0 0 .0415"/>
+        <geometry>
+          <box size=".7260 .225 .09"/>
         </geometry>
       </collision>
     </link>
     <link name="control_box_mount">
-      <visual>
-        <origin rpy="0 0 0" xyz="0 0 0"/>
-        <geometry>
-          <mesh filename="package://tahoma_description/meshes/stand/visual/control_box_mount.stl"/>
-        </geometry>
-        <material name="blue_aluminum"/>
-      </visual>
-      <collision>
-        <origin rpy="0 0 0" xyz="0 0 0"/>
-        <geometry>
-          <mesh filename="package://tahoma_description/meshes/stand/visual/control_box_mount.stl"/>
+      <inertial>
+        <mass value="3"/>
+        <inertia ixx="0.0002835" ixy="0.0" ixz="0.0" iyy="0.0002835" iyz="0.0" izz="0.000324"/>
+      </inertial>
+      <visual>
+        <origin rpy="0 0 0" xyz="0 0 0"/>
+        <geometry>
+          <mesh filename="package://tahoma_description/meshes/stand/control_box_mount.stl"/>
+        </geometry>
+        <material name="blue_aluminum"/>
+      </visual>
+      <collision>
+        <origin rpy="0 0 0" xyz="0 0 0"/>
+        <geometry>
+          <box size=".585 .0602 .1790"/>
+        </geometry>
+      </collision>
+    </link>
+    <link name="control_box">
+      <inertial>
+        <mass value="7"/>
+        <inertia ixx="0.0002835" ixy="0.0" ixz="0.0" iyy="0.0002835" iyz="0.0" izz="0.000324"/>
+      </inertial>
+      <visual>
+        <origin rpy="0 0 0" xyz="0 0 0"/>
+        <geometry>
+          <mesh filename="package://tahoma_description/meshes/stand/control_box.stl"/>
+        </geometry>
+        <material name="aluminum"/>
+      </visual>
+      <collision>
+        <origin rpy="0 0 0" xyz="0 0 0"/>
+        <geometry>
+          <box size=".46 .25 .44"/>
         </geometry>
       </collision>
     </link>
     <link name="robot_plate">
-      <visual>
-        <origin rpy="0 0 0" xyz="0 0 0"/>
-        <geometry>
-          <mesh filename="package://tahoma_description/meshes/stand/visual/robot_plate.stl"/>
-        </geometry>
-        <material name="blue_aluminum"/>
-      </visual>
-      <collision>
-        <origin rpy="0 0 0" xyz="0 0 0"/>
-        <geometry>
-          <mesh filename="package://tahoma_description/meshes/stand/visual/robot_plate.stl"/>
+      <inertial>
+        <mass value=".5"/>
+        <inertia ixx="0.0002835" ixy="0.0" ixz="0.0" iyy="0.0002835" iyz="0.0" izz="0.000324"/>
+      </inertial>
+      <visual>
+        <origin rpy="0 0 0" xyz="0 0 0"/>
+        <geometry>
+          <mesh filename="package://tahoma_description/meshes/stand/robot_plate.stl"/>
+        </geometry>
+        <material name="blue_aluminum"/>
+      </visual>
+      <collision>
+        <origin rpy="0 0 0" xyz="0 0 0"/>
+        <geometry>
+          <box size=".225 .225 .0225"/>
         </geometry>
       </collision>
@@ -120,13 +196,18 @@
       <origin rpy="0 0 0" xyz="-.1725 .7475 0"/>
     </joint>
-    <joint name="stand_robot_beam_joint" type="fixed">
-      <parent link="stand_upright"/>
-      <child link="robot_beam"/>
+    <joint name="control_box_mount_control_box_joint" type="fixed">
+      <parent link="control_box_mount"/>
+      <child link="control_box"/>
+      <origin rpy="0.05 0 ${M_PI}" xyz="-.003 .1375 -0.13"/>
+    </joint>
+    <joint name="stand_cantilever_joint" type="fixed">
+      <parent link="stand_upright"/>
+      <child link="cantilever"/>
       <origin rpy="0 0 0" xyz=".0775 0  0.9475"/>
     </joint>
-    <joint name="robot_beam_robot_plate_joint" type="fixed">
-      <parent link="robot_beam"/>
+    <joint name="cantilever_robot_plate_joint" type="fixed">
+      <parent link="cantilever"/>
       <child link="robot_plate"/>
-      <origin rpy="0 0 0" xyz="0.2 0 -.015"/>
+      <origin rpy="0 0 0" xyz="0.2505 0 -.015"/>
     </joint>
     <joint name="stand_front_right_caster_joint" type="fixed">

Commit message: Add Robotiq coupling
It's particular to e series integration and not reflected in most URDFs floating around
GRP-ES-CPL-062

File: tahoma_description/robots/tahoma.xacro (robot description, xacro)
@@ -7,5 +7,4 @@
   <xacro:arg name="realsense" default="true" />
   <xacro:arg name="transmission_hw_interface" default="hardware_interface/EffortJointInterface"/>
-  <xacro:property name="M_PI" value="3.1415926535897931"/>
   <xacro:stand/>
   <xacro:ur16e_robot prefix="arm_"/>
@@ -22,9 +21,30 @@
     <parent link="robot_plate"/>
     <child link="arm_base_link"/>
-    <origin rpy="0 ${M_PI} ${M_PI}" xyz="0 -0.01 0"/>
+    <origin rpy="0 ${pi} ${pi}" xyz="0 -0.01 0"/>
   </joint>
-  <joint name="arm_tool0-gripper_robotiq_arg2f_base_link" type="fixed">
+  <link name="coupling">
+    <visual>
+      <origin xyz="0 0 0" rpy="0 0 ${pi}" />
+      <geometry>
+        <mesh filename="package://tahoma_description/meshes/robotiq_gripper_coupling.stl"/>
+      </geometry>
+      <material name="">
+        <color rgba="0.1 0.1 0.1 1" />
+      </material>
+    </visual>
+    <collision>
+      <geometry>
+          <cylinder radius=".0375" length=".0139"/>
+      </geometry>
+    </collision>
+  </link>
+  <joint name="coupling_link_gripper_robotiq_arg2f_base_link_joint" type="fixed">
+    <origin xyz="0 0 0.008" rpy="0 0 ${pi/2}"/>
+    <parent link="coupling" />
+    <child link="gripper_base_link" />
+  </joint>
+  <joint name="arm_tool0-coupling_joint" type="fixed">
     <parent link="arm_tool0"/>
-    <child link="gripper_base_link"/>
+    <child link="coupling"/>
   </joint>
   <link name="mid_camera_mount"/>

Commit message: Fix robot mount orientation and offset
For real this time ;)

File: tahoma_description/robots/tahoma.xacro (robot description, xacro)
@@ -21,5 +21,5 @@
     <parent link="robot_plate"/>
     <child link="arm_base_link"/>
-    <origin rpy="0 ${pi} ${pi}" xyz="0 -0.01 0"/>
+    <origin rpy="0 ${pi} ${1.5 * pi}" xyz="0 0.0 -0.01125"/>
   </joint>
   <link name="coupling">

Commit message: adjust stand_camera xyz position to reflect reality

File: tahoma_description/robots/tahoma.xacro (robot description, xacro)
@@ -50,10 +50,10 @@
   <link name="mid_camera_mount"/>
   <joint name="stand_upright_mid_camera_mount_joint" type="fixed">
-      <parent link="stand_upright"/>
+      <parent link="stand_brace"/>
       <child link="mid_camera_mount"/>
-      <origin rpy="0 0 0" xyz="-.2 0 0"/>
+      <origin rpy="0 0 0" xyz="0 0 0"/>
   </joint>
   <xacro:sensor_l515 name="stand_camera" parent="mid_camera_mount" use_nominal_extrinsics="true">
-      <origin xyz="0.025 -0.025 0.003" rpy="0 0 0"/>
+      <origin xyz="0.125 0 0.685" rpy="0 0 0" /> <!-- z = 0.245 + 0.44 = 0.685   x=0.045+0.08=0.125-->
   </xacro:sensor_l515>
 </robot>

Commit message: Hack first-pick bits into shape
Make planning scene synchronous to force geometry to update before proceeding
Move collision geometry into states that check for the successful addition of the geometry before returning
Don't check for collisions when doing cartesian grasp approach, lift, and extract motions
Ask for gripper to be opened before executing the grasp linear motion (because there's no guarantee it's open otherwise)
Query for points in base link to make debugging easier, avoid coordinates that change when the arm moves out of the hide pose
Tune camera calibration
Move control box mount up to match real robot
Declare realsense2_camera dependency
Install and launch grasp code correctly
Fix usage errors in grasp pose calculations
Compensate for occlusion induced z bias in grasp pose selection with manual offset

File: tahoma_description/robots/tahoma.xacro (robot description, xacro)
@@ -49,11 +49,11 @@
   </joint>
   <link name="mid_camera_mount"/>
-  <joint name="stand_upright_mid_camera_mount_joint" type="fixed">
+  <joint name="stand_brace_mid_camera_mount_joint" type="fixed">
       <parent link="stand_brace"/>
       <child link="mid_camera_mount"/>
-      <origin rpy="0 0 0" xyz="0 0 0"/>
+      <origin xyz="0.1375 0.075 0.685" rpy="0 0 0"/>
   </joint>
   <xacro:sensor_l515 name="stand_camera" parent="mid_camera_mount" use_nominal_extrinsics="true">
-      <origin xyz="0.125 0 0.685" rpy="0 0 0" /> <!-- z = 0.245 + 0.44 = 0.685   x=0.045+0.08=0.125-->
+      <origin xyz="0 0 0" rpy="0 0 0" /> <!-- z = 0.245 + 0.44 = 0.685   x=0.045+0.08=0.125-->
   </xacro:sensor_l515>
 </robot>

File: tahoma_description/urdf/stand.xacro (robot description, xacro)
@@ -194,5 +194,5 @@
       <parent link="stand_upright"/>
       <child link="control_box_mount"/>
-      <origin rpy="0 0 0" xyz="-.1725 .7475 0"/>
+      <origin rpy="0 0 0" xyz="-.1725 .7475 .21"/>
     </joint>
     <joint name="control_box_mount_control_box_joint" type="fixed">

Commit message: Tune stand model
Add offsets to robot mount, cantilever and gripper based on placing the end effector (at the end of the UR, before the coupling) up against parts of the frame and manually adjusting
Add fake gripper node which publishes gripper aperture state so that we can visualize the gripper on the robot without the working driver
Add pod to robot bringup, making its frames accessible to tasks programs
Attach camera to the new beam

Co-authored-by: Collin Dang <collindang88@gmail.com>

File: tahoma_description/robots/tahoma.xacro (robot description, xacro)
@@ -21,5 +21,5 @@
     <parent link="robot_plate"/>
     <child link="arm_base_link"/>
-    <origin rpy="0 ${pi} ${1.5 * pi}" xyz="0 0.0 -0.01125"/>
+    <origin rpy="0 ${pi} ${1.5 * pi}" xyz="0 0.00175 -0.00885"/>
   </joint>
   <link name="coupling">
@@ -40,5 +40,5 @@
   </link>
   <joint name="coupling_link_gripper_robotiq_arg2f_base_link_joint" type="fixed">
-    <origin xyz="0 0 0.008" rpy="0 0 ${pi/2}"/>
+    <origin xyz="0 0 0.012" rpy="0 0 ${pi/2}"/>
     <parent link="coupling" />
     <child link="gripper_base_link" />
@@ -49,8 +49,8 @@
   </joint>
   <link name="mid_camera_mount"/>
-  <joint name="stand_brace_mid_camera_mount_joint" type="fixed">
-      <parent link="stand_brace"/>
+  <joint name="camera_beam_lower_mid_camera_mount_joint" type="fixed">
+      <parent link="camera_beam_lower"/>
       <child link="mid_camera_mount"/>
-      <origin xyz="0.1375 0.075 0.685" rpy="0 0 0"/>
+      <origin xyz="0.08 -0.075 0.07" rpy="0 0 0"/>
   </joint>
   <xacro:sensor_l515 name="stand_camera" parent="mid_camera_mount" use_nominal_extrinsics="true">

File: tahoma_description/urdf/stand.xacro (robot description, xacro)
@@ -213,5 +213,5 @@
       <parent link="stand_upright"/>
       <child link="camera_beam_lower"/>
-      <origin rpy="0 0 0" xyz="-.128 0 0"/>
+      <origin rpy="0 0 0" xyz="-.128 0 .15"/>
     </joint>
     <joint name="stand_upright_robot_control_box_mount_joint" type="fixed">
@@ -228,5 +228,5 @@
       <parent link="stand_upright"/>
       <child link="cantilever"/>
-      <origin rpy="0 0 0" xyz=".0775 0  0.9475"/>
+      <origin rpy="0 0 0" xyz=".0775 0  0.9442"/>
     </joint>
     <joint name="cantilever_robot_plate_joint" type="fixed">
