Commit message: Update lower camera configuration
Orient cameras on their side to maximize view of the pod
Add second camera, separate the cameras by a configurable baseline parameter, and orient cameras inward slightly to keep their FOV on the pod
Add hide pose to moveit config for easy retrieval
Raise camera beam to spend more pixels on reachable bins
Update default pod pose in view models launch

File: tahoma_description/robots/tahoma.xacro (robot description, xacro)
@@ -5,5 +5,7 @@
   <xacro:include filename="$(find robotiq_2f_85_gripper_visualization)/urdf/robotiq_arg2f_85_macro.xacro"/>
   <xacro:include filename="$(find realsense2_description)/urdf/_l515.urdf.xacro"/>
-  <xacro:arg name="realsense" default="true" />
+  <xacro:arg name="realsense" default="true"/>
+  <xacro:arg name="camera_baseline" default=".5"/>
+  <xacro:arg name="camera_focal_depth" default="1.4"/>
   <xacro:arg name="transmission_hw_interface" default="hardware_interface/EffortJointInterface"/>
   <xacro:stand/>
@@ -25,15 +27,15 @@
   <link name="coupling">
     <visual>
-      <origin xyz="0 0 0" rpy="0 0 ${pi}" />
+      <origin xyz="0 0 0" rpy="0 0 ${pi}"/>
       <geometry>
         <mesh filename="package://tahoma_description/meshes/robotiq_gripper_coupling.stl"/>
       </geometry>
       <material name="">
-        <color rgba="0.1 0.1 0.1 1" />
+        <color rgba="0.1 0.1 0.1 1"/>
       </material>
     </visual>
     <collision>
       <geometry>
-          <cylinder radius=".0375" length=".0139"/>
+        <cylinder radius=".0375" length=".0139"/>
       </geometry>
     </collision>
@@ -41,6 +43,6 @@
   <joint name="coupling_link_gripper_robotiq_arg2f_base_link_joint" type="fixed">
     <origin xyz="0 0 0.012" rpy="0 0 ${pi/2}"/>
-    <parent link="coupling" />
-    <child link="gripper_base_link" />
+    <parent link="coupling"/>
+    <child link="gripper_base_link"/>
   </joint>
   <joint name="arm_tool0-coupling_joint" type="fixed">
@@ -48,12 +50,24 @@
     <child link="coupling"/>
   </joint>
-  <link name="mid_camera_mount"/>
-  <joint name="camera_beam_lower_mid_camera_mount_joint" type="fixed">
-      <parent link="camera_beam_lower"/>
-      <child link="mid_camera_mount"/>
-      <origin xyz="0.08 -0.075 0.07" rpy="0 0 0"/>
+  <link name="camera_lower_right_mount"/>
+  <joint name="camera_beam_lower_camera_lower_right_mount_joint" type="fixed">
+    <parent link="camera_beam_lower"/>
+    <child link="camera_lower_right_mount"/>
+    <origin xyz="-0.00 ${-0.0215 + -$(arg camera_baseline) / 2} 0.09"
+            rpy="${-pi / 2} 0 ${math.atan2(($(arg camera_baseline) /2),$(arg camera_focal_depth))}"/>
   </joint>
-  <xacro:sensor_l515 name="stand_camera" parent="mid_camera_mount" use_nominal_extrinsics="true">
-      <origin xyz="0 0 0" rpy="0 0 0" /> <!-- z = 0.245 + 0.44 = 0.685   x=0.045+0.08=0.125-->
+  <link name="camera_lower_left_mount"/>
+  <joint name="camera_beam_lower_camera_lower_left_mount_joint" type="fixed">
+    <parent link="camera_beam_lower"/>
+    <child link="camera_lower_left_mount"/>
+    <!-- Link is centered on the optical frames. Slight offset in Y direction to compensate -->
+    <origin xyz="-0.00 ${-0.0215 + $(arg camera_baseline) / 2} 0.09"
+            rpy="${-pi / 2} 0 ${-math.atan2(($(arg camera_baseline) /2),$(arg camera_focal_depth))}"/>
+  </joint>
+  <xacro:sensor_l515 name="camera_lower_right" parent="camera_lower_right_mount" use_nominal_extrinsics="true">
+    <origin xyz="0 0 0" rpy="0 0 0"/>
+  </xacro:sensor_l515>
+  <xacro:sensor_l515 name="camera_lower_left" parent="camera_lower_left_mount" use_nominal_extrinsics="true">
+    <origin xyz="0 0 0" rpy="0 0 0"/>
   </xacro:sensor_l515>
 </robot>

File: tahoma_description/urdf/stand.xacro (robot description, xacro)
@@ -211,5 +211,5 @@
       <parent link="stand_upright"/>
       <child link="camera_beam_lower"/>
-      <origin rpy="0 0 0" xyz="-.128 0 .15"/>
+      <origin rpy="0 0 0" xyz="-.228 0 .35"/>
     </joint>
     <joint name="stand_upright_robot_control_box_mount_joint" type="fixed">

Commit message: Centralize calibrations into transform launch files
This makes it easier to change the values while the system is live, then relaunch the transform broadcaster and see the updates
Add placeholder identity calibrations for camera mounts

File: tahoma_description/robots/tahoma.xacro (robot description, xacro)
@@ -6,12 +6,30 @@
   <xacro:include filename="$(find realsense2_description)/urdf/_l515.urdf.xacro"/>
   <xacro:arg name="realsense" default="true"/>
+  <xacro:arg name="use_nominal_camera_extrinsics" default="false"/>
   <xacro:arg name="camera_baseline" default=".5"/>
   <xacro:arg name="camera_focal_depth" default="1.4"/>
-  <xacro:arg name="transmission_hw_interface" default="hardware_interface/EffortJointInterface"/>
+  <xacro:arg name="gripper_transmission_hw_interface" default="hardware_interface/EffortJointInterface" />
+  <xacro:arg name="joint_limits_params" default="$(find ur_description)/config/ur16e/joint_limits.yaml" />
+  <xacro:arg name="kinematics_params" default="$(find tahoma_description)/config/arm_calibration.yaml" />
+  <xacro:arg name="physical_params" default="$(find ur_description)/config/ur16e/physical_parameters.yaml" />
+  <xacro:arg name="visual_params"  default="$(find ur_description)/config/ur16e/visual_parameters.yaml" />
+  <!--common parameters  -->
+  <xacro:arg name="transmission_hw_interface" default="hardware_interface/PositionJointInterface" />
+  <xacro:arg name="safety_limits" default="false" />
+  <xacro:arg name="safety_pos_margin" default="0.15" />
+  <xacro:arg name="safety_k_position" default="20" />
   <xacro:stand/>
-  <xacro:ur16e_robot prefix="arm_"/>
+  <xacro:ur16e_robot prefix="arm_"
+      joint_limits_parameters_file="$(arg joint_limits_params)"
+      kinematics_parameters_file="$(arg kinematics_params)"
+      physical_parameters_file="$(arg physical_params)"
+      visual_parameters_file="$(arg visual_params)"
+      transmission_hw_interface="$(arg transmission_hw_interface)"
+      safety_limits="$(arg safety_limits)"
+      safety_pos_margin="$(arg safety_pos_margin)"
+      safety_k_position="$(arg safety_k_position)"/>
   <xacro:robotiq_arg2f_85
           prefix="gripper_"
-          transmission_hw_interface="$(arg transmission_hw_interface)"/>
+          transmission_hw_interface="$(arg gripper_transmission_hw_interface)"/>
   <link name="base_link"/>
   <joint name="base_joint" type="fixed">
@@ -51,11 +69,7 @@
   </joint>
   <link name="camera_lower_right_mount"/>
-  <joint name="camera_beam_lower_camera_lower_right_mount_joint" type="fixed">
-    <parent link="camera_beam_lower"/>
-    <child link="camera_lower_right_mount"/>
-    <origin xyz="-0.00 ${-0.0215 + -$(arg camera_baseline) / 2} 0.09"
-            rpy="${-pi / 2} 0 ${math.atan2(($(arg camera_baseline) /2),$(arg camera_focal_depth))}"/>
-  </joint>
   <link name="camera_lower_left_mount"/>
+  <!-- These are the planned ("nominal") mount placements. On the real system, these should
+       be overridden by calibrated transforms published separately -->
   <joint name="camera_beam_lower_camera_lower_left_mount_joint" type="fixed">
     <parent link="camera_beam_lower"/>
@@ -65,8 +79,14 @@
             rpy="${-pi / 2} 0 ${-math.atan2(($(arg camera_baseline) /2),$(arg camera_focal_depth))}"/>
   </joint>
-  <xacro:sensor_l515 name="camera_lower_right" parent="camera_lower_right_mount" use_nominal_extrinsics="true">
+  <joint name="camera_beam_lower_camera_lower_right_mount_joint" type="fixed">
+    <parent link="camera_beam_lower"/>
+    <child link="camera_lower_right_mount"/>
+    <origin xyz="-0.00 ${-0.0215 + -$(arg camera_baseline) / 2} 0.09"
+            rpy="${-pi / 2} 0 ${math.atan2(($(arg camera_baseline) /2),$(arg camera_focal_depth))}"/>
+  </joint>
+  <xacro:sensor_l515 name="camera_lower_right" parent="camera_lower_right_mount" use_nominal_extrinsics="$(arg use_nominal_camera_extrinsics)">
     <origin xyz="0 0 0" rpy="0 0 0"/>
   </xacro:sensor_l515>
-  <xacro:sensor_l515 name="camera_lower_left" parent="camera_lower_left_mount" use_nominal_extrinsics="true">
+  <xacro:sensor_l515 name="camera_lower_left" parent="camera_lower_left_mount" use_nominal_extrinsics="$(arg use_nominal_camera_extrinsics)">
     <origin xyz="0 0 0" rpy="0 0 0"/>
   </xacro:sensor_l515>

Commit message: Refactor Tahmoma into a macro
Check and pass through parameters from launch through to the UR16e macro
Using macro params makes it possible for the gazebo wrapper to turn on the default camera extrinsics without relying on the xacro caller to configure an argument
This macro makes it easier to create a full workspace URDF by including the robot and a pod

File: tahoma_description/robots/tahoma.xacro (robot description, xacro)
@@ -1,93 +1,9 @@
 <?xml version="1.0"?>
 <robot xmlns:xacro="http://www.ros.org/wiki/xacro" name="tahoma">
-  <xacro:include filename="$(find ur_description)/urdf/inc/ur16e_macro.xacro"/>
-  <xacro:include filename="$(find tahoma_description)/urdf/stand.xacro"/>
-  <xacro:include filename="$(find robotiq_2f_85_gripper_visualization)/urdf/robotiq_arg2f_85_macro.xacro"/>
-  <xacro:include filename="$(find realsense2_description)/urdf/_l515.urdf.xacro"/>
+  <xacro:arg name="kinematics_params" default="$(find tahoma_description)/config/arm_calibration.yaml" />
   <xacro:arg name="realsense" default="true"/>
   <xacro:arg name="use_nominal_camera_extrinsics" default="false"/>
-  <xacro:arg name="camera_baseline" default=".5"/>
-  <xacro:arg name="camera_focal_depth" default="1.4"/>
-  <xacro:arg name="gripper_transmission_hw_interface" default="hardware_interface/EffortJointInterface" />
-  <xacro:arg name="joint_limits_params" default="$(find ur_description)/config/ur16e/joint_limits.yaml" />
-  <xacro:arg name="kinematics_params" default="$(find tahoma_description)/config/arm_calibration.yaml" />
-  <xacro:arg name="physical_params" default="$(find ur_description)/config/ur16e/physical_parameters.yaml" />
-  <xacro:arg name="visual_params"  default="$(find ur_description)/config/ur16e/visual_parameters.yaml" />
-  <!--common parameters  -->
-  <xacro:arg name="transmission_hw_interface" default="hardware_interface/PositionJointInterface" />
   <xacro:arg name="safety_limits" default="false" />
-  <xacro:arg name="safety_pos_margin" default="0.15" />
-  <xacro:arg name="safety_k_position" default="20" />
-  <xacro:stand/>
-  <xacro:ur16e_robot prefix="arm_"
-      joint_limits_parameters_file="$(arg joint_limits_params)"
-      kinematics_parameters_file="$(arg kinematics_params)"
-      physical_parameters_file="$(arg physical_params)"
-      visual_parameters_file="$(arg visual_params)"
-      transmission_hw_interface="$(arg transmission_hw_interface)"
-      safety_limits="$(arg safety_limits)"
-      safety_pos_margin="$(arg safety_pos_margin)"
-      safety_k_position="$(arg safety_k_position)"/>
-  <xacro:robotiq_arg2f_85
-          prefix="gripper_"
-          transmission_hw_interface="$(arg gripper_transmission_hw_interface)"/>
-  <link name="base_link"/>
-  <joint name="base_joint" type="fixed">
-    <origin rpy="0 0 0" xyz="0 0 0.15"/>
-    <parent link="base_link"/>
-    <child link="stand"/>
-  </joint>
-  <joint name="robot_plate_arm_base_link_joint" type="fixed">
-    <parent link="robot_plate"/>
-    <child link="arm_base_link"/>
-    <origin rpy="0 ${pi} ${1.5 * pi}" xyz="0 0.00175 -0.00885"/>
-  </joint>
-  <link name="coupling">
-    <visual>
-      <origin xyz="0 0 0" rpy="0 0 ${pi}"/>
-      <geometry>
-        <mesh filename="package://tahoma_description/meshes/robotiq_gripper_coupling.stl"/>
-      </geometry>
-      <material name="">
-        <color rgba="0.1 0.1 0.1 1"/>
-      </material>
-    </visual>
-    <collision>
-      <geometry>
-        <cylinder radius=".0375" length=".0139"/>
-      </geometry>
-    </collision>
-  </link>
-  <joint name="coupling_link_gripper_robotiq_arg2f_base_link_joint" type="fixed">
-    <origin xyz="0 0 0.012" rpy="0 0 ${pi/2}"/>
-    <parent link="coupling"/>
-    <child link="gripper_base_link"/>
-  </joint>
-  <joint name="arm_tool0-coupling_joint" type="fixed">
-    <parent link="arm_tool0"/>
-    <child link="coupling"/>
-  </joint>
-  <link name="camera_lower_right_mount"/>
-  <link name="camera_lower_left_mount"/>
-  <!-- These are the planned ("nominal") mount placements. On the real system, these should
-       be overridden by calibrated transforms published separately -->
-  <joint name="camera_beam_lower_camera_lower_left_mount_joint" type="fixed">
-    <parent link="camera_beam_lower"/>
-    <child link="camera_lower_left_mount"/>
-    <!-- Link is centered on the optical frames. Slight offset in Y direction to compensate -->
-    <origin xyz="-0.00 ${-0.0215 + $(arg camera_baseline) / 2} 0.09"
-            rpy="${-pi / 2} 0 ${-math.atan2(($(arg camera_baseline) /2),$(arg camera_focal_depth))}"/>
-  </joint>
-  <joint name="camera_beam_lower_camera_lower_right_mount_joint" type="fixed">
-    <parent link="camera_beam_lower"/>
-    <child link="camera_lower_right_mount"/>
-    <origin xyz="-0.00 ${-0.0215 + -$(arg camera_baseline) / 2} 0.09"
-            rpy="${-pi / 2} 0 ${math.atan2(($(arg camera_baseline) /2),$(arg camera_focal_depth))}"/>
-  </joint>
-  <xacro:sensor_l515 name="camera_lower_right" parent="camera_lower_right_mount" use_nominal_extrinsics="$(arg use_nominal_camera_extrinsics)">
-    <origin xyz="0 0 0" rpy="0 0 0"/>
-  </xacro:sensor_l515>
-  <xacro:sensor_l515 name="camera_lower_left" parent="camera_lower_left_mount" use_nominal_extrinsics="$(arg use_nominal_camera_extrinsics)">
-    <origin xyz="0 0 0" rpy="0 0 0"/>
-  </xacro:sensor_l515>
+  <xacro:include filename="$(find tahoma_description)/urdf/tahoma.xacro"/>
+  <xacro:tahoma safety_limits="$(arg safety_limits)" use_nominal_camera_extrinsics="$(arg use_nominal_camera_extrinsics)" kinematics_parameters_file="$(arg kinematics_params)" />
 </robot>

Commit message: Add xacro argument for toggling camera arrangement
Add tilted configuration ahead of next draft of mounts
Add coarse collision bounding box to prevent further robot to camera collisions

File: tahoma_description/robots/tahoma.xacro (robot description, xacro)
@@ -1,4 +1,5 @@
 <?xml version="1.0"?>
 <robot xmlns:xacro="http://www.ros.org/wiki/xacro" name="tahoma">
+  <xacro:arg name="camera_arrangement" default="manual" />
   <xacro:arg name="kinematics_params" default="$(find tahoma_description)/config/arm_calibration.yaml" />
   <xacro:arg name="realsense" default="true"/>
@@ -6,4 +7,4 @@
   <xacro:arg name="safety_limits" default="false" />
   <xacro:include filename="$(find tahoma_description)/urdf/tahoma.xacro"/>
-  <xacro:tahoma safety_limits="$(arg safety_limits)" use_nominal_camera_extrinsics="$(arg use_nominal_camera_extrinsics)" kinematics_parameters_file="$(arg kinematics_params)" />
+  <xacro:tahoma camera_arrangement="$(arg camera_arrangement)" safety_limits="$(arg safety_limits)" use_nominal_camera_extrinsics="$(arg use_nominal_camera_extrinsics)" kinematics_parameters_file="$(arg kinematics_params)" />
 </robot>

File: tahoma_description/urdf/tahoma.xacro (robot description, xacro)
@@ -8,4 +8,5 @@
   realsense:=true
   use_nominal_camera_extrinsics:=false
+  camera_arrangement:='manual'
   camera_baseline:=.5
   camera_focal_depth:=1.4
@@ -87,20 +88,93 @@
       <child link="coupling"/>
     </joint>
-    <link name="camera_lower_right_mount"/>
-    <link name="camera_lower_left_mount"/>
+    <link name="camera_lower_right_mount">
+      <collision>
+        <origin xyz="0 0 0" rpy="0 0 0"/>
+        <geometry>
+          <box size=".1 .15 .15"/>
+        </geometry>
+      </collision>
+    </link>
+    <link name="camera_lower_left_mount">
+      <collision>
+        <origin xyz="0 0 0" rpy="0 0 0"/>
+        <geometry>
+          <box size=".1 .15 .15"/>
+        </geometry>
+      </collision>
+    </link>
     <!-- These are the planned ("nominal") mount placements. On the real system, these should
-         be overridden by calibrated transforms published separately -->
-    <joint name="camera_beam_lower_camera_lower_left_mount_joint" type="fixed">
-      <parent link="camera_beam_lower"/>
-      <child link="camera_lower_left_mount"/>
-      <!-- Link is centered on the optical frames. Slight offset in Y direction to compensate -->
-      <origin xyz="-0.00 0.02 0.06"
-              rpy="0 0 0"/>
+     be overridden by calibrated transforms published separately -->
+    <xacro:if value="${camera_arrangement == 'manual' }">
+      <joint name="camera_beam_lower_camera_lower_left_mount_joint" type="fixed">
+        <parent link="camera_beam_lower"/>
+        <child link="camera_lower_left_mount"/>
+        <!-- Link is centered on the optical frames. Slight offset in Y direction to compensate -->
+        <origin xyz="-0.00 0.02 0.06"
+                rpy="0 0 0"/>
+      </joint>
+      <joint name="camera_beam_lower_camera_lower_right_mount_joint" type="fixed">
+        <parent link="camera_beam_lower"/>
+        <child link="camera_lower_right_mount"/>
+        <origin xyz="-0.00 ${-0.0215 + -camera_baseline / 2} 0.09"
+                rpy="${pi / 2} 0 ${math.atan2((camera_baseline /2),camera_focal_depth)}"/>
+      </joint>
+    </xacro:if>
+    <xacro:if value="${camera_arrangement == 'convergent' }">
+      <joint name="camera_beam_lower_camera_lower_left_mount_joint" type="fixed">
+        <parent link="camera_beam_lower"/>
+        <child link="camera_lower_left_mount"/>
+        <!-- Link is centered on the optical frames. Slight offset in Y direction to compensate -->
+        <origin xyz="0 ${-0.0215 + -camera_baseline / 2} 0.09"
+                rpy="${pi / 2} 0 ${-math.atan2((camera_baseline /2),camera_focal_depth)}"/>
+      </joint>
+      <joint name="camera_beam_lower_camera_lower_right_mount_joint" type="fixed">
+        <parent link="camera_beam_lower"/>
+        <child link="camera_lower_right_mount"/>
+        <origin xyz="0 ${-0.0215 + -camera_baseline / 2} 0.09"
+                rpy="${pi / 2} 0 ${math.atan2((camera_baseline /2),camera_focal_depth)}"/>
+      </joint>
+    </xacro:if>
+    <xacro:if value="${camera_arrangement == 'convergent_tilted' }">
+      <joint name="camera_beam_lower_camera_lower_left_mount_joint" type="fixed">
+        <parent link="camera_beam_lower"/>
+        <child link="camera_lower_left_mount"/>
+        <!-- Link is centered on the optical frames. Slight offset in Y direction to compensate -->
+        <origin xyz="-0.00 ${-0.0215 + (camera_baseline / 2)} 0.09"
+                rpy="${pi / 2} ${radians(15)} ${-math.atan2((camera_baseline /2),camera_focal_depth)}"/>
+      </joint>
+      <joint name="camera_beam_lower_camera_lower_right_mount_joint" type="fixed">
+        <parent link="camera_beam_lower"/>
+        <child link="camera_lower_right_mount"/>
+        <origin xyz="-0.00 ${0.0215 + (-camera_baseline / 2)} 0.09"
+                rpy="${pi / 2} ${radians(15)} ${math.atan2((camera_baseline /2),camera_focal_depth)}"/>
+      </joint>
+    </xacro:if>
+    <!-- Upper cameras -->
+    <!-- Link is centered on the optical frames. Slight offset in Y direction to compensate -->
+    <!-- Z=1.10 for on top of the top beam -->
+    <!-- Z=0.80 for underneath the top beam -->
+    <!-- Disabled until we know about manipulability in upper bins
+    <link name="camera_upper_right_mount"/>
+    <link name="camera_upper_left_mount"/>
+    <joint name="stand_upright_camera_upper_left_mount_joint" type="fixed">
+      <parent link="stand_upright"/>
+      <child link="camera_upper_left_mount"/>
+      <origin xyz="-.1 ${-0.0215 + (camera_baseline / 2)} 0.80"
+              rpy="${pi / 2} ${radians(15)} ${-math.atan2((camera_baseline /2),camera_focal_depth)}"/>
     </joint>
-    <joint name="camera_beam_lower_camera_lower_right_mount_joint" type="fixed">
-      <parent link="camera_beam_lower"/>
-      <child link="camera_lower_right_mount"/>
-      <origin xyz="-0.00 ${-0.0215 + -camera_baseline / 2} 0.09"
-              rpy="${pi / 2} 0 ${math.atan2((camera_baseline /2),camera_focal_depth)}"/>
+    <joint name="stand_upright_camera_upper_right_mount_joint" type="fixed">
+      <parent link="stand_upright"/>
+      <child link="camera_upper_right_mount"/>
+      <origin xyz="-.1 ${0.0215 + (-camera_baseline / 2)} 0.80"
+              rpy="${pi / 2} ${radians(15)} ${math.atan2((camera_baseline /2),camera_focal_depth)}"/>
+    </joint>
+    -->
+    <link name="camera_upper_mount"/>
+    <joint name="cantilever_camera_upper_mount_joint" type="fixed">
+      <parent link="cantilever"/>
+      <child link="camera_upper_mount"/>
+      <origin xyz=".02 0 0.37"
+              rpy="0 ${radians(15)} 0"/>
     </joint>
     <xacro:if value="${realsense}">
@@ -111,4 +185,14 @@
         <origin xyz="0 0 0" rpy="0 0 0"/>
       </xacro:sensor_l515>
+      <xacro:sensor_l515 name="camera_upper" parent="camera_upper_mount" use_nominal_extrinsics="${use_nominal_camera_extrinsics}">
+        <origin xyz="0 0 0" rpy="0 0 0"/>
+      </xacro:sensor_l515>
+      <!-- Upper cameras
+      <xacro:sensor_l515 name="camera_upper_right" parent="camera_upper_right_mount" use_nominal_extrinsics="${use_nominal_camera_extrinsics}">
+        <origin xyz="0 0 0" rpy="0 0 0"/>
+      </xacro:sensor_l515>
+      <xacro:sensor_l515 name="camera_upper_left" parent="camera_upper_left_mount" use_nominal_extrinsics="${use_nominal_camera_extrinsics}">
+        <origin xyz="0 0 0" rpy="0 0 0"/>
+      </xacro:sensor_l515> -->
     </xacro:if>
   </xacro:macro>
