Commit message: Update on new computer

File: tahoma_description/robots/tahoma.xacro (robot description, xacro)
@@ -3,5 +3,6 @@
   <xacro:arg name="camera_arrangement" default="manual" />
   <xacro:arg name="kinematics_params" default="$(find tahoma_description)/config/arm_calibration.yaml" />
-  <xacro:arg name="realsense" default="true"/>
+  <xacro:arg name="realsense" default="false"/>
+  <xacro:arg name="azure_kinect" default="true"/>
   <xacro:arg name="use_nominal_camera_extrinsics" default="false"/>
   <xacro:arg name="safety_limits" default="false" />

File: tahoma_description/urdf/tahoma.xacro (robot description, xacro)
@@ -4,7 +4,8 @@
   <xacro:include filename="$(find tahoma_description)/urdf/stand.xacro"/>
   <xacro:include filename="$(find robotiq_2f_85_gripper_visualization)/urdf/robotiq_arg2f_85_macro.xacro"/>
-  <xacro:include filename="$(find realsense2_description)/urdf/_l515.urdf.xacro"/>
+  <!-- <xacro:include filename="$(find realsense2_description)/urdf/_l515.urdf.xacro"/> -->
   <xacro:macro name="tahoma" params="
-  realsense:=true
+  realsense:=false
+  azure_kinect:=true
   use_nominal_camera_extrinsics:=false
   camera_arrangement:='manual'
@@ -178,4 +179,14 @@
               rpy="0 ${radians(15)} 0"/>
     </joint>
+    <xacro:if value="${azure_kinect}">
+      <xacro:include filename="$(find tahoma_description)/urdf/azure_kinect.urdf.xacro"/>
+      <joint name="kinect_base_joint" type="fixed">
+        <parent link="camera_beam_lower"/>
+        <child link="camera_base"/>
+        <!-- Link is centered on the optical frames. Slight offset in Y direction to compensate -->
+        <origin xyz="0 0 .09"
+                rpy="0 0 0"/>
+      </joint>
+    </xacro:if>
     <xacro:if value="${realsense}">
       <xacro:sensor_l515 name="camera_lower_right" parent="camera_lower_right_mount" use_nominal_extrinsics="${use_nominal_camera_extrinsics}">
@@ -188,5 +199,5 @@
         <origin xyz="0 0 0" rpy="0 0 0"/>
       </xacro:sensor_l515>
-      <!-- Upper cameras
+       <!-- Upper cameras -->
       <xacro:sensor_l515 name="camera_upper_right" parent="camera_upper_right_mount" use_nominal_extrinsics="${use_nominal_camera_extrinsics}">
         <origin xyz="0 0 0" rpy="0 0 0"/>
@@ -194,5 +205,5 @@
       <xacro:sensor_l515 name="camera_upper_left" parent="camera_upper_left_mount" use_nominal_extrinsics="${use_nominal_camera_extrinsics}">
         <origin xyz="0 0 0" rpy="0 0 0"/>
-      </xacro:sensor_l515> -->
+      </xacro:sensor_l515>
     </xacro:if>
   </xacro:macro>
