Commit message: IMPL: single files (pod.gazebo.xacro, robots/pod.xacro, urdf/pod.xacro) for 2 pods with 4 faces each are implemented/tested Also, MoveIt collision scene spawner function is implemented pod_sizes.yaml and end_effector_sizes.yaml files are created and used in tahoma.py

File: tahoma_description/urdf/pod.xacro (robot description, xacro)
@@ -1,30 +1,35 @@
 <?xml version="1.0"?>
-<robot xmlns:xacro="http://www.ros.org/wiki/xacro" name="pod_urdf">
+<robot xmlns:xacro="http://www.ros.org/wiki/xacro" name="pod">
   <xacro:macro name="pod_urdf" params="prefix:=pod_
-                                       BASE_WIDTH:=0.9400
-                                       BASE_HEIGHT:=0.265
-                                       BRACE_WIDTH:=0.9390
-                                       BRACE_HEIGHT:=2.308
-                                       BRACE_TO_FABRIC_XY_OFFSET:=0.004
-                                       BIN_WALL_THICKNESS:=0.002
-                                       BIN_FLAP_HEIGHT:=0.032
-                                       BRACE_TO_FABRIC_Z_OFFSET:=0.000
-                                       BIN_DEPTH:=0.152
-                                       TOP_BIN_DEPTH:=0.000
-                                       BIN_WIDTH:=0.234
-                                       BOTTOM_BIN_WIDTH:=0.000
-                                       BIN_BOTTOM_THICKNESS:=0.007
-                                       BIN_HEIGHTS:=[]
-                                       PODFACE_ID:=1A
-                                       ">
-    <!-- Pod's frame sizes (meters), universal for all pods in the Robotics Lab -->
-    <!-- BASE_WIDTH: 0.9398 in .stl file, but in reality - 0.9400 -->
-    <!-- BASE_HEIGHT: 0.295 in .stl file, but in reality - 0.265 -->
-    <!-- BRACE_WIDTH: 0.9188 in .stl file, but in reality - 0.9390 -->
-    <!-- BRACE_HEIGHT: 2.311 in .stl file, but in reality 2.308 -->
-    <!-- BRACE_TO_FABRIC_XY_OFFSET: 0.010 in .stl file, but in reality 0.004 -->
-    <!-- BIN_FLAP_HEIGHT: in recipe 0.026 or 0.022, but in reality 0.032 -->
-    <!-- ################################################################# -->
-    <!-- Pod's unique sizes (meters). By default, current 13x4 pod's sizes -->
+                                  BASE_WIDTH:=0.9400
+                                  BASE_HEIGHT:=0.265
+                                  BRACE_WIDTH:=0.9390
+                                  BRACE_HEIGHT:=2.308
+                                  BIN_WALL_THICKNESS:=0.002
+                                  BIN_FLAP_HEIGHT:=0.032
+                                  BRACE_TO_FABRIC_XY_OFFSET:=0.004
+                                  BRACE_TO_FABRIC_Z_OFFSET:=0.000
+                                  BIN_DEPTH:=0.152
+                                  TOP_BIN_DEPTH:=0.000
+                                  BIN_WIDTH:=0.234
+                                  BOTTOM_BIN_WIDTH:=0.000
+                                  BIN_BOTTOM_THICKNESS:=0.005
+                                  BIN_HEIGHTS:=[]
+                                  PODFACE_ID:=1A
+                                  INCLUDE_FLAPS:=true
+                                  ">
+    <!-- ############################################################################## -->
+    <!-- ### Pod's frame sizes (meters), universal for all pods in the Robotics Lab ### -->
+    <!-- ############################################################################## -->
+    <!-- BASE_WIDTH: 0.9398 in .stl file, but in reality - 0.940
+         BASE_HEIGHT: 0.295 in .stl file, but in reality - 0.265
+         BRACE_WIDTH: 0.9188 in .stl file, but in reality - 0.9390
+         BRACE_HEIGHT: 2.311 in .stl file, but in reality 2.308
+         BRACE_TO_FABRIC_XY_OFFSET: 0.010 in .stl file, but in reality 0.004
+         BIN_FLAP_HEIGHT: in recipe 0.026 or 0.022, but in reality 0.032
+         -->
+    <!-- ######################################################################### -->
+    <!-- ### Pod's unique sizes (meters). By default, current 13x4 pod's sizes ### -->
+    <!-- ######################################################################### -->
     <!-- BRACE_TO_FABRIC_Z_OFFSET
          BIN_DEPTH
@@ -34,5 +39,6 @@
          BIN_BOTTOM_THICKNESS
          BIN_HEIGHTS
-         PODFACE_ID -->
+         PODFACE_ID
+         -->
     <xacro:property name="alphabet" value="abcdefghijklmnopqrstuvwxyz"/>
     <xacro:property name="POD_ID"  value="${PODFACE_ID[0]}"/>
@@ -62,5 +68,5 @@
       <color rgba=".6 .6 .6 1"/>
     </material>
-    <link name="${prefix}base">
+    <link name="${prefix}base_link">
       <inertial>
         <mass value="30.0"/>
@@ -84,5 +90,5 @@
     <joint name="${prefix}base_${prefix}brace_joint" type="fixed">
       <origin xyz="0 0 ${BASE_HEIGHT}"/>
-      <parent link="${prefix}base"/>
+      <parent link="${prefix}base_link"/>
       <child link="${prefix}brace"/>
     </joint>
@@ -100,5 +106,5 @@
         </inertial>
         <visual>
-          <origin xyz="${x_len / 2} ${y_len / 2} 0"/> <!-- <origin xyz="${x_len / 2} ${y_len / 2} -${z_len / 2}"/> -->
+          <origin xyz="${x_len / 2} ${y_len / 2} ${z_len / 2}"/> <!-- <origin xyz="${x_len / 2} ${y_len / 2} -${z_len / 2}"/> -->
           <geometry>
             <box size="${x_len} ${y_len} ${z_len}"/>
@@ -107,5 +113,5 @@
         </visual>
         <collision>
-          <origin xyz="${x_len / 2} ${y_len / 2} 0"/> <!-- <origin xyz="${x_len / 2} ${y_len / 2} -${z_len / 2}"/> -->
+          <origin xyz="${x_len / 2} ${y_len / 2} ${z_len / 2}"/> <!-- <origin xyz="${x_len / 2} ${y_len / 2} -${z_len / 2}"/> -->
           <geometry>
             <box size="${x_len} ${y_len} ${z_len}"/>
@@ -114,5 +120,5 @@
       </link>
     </xacro:macro>
-    <xacro:macro name="bin" params="prefix colrow_id width depth height rightmost:=false top_shelf:=false">
+    <xacro:macro name="bin" params="prefix:=^ colrow_id width depth height rightmost:=false">
       <xacro:property name="bin_name" value="${prefix}bin_${colrow_id}"/>
       <link name="${bin_name}"/>
@@ -123,4 +129,10 @@
         <child link="${bin_name}_bottom"/>
       </joint>
+      <xacro:shifted_box name="${bin_name}_top" x_len="${width}" y_len="${depth}" z_len="${BIN_WALL_THICKNESS}"/>
+      <joint name="${bin_name}_${bin_name}_top" type="fixed">
+        <origin xyz="0 0 ${height - BIN_WALL_THICKNESS}" rpy="0 0 0"/>
+        <parent link="${bin_name}"/>
+        <child link="${bin_name}_top"/>
+      </joint>
       <xacro:shifted_box name="${bin_name}_left" x_len="${BIN_WALL_THICKNESS}" y_len="${depth}" z_len="${height}"/>
       <joint name="${bin_name}_${bin_name}_left" type="fixed">
@@ -128,16 +140,4 @@
         <parent link="${bin_name}"/>
         <child link="${bin_name}_left"/>
-      </joint>
-      <xacro:shifted_box name="${bin_name}_back" x_len="${width}" y_len="${BIN_WALL_THICKNESS}" z_len="${height}"/>
-      <joint name="${bin_name}_${bin_name}_back" type="fixed">
-        <origin xyz="0 ${depth} 0" rpy="0 0 0"/>
-        <parent link="${bin_name}"/>
-        <child link="${bin_name}_back"/>
-      </joint>
-      <xacro:shifted_box name="${bin_name}_flap" x_len="${width}" y_len="${BIN_WALL_THICKNESS}" z_len="${BIN_FLAP_HEIGHT}"/>
-      <joint name="${bin_name}_${bin_name}_flap" type="fixed">
-        <origin xyz="0 0 0" rpy="0 0 0"/>
-        <parent link="${bin_name}"/>
-        <child link="${bin_name}_flap"/>
       </joint>
       <xacro:if value="${rightmost}">
@@ -149,15 +149,21 @@
         </joint>
       </xacro:if>
-      <xacro:if value="${top_shelf}">
-        <xacro:shifted_box name="${bin_name}_top" x_len="${width}" y_len="${depth}" z_len="${BIN_WALL_THICKNESS}"/>
-        <joint name="${bin_name}_${bin_name}_top" type="fixed">
-          <origin xyz="0 0 ${height}" rpy="0 0 0"/>
+      <xacro:shifted_box name="${bin_name}_back" x_len="${width}" y_len="${BIN_WALL_THICKNESS}" z_len="${height}"/>
+      <joint name="${bin_name}_${bin_name}_back" type="fixed">
+        <origin xyz="0 ${depth - BIN_WALL_THICKNESS} 0" rpy="0 0 0"/>
+        <parent link="${bin_name}"/>
+        <child link="${bin_name}_back"/>
+      </joint>
+      <xacro:if value="${INCLUDE_FLAPS}">
+        <xacro:shifted_box name="${bin_name}_flap" x_len="${width}" y_len="${BIN_WALL_THICKNESS}" z_len="${BIN_FLAP_HEIGHT}"/>
+        <joint name="${bin_name}_${bin_name}_flap" type="fixed">
+          <origin xyz="0 0 0" rpy="0 0 0"/>
           <parent link="${bin_name}"/>
-          <child link="${bin_name}_top"/>
-        </joint>
-      </xacro:if>
-    </xacro:macro>
-    <xacro:macro name="bin_row" params="prefix row_id bin_row_base sections bin_width bin_depth bin_height i:=0 top_shelf:=false">
-      <xacro:property name="bin_name" value="${prefix}bin_${i+1}${id}"/>
+          <child link="${bin_name}_flap"/>
+        </joint>
+      </xacro:if>
+    </xacro:macro>
+    <xacro:macro name="bin_row" params="prefix:=^ row_id bin_row_base sections bin_width bin_depth bin_height i:=0">
+      <xacro:property name="bin_name" value="${prefix}bin_${i+1}${row_id}"/>
       <xacro:if value="${sections == 1}">
         <xacro:property name="rightmost" value="true"/>
@@ -166,5 +172,5 @@
         <xacro:property name="rightmost" value="false"/>
       </xacro:unless>
-      <xacro:bin prefix="${prefix}" colrow_id="${i+1}${row_id}" rightmost="${rightmost}" top_shelf="${top_shelf}"
+      <xacro:bin colrow_id="${i+1}${row_id}" rightmost="${rightmost}"
                  width="${bin_width}" depth="${bin_depth}" height="${bin_height}"/>
       <joint name="${bin_row_base}_${bin_name}_joint" type="fixed">
@@ -174,13 +180,13 @@
       </joint>
       <xacro:if value="${sections > 1}"><!-- recurse for the remaining bins -->
-        <xacro:bin_row prefix="${prefix}" row_id="${row_id}" bin_row_base="${bin_row_base}" sections="${sections-1}" i="${i+1}" top_shelf="${top_shelf}"
+        <xacro:bin_row row_id="${row_id}" bin_row_base="${bin_row_base}" sections="${sections-1}" i="${i+1}"
                        bin_width="${bin_width}" bin_depth="${bin_depth}" bin_height="${bin_height}"/><!-- no prefix passing -->
       </xacro:if>
     </xacro:macro>
-    <xacro:macro name="shelf" params="prefix row_id bin_width:=${BIN_WIDTH} shelf_depth:=${BIN_DEPTH} shelf_height sections:=4 top_shelf:=false">
+    <xacro:macro name="shelf" params="prefix:=^ row_id bin_width:=${BIN_WIDTH} shelf_depth:=${BIN_DEPTH} shelf_height sections:=4">
       <xacro:property name="shelf_name" value="${prefix}shelf_${row_id}"/>
       <xacro:if value="${X_OFFSET != 0}"><!-- left margin, relates to B & D faces of pods -->
         <xacro:shifted_box name="${shelf_name}_left_margin" x_len="${X_OFFSET}" y_len="${BIN_WALL_THICKNESS}" z_len="${shelf_height}"/>
-        <joint name="${shelf_name}_${shelf_name}_left_margin" type="fixed">
+        <joint name="${shelf_name}_${shelf_name}_left_margin_joint" type="fixed">
           <origin xyz="0 0 0" rpy="0 0 0"/>
           <parent link="${shelf_name}"/>
@@ -189,9 +195,9 @@
       </xacro:if>
       <link name="${shelf_name}"/>
-      <xacro:bin_row prefix="${prefix}" row_id="${row_id}" bin_row_base="${shelf_name}" sections="${sections}" top_shelf="${top_shelf}"
+      <xacro:bin_row row_id="${row_id}" bin_row_base="${shelf_name}" sections="${sections}"
                      bin_width="${bin_width}" bin_depth="${shelf_depth}" bin_height="${shelf_height}"/><!-- no prefix passing -->
       <xacro:if value="${X_OFFSET != 0}"><!-- right margin, relates to B & D faces of pods -->
         <xacro:shifted_box name="${shelf_name}_right_margin" x_len="${X_OFFSET}" y_len="${BIN_WALL_THICKNESS}" z_len="${shelf_height}"/>
-        <joint name="${shelf_name}_${shelf_name}_right_margin" type="fixed">
+        <joint name="${shelf_name}_${shelf_name}_right_margin_joint" type="fixed">
           <origin xyz="${X_OFFSET + bin_width * sections} 0 0" rpy="0 0 0"/>
           <parent link="${shelf_name}"/>
@@ -200,5 +206,5 @@
       </xacro:if>
     </xacro:macro>
-    <xacro:macro name="shelf_stack" params="prefix shelf_stack_base shelf_heights z_offset:=0 i:=0">
+    <xacro:macro name="shelf_stack" params="prefix:=^ shelf_stack_base shelf_heights z_offset:=0 i:=0">
       <xacro:property name="shelf_height" value="${shelf_heights[0]}"/>
       <xacro:property name="shelf_name" value="${prefix}shelf_${alphabet[i]}"/>
@@ -216,5 +222,7 @@
         <xacro:unless value="${POD_ID == 1 and i == 0}">
           <xacro:property name="bin_width" value="${BIN_WIDTH}"/>
-          <xacro:property name="NUM_COLUMNS" value="2"/>
+          <xacro:if value="${POD_ID == 1}">
+            <xacro:property name="NUM_COLUMNS" value="2"/>
+          </xacro:if>
         </xacro:unless>
       </xacro:if>
@@ -223,12 +231,6 @@
         <xacro:property name="bin_width" value="${BIN_WIDTH}"/>
       </xacro:unless>
-      <xacro:if value="${len(shelf_heights) == 1}">
-        <xacro:property name="top_shelf" value="true"/>
-      </xacro:if>
-      <xacro:unless value="${len(shelf_heights) == 1}">
-        <xacro:property name="top_shelf" value="false"/>
-      </xacro:unless>
       <xacro:shelf prefix="${prefix}" row_id="${alphabet[i]}" sections="${NUM_COLUMNS}"
-                   bin_width="${bin_width}" shelf_depth="${shelf_depth}" shelf_height="${shelf_height}" top_shelf="${top_shelf}"/>
+                   bin_width="${bin_width}" shelf_depth="${shelf_depth}" shelf_height="${shelf_height}"/>
       <joint name="${shelf_stack_base}_${shelf_name}_joint" type="fixed">
         <origin xyz="0 0 ${z_offset}"/>
@@ -237,5 +239,5 @@
       </joint>
       <xacro:if value="${len(shelf_heights) > 1}"><!-- recurse for the remaining shelves-->
-        <xacro:shelf_stack prefix="${prefix}" shelf_stack_base="${shelf_stack_base}" shelf_heights="${shelf_heights[1:]}" z_offset="${z_offset + shelf_height[0]}" i="${i+1}"/><!-- no prefix passing -->
+        <xacro:shelf_stack shelf_stack_base="${shelf_stack_base}" shelf_heights="${shelf_heights[1:]}" z_offset="${z_offset + shelf_height}" i="${i+1}"/><!-- no prefix passing -->
       </xacro:if>
     </xacro:macro>

File: tahoma_description/urdf/tahoma.xacro (robot description, xacro)
@@ -40,10 +40,10 @@
       <xacro:property name="cover_orgZ_offset" value="0.020" />
       <link name="base_link" />
-      <joint name="base_link-stand_joint" type="fixed">
+      <joint name="base_link__stand__joint" type="fixed">
         <origin rpy="0 0 0" xyz="0 0 0.15"/>
         <parent link="base_link"/>
         <child link="stand"/>
       </joint>
-      <joint name="robot_plate-arm_base_link_joint" type="fixed">
+      <joint name="robot_plate__arm_base_link__joint" type="fixed">
         <parent link="robot_plate" />
         <child link="arm_base_link" />
@@ -84,16 +84,16 @@
         </collision>
       </link>
-      <joint name="coupling-connector_cover_joint" type="fixed">
+      <joint name="coupling__connector_cover__joint" type="fixed">
         <origin xyz="${coupling_flat_edge_X_offset} 0 ${coupling_flat_edge_Z_offset}" rpy="0 0 0" />
         <parent link="coupling" />
         <child link="connector_cover"/>
       </joint>
-      <joint name="coupling-gripper_base_link_joint" type="fixed">
-        <origin xyz="0 0 ${coupling_H - coupling_h}" rpy="0 0 0" />
+      <joint name="coupling__gripper_base_link__joint" type="fixed">
+        <origin xyz="0 0 ${coupling_H - coupling_h}" rpy="0 0 ${0.5 * pi}" />
         <parent link="coupling" />
         <child link="gripper_base_link" />
       </joint>
       <!-- Coupling edge height = 0.003. Rotate -90(270)deg around z to align with the robot's wrist electric connection -->
-      <joint name="arm_tool0-coupling_joint" type="fixed">
+      <joint name="arm_tool0__coupling___joint" type="fixed">
         <origin xyz="0 0 ${-coupling_h}" rpy="0 0 ${1.5 * pi}" />
         <parent link="arm_tool0" />

Commit message: Change pod 0 recipe to better match reality
Fix args for pod ID and face in bringup and view_models

File: tahoma_description/robots/pod.xacro (robot description, xacro)
@@ -3,13 +3,13 @@
   <xacro:arg name="pod_id" default="1A"/>
   <xacro:arg name="include_flaps" default="true"/>
-  <xacro:arg name="call_macro" default="false"/>
   <xacro:macro name="pod_recipe" params="pod_id:=1A include_flaps:=true">
     <xacro:include filename="$(find tahoma_description)/urdf/pod.xacro"/>
       <xacro:property name="POD_ID"  value="${pod_id[0]}"/>
       <xacro:property name="FACE_ID" value="${pod_id[1]}"/>
-      <!-- Current pod -->
+      <!-- Recipes are bottom shelf to top-->
+      <!-- Small bin bod. -->
       <xacro:if value="${POD_ID == 1}">
         <xacro:if value="${FACE_ID == 'A'}"><!-- (13x4) Ref. -> pod1_recipe_790-00265-021.txt "bindDimensions" : A1-A13. corresponds to reality. Current face -->
-          <xacro:pod_urdf
+          <xacro:pod
             prefix="pod_"
             BRACE_TO_FABRIC_Z_OFFSET="0.085"
@@ -18,9 +18,9 @@
             BIN_WIDTH="0.234"
             BIN_BOTTOM_THICKNESS="0.005"
-            BIN_HEIGHTS="${[0.223, 0.146, 0.197, 0.146, 0.121, 0.223, 0.121, 0.146, 0.121, 0.223, 0.121, 0.146, 0.261]}"
+            BIN_HEIGHTS="${[0.234, 0.166, 0.173, 0.146, 0.187, 0.160, 0.116, 0.223, 0.146, 0.223, 0.146, 0.261]}"
             INCLUDE_FLAPS="${include_flaps}"/>
         </xacro:if>
         <xacro:if value="${FACE_ID == 'B'}"><!-- (8x2) Ref. -> pod1_recipe_790-00265-021.txt "bindDimensions" : B1-B8. corresponds to reality -->
-          <xacro:pod_urdf
+          <xacro:pod
             prefix="pod_"
             BRACE_TO_FABRIC_Z_OFFSET="0.085"
@@ -34,6 +34,6 @@
             INCLUDE_FLAPS="${include_flaps}"/>
         </xacro:if>
-        <xacro:if value="${FACE_ID == 'C'}"><!-- (12x4) Ref. -> pod1_recipe_790-00265-021.txt "bindDimensions" : C1-C12. haven't been measured in reality -->
-          <xacro:pod_urdf
+        <xacro:if value="${FACE_ID == 'C'}"><!-- (12x4) Ref. -> .02  .006  .005 pod1_recipe_790-00265-021.txt "bindDimensions" : C1-C12. haven't been measured in reality -->
+          <xacro:pod
             prefix="pod_"
             BRACE_TO_FABRIC_Z_OFFSET="0.085"
@@ -42,9 +42,9 @@
             BIN_WIDTH="0.234"
             BIN_BOTTOM_THICKNESS="0.005"
-            BIN_HEIGHTS="${[0.223, 0.146, 0.223, 0.146, 0.197, 0.146, 0.121, 0.223, 0.146, 0.223, 0.146, 0.261]}"
+            BIN_HEIGHTS="${[0.234, 0.166, 0.173, 0.146, 0.187, 0.160, 0.116, 0.223, 0.146, 0.223, 0.146, 0.261]}"
             INCLUDE_FLAPS="${include_flaps}"/>
         </xacro:if>
         <xacro:if value="${FACE_ID == 'D'}"><!-- (7x2) Ref. -> pod1_recipe_790-00265-021.txt "bindDimensions" : D1-D7. corresponds to reality -->
-          <xacro:pod_urdf
+          <xacro:pod
             prefix="pod_"
             BRACE_TO_FABRIC_Z_OFFSET="0.085"
@@ -62,5 +62,5 @@
       <xacro:if value="${POD_ID == 2}">
         <xacro:if value="${FACE_ID == 'A'}"><!-- (8x3) Ref. -> pod2_recipe_790-00265-022.txt "bindDimensions" : A1-A8 with minor changes corresponding to reality. Henry using face -->
-          <xacro:pod_urdf
+          <xacro:pod
             prefix="pod_"
             BRACE_TO_FABRIC_Z_OFFSET="0.035"
@@ -73,5 +73,5 @@
         </xacro:if>
         <xacro:if value="${FACE_ID == 'B'}"><!-- (8x1) Ref. -> pod2_recipe_790-00265-022.txt "bindDimensions" : B1-B8. haven't been measured in reality -->
-          <xacro:pod_urdf
+          <xacro:pod
             prefix="pod_"
             BRACE_TO_FABRIC_Z_OFFSET="0.035"
@@ -85,5 +85,5 @@
         </xacro:if>
         <xacro:if value="${FACE_ID == 'C'}"><!-- (8x3) Ref. -> pod2_recipe_790-00265-022.txt "bindDimensions" : C1-C8. haven't been measured in reality -->
-          <xacro:pod_urdf
+          <xacro:pod
             prefix="pod_"
             BRACE_TO_FABRIC_Z_OFFSET="0.035"
@@ -96,5 +96,5 @@
         </xacro:if>
         <xacro:if value="${FACE_ID == 'D'}"><!-- (7x1) Ref. -> pod2_recipe_790-00265-022.txt "bindDimensions" : D1-D7. haven't been measured in reality -->
-          <xacro:pod_urdf
+          <xacro:pod
             prefix="pod_"
             BRACE_TO_FABRIC_Z_OFFSET="0.035"
@@ -109,6 +109,4 @@
       </xacro:if>
   </xacro:macro>
-  <xacro:if value="$(arg call_macro)"><!-- (7x1) Ref. -> pod2_recipe_790-00265-022.txt "bindDimensions" : D1-D7. haven't been measured in reality -->
-    <xacro:pod_recipe pod_id="$(arg pod_id)" include_flaps="$(arg include_flaps)"/>
-  </xacro:if>
+  <xacro:pod_recipe pod_id="$(arg pod_id)" include_flaps="$(arg include_flaps)"/>
 </robot>

File: tahoma_description/urdf/pod.xacro (robot description, xacro)
@@ -1,5 +1,5 @@
 <?xml version="1.0"?>
 <robot xmlns:xacro="http://www.ros.org/wiki/xacro" name="pod">
-  <xacro:macro name="pod_urdf" params="prefix:=pod_
+  <xacro:macro name="pod" params="prefix:=pod_
                                   BASE_WIDTH:=0.9400
                                   BASE_HEIGHT:=0.265
