Commit message: index on henri-continual: 0b51c55 Calibrated camera pose and gripper camera orientation with mount

File: tahoma_description/robots/pod.xacro (robot description, xacro)
@@ -3,13 +3,13 @@
   <xacro:arg name="pod_id" default="1A"/>
   <xacro:arg name="include_flaps" default="true"/>
+  <xacro:arg name="call_macro" default="false"/>
   <xacro:macro name="pod_recipe" params="pod_id:=1A include_flaps:=true">
     <xacro:include filename="$(find tahoma_description)/urdf/pod.xacro"/>
       <xacro:property name="POD_ID"  value="${pod_id[0]}"/>
       <xacro:property name="FACE_ID" value="${pod_id[1]}"/>
-      <!-- Recipes are bottom shelf to top-->
-      <!-- Small bin bod. -->
+      <!-- Current pod -->
       <xacro:if value="${POD_ID == 1}">
         <xacro:if value="${FACE_ID == 'A'}"><!-- (13x4) Ref. -> pod1_recipe_790-00265-021.txt "bindDimensions" : A1-A13. corresponds to reality. Current face -->
-          <xacro:pod
+          <xacro:pod_urdf
             prefix="pod_"
             BRACE_TO_FABRIC_Z_OFFSET="0.085"
@@ -18,9 +18,9 @@
             BIN_WIDTH="0.234"
             BIN_BOTTOM_THICKNESS="0.005"
-            BIN_HEIGHTS="${[0.234, 0.166, 0.173, 0.146, 0.187, 0.160, 0.116, 0.223, 0.146, 0.223, 0.146, 0.261]}"
+            BIN_HEIGHTS="${[0.223, 0.146, 0.197, 0.146, 0.121, 0.223, 0.121, 0.146, 0.121, 0.223, 0.121, 0.146, 0.261]}"
             INCLUDE_FLAPS="${include_flaps}"/>
         </xacro:if>
         <xacro:if value="${FACE_ID == 'B'}"><!-- (8x2) Ref. -> pod1_recipe_790-00265-021.txt "bindDimensions" : B1-B8. corresponds to reality -->
-          <xacro:pod
+          <xacro:pod_urdf
             prefix="pod_"
             BRACE_TO_FABRIC_Z_OFFSET="0.085"
@@ -34,6 +34,6 @@
             INCLUDE_FLAPS="${include_flaps}"/>
         </xacro:if>
-        <xacro:if value="${FACE_ID == 'C'}"><!-- (12x4) Ref. -> .02  .006  .005 pod1_recipe_790-00265-021.txt "bindDimensions" : C1-C12. haven't been measured in reality -->
-          <xacro:pod
+        <xacro:if value="${FACE_ID == 'C'}"><!-- (12x4) Ref. -> pod1_recipe_790-00265-021.txt "bindDimensions" : C1-C12. haven't been measured in reality -->
+          <xacro:pod_urdf
             prefix="pod_"
             BRACE_TO_FABRIC_Z_OFFSET="0.085"
@@ -42,9 +42,9 @@
             BIN_WIDTH="0.234"
             BIN_BOTTOM_THICKNESS="0.005"
-            BIN_HEIGHTS="${[0.234, 0.166, 0.173, 0.146, 0.187, 0.160, 0.116, 0.223, 0.146, 0.223, 0.146, 0.261]}"
+            BIN_HEIGHTS="${[0.223, 0.146, 0.223, 0.146, 0.197, 0.146, 0.121, 0.223, 0.146, 0.223, 0.146, 0.261]}"
             INCLUDE_FLAPS="${include_flaps}"/>
         </xacro:if>
         <xacro:if value="${FACE_ID == 'D'}"><!-- (7x2) Ref. -> pod1_recipe_790-00265-021.txt "bindDimensions" : D1-D7. corresponds to reality -->
-          <xacro:pod
+          <xacro:pod_urdf
             prefix="pod_"
             BRACE_TO_FABRIC_Z_OFFSET="0.085"
@@ -62,5 +62,5 @@
       <xacro:if value="${POD_ID == 2}">
         <xacro:if value="${FACE_ID == 'A'}"><!-- (8x3) Ref. -> pod2_recipe_790-00265-022.txt "bindDimensions" : A1-A8 with minor changes corresponding to reality. Henry using face -->
-          <xacro:pod
+          <xacro:pod_urdf
             prefix="pod_"
             BRACE_TO_FABRIC_Z_OFFSET="0.035"
@@ -73,5 +73,5 @@
         </xacro:if>
         <xacro:if value="${FACE_ID == 'B'}"><!-- (8x1) Ref. -> pod2_recipe_790-00265-022.txt "bindDimensions" : B1-B8. haven't been measured in reality -->
-          <xacro:pod
+          <xacro:pod_urdf
             prefix="pod_"
             BRACE_TO_FABRIC_Z_OFFSET="0.035"
@@ -85,5 +85,5 @@
         </xacro:if>
         <xacro:if value="${FACE_ID == 'C'}"><!-- (8x3) Ref. -> pod2_recipe_790-00265-022.txt "bindDimensions" : C1-C8. haven't been measured in reality -->
-          <xacro:pod
+          <xacro:pod_urdf
             prefix="pod_"
             BRACE_TO_FABRIC_Z_OFFSET="0.035"
@@ -96,5 +96,5 @@
         </xacro:if>
         <xacro:if value="${FACE_ID == 'D'}"><!-- (7x1) Ref. -> pod2_recipe_790-00265-022.txt "bindDimensions" : D1-D7. haven't been measured in reality -->
-          <xacro:pod
+          <xacro:pod_urdf
             prefix="pod_"
             BRACE_TO_FABRIC_Z_OFFSET="0.035"
@@ -109,4 +109,6 @@
       </xacro:if>
   </xacro:macro>
-  <xacro:pod_recipe pod_id="$(arg pod_id)" include_flaps="$(arg include_flaps)"/>
+  <xacro:if value="$(arg call_macro)"><!-- (7x1) Ref. -> pod2_recipe_790-00265-022.txt "bindDimensions" : D1-D7. haven't been measured in reality -->
+    <xacro:pod_recipe pod_id="$(arg pod_id)" include_flaps="$(arg include_flaps)"/>
+  </xacro:if>
 </robot>

File: tahoma_description/urdf/pod.xacro (robot description, xacro)
@@ -1,5 +1,5 @@
 <?xml version="1.0"?>
 <robot xmlns:xacro="http://www.ros.org/wiki/xacro" name="pod">
-  <xacro:macro name="pod" params="prefix:=pod_
+  <xacro:macro name="pod_urdf" params="prefix:=pod_
                                   BASE_WIDTH:=0.9400
                                   BASE_HEIGHT:=0.265

File: tahoma_description/urdf/tahoma.xacro (robot description, xacro)
@@ -5,4 +5,5 @@
   <!-- <xacro:include filename="$(find robotiq_2f_85_gripper_visualization)/urdf/robotiq_arg2f_85_macro.xacro"/> -->
   <xacro:include filename="$(find robotiq_epick_visualization)/urdf/robotiq_epick_model_macro.xacro" />
+  <xacro:include filename="$(find tahoma_description)/urdf/_l515.urdf.xacro" />
   <!-- <xacro:include filename="$(find realsense2_description)/urdf/_l515.urdf.xacro"/> -->
   <xacro:macro name="tahoma" params="
@@ -160,5 +161,5 @@
         <child link="camera_base"/>
         <!-- Link is centered on the optical frames. Slight offset in Y direction to compensate -->
-        <origin xyz="-0.21 -0.01  1.375" rpy="0.0 -0.08 0.0" />
+        <origin xyz="-0.20750794 -0.01815336  1.40753882" rpy="3.14 3.14 -3.14" />
         <!-- <origin xyz="-0.2426 -0.0277 1.4078" rpy="3.14 3.14 -3.14" /> -->
       </joint>
@@ -182,17 +183,32 @@
       </visual>
     </link>
-    <xacro:sensor_l515 parent="coupling" use_nominal_extrinsics="$(arg use_nominal_extrinsics)" add_plug="$(arg add_plug)" use_mesh="$(arg use_mesh)">
+    <xacro:if value="${realsense}">
+      <xacro:sensor_l515 name="camera_lower_right" parent="camera_lower_right_mount" use_nominal_extrinsics="${use_nominal_camera_extrinsics}">
+        <origin xyz="0 0 0" rpy="0 0 0"/>
+      </xacro:sensor_l515>
+    <link name="realsense_back_gripper_mount">
+      <collision>
+        <origin xyz="0.010227 -0.005 0.035" rpy="0 0 0"/>
+        <geometry>
+          <box size="0.04 0.02 0.08"/>
+        </geometry>
+      </collision>
+      <visual>
+        <origin xyz="0 0 0" rpy="0 0 0"/>
+        <geometry>
+          <mesh filename="package://tahoma_description/meshes/realsense/couple_l515_mount.obj"/>
+        </geometry>
+      </visual>
+    </link>
+    </xacro:if>
+    <!-- L515 Realsense Camera -->
+    <xacro:sensor_l515 parent="realsense_back_gripper_mount" use_nominal_extrinsics="${use_nominal_camera_extrinsics}" add_plug="false" use_mesh="true">
       <origin xyz="0.0 0.046 0.06" rpy="${pi} -${0.5 * pi} ${0.5 * pi}"/>
     </xacro:sensor_l515>
     <joint name="realsense_back_gripper_mount_joint" type="fixed">
-        <parent link="camera_link"/>
+        <parent link="coupling"/>
         <child link="realsense_back_gripper_mount"/>
         <origin xyz="-0.018 0.010227 -0.036" rpy="0 0 ${-0.5 * pi}" />
     </joint>
-    <xacro:if value="${realsense}">
-      <xacro:sensor_l515 name="camera_lower_right" parent="camera_lower_right_mount" use_nominal_extrinsics="${use_nominal_camera_extrinsics}">
-        <origin xyz="0 0 0" rpy="0 0 0"/>
-      </xacro:sensor_l515>
-    </xacro:if>
   <link name="gripper_equilibrium_grasp"/>
   <joint name="gripper_base_link_gripper_equilibrium_grasp" type="fixed">
