Commit message: Add camera beam to robot model
Eventual home for stand cameras. Just need for collision geometry right now

File: tahoma_description/urdf/stand.xacro (robot description, xacro)
@@ -99,4 +99,23 @@
       </collision>
     </link>
+    <link name="camera_beam_lower">
+      <inertial>
+        <mass value="5"/>
+        <inertia ixx="0.0002835" ixy="0.0" ixz="0.0" iyy="0.0002835" iyz="0.0" izz="0.000324"/>
+      </inertial>
+      <visual>
+        <origin rpy="0 0 0" xyz="0 0 0"/>
+        <geometry>
+          <mesh filename="package://tahoma_description/meshes/stand/camera_beam.stl"/>
+        </geometry>
+        <material name="blue_aluminum"/>
+      </visual>
+      <collision>
+        <origin rpy="0 0 .022" xyz="0 0 0"/>
+        <geometry>
+          <box size="0.045 1.25 0.045"/>
+        </geometry>
+      </collision>
+    </link>
     <link name="cantilever">
       <inertial>
@@ -191,4 +210,9 @@
       <origin rpy="0 0 0" xyz="-.24 0 -.59"/>
     </joint>
+    <joint name="stand_upright_camera_beam_lower_joint" type="fixed">
+      <parent link="stand_upright"/>
+      <child link="camera_beam_lower"/>
+      <origin rpy="0 0 0" xyz="-.128 0 0"/>
+    </joint>
     <joint name="stand_upright_robot_control_box_mount_joint" type="fixed">
       <parent link="stand_upright"/>

Commit message: Add basic workspace analysis script
Queries IK for poses of interest, publishes markers to visualize
Add RViz config which displays the results with a couple views
Remove hardcoded pi property from stand xacro
Fix a log statement in Tahoma wrapper

File: tahoma_description/urdf/stand.xacro (robot description, xacro)
@@ -4,6 +4,4 @@
   <xacro:include filename="$(find tahoma_description)/urdf/light_panel.xacro"/>
   <xacro:macro name="stand">
-    <xacro:property name="M_PI" value="3.1415926535897931"/>
-    <xacro:property name="M_PI_2" value="1.57079632679489661923"/>
     <material name="blue_aluminum">
       <!-- more accurate but less pretty :) -->
@@ -223,5 +221,5 @@
       <parent link="control_box_mount"/>
       <child link="control_box"/>
-      <origin rpy="0.05 0 ${M_PI}" xyz="-.003 .1375 -0.13"/>
+      <origin rpy="0.05 0 ${pi}" xyz="-.003 .1375 -0.13"/>
     </joint>
     <joint name="stand_cantilever_joint" type="fixed">
@@ -258,10 +256,10 @@
       <parent link="stand_upright"/>
       <child link="left_light_panel"/>
-      <origin rpy="0 ${M_PI_2} 0" xyz="-.2625 .35 .25"/>
+      <origin rpy="0 ${pi / 2} 0" xyz="-.2625 .35 .25"/>
     </joint>
     <joint name="stand_left_right_panel_joint" type="fixed">
       <parent link="stand_upright"/>
       <child link="right_light_panel"/>
-      <origin rpy="0 ${M_PI_2} 0" xyz="-.2625 -.35 .25"/>
+      <origin rpy="0 ${pi / 2} 0" xyz="-.2625 -.35 .25"/>
     </joint>
   </xacro:macro>

Commit message: Update camera mount and beam placement
Tuned to be good enough for testing in the center bins

File: tahoma_description/urdf/stand.xacro (robot description, xacro)
@@ -211,5 +211,5 @@
       <parent link="stand_upright"/>
       <child link="camera_beam_lower"/>
-      <origin rpy="0 0 0" xyz="-.228 0 .35"/>
+      <origin rpy="0 0 0" xyz="-.1225 0 .465"/>
     </joint>
     <joint name="stand_upright_robot_control_box_mount_joint" type="fixed">

File: tahoma_description/urdf/tahoma.xacro (robot description, xacro)
@@ -76,6 +76,6 @@
       <child link="camera_lower_left_mount"/>
       <!-- Link is centered on the optical frames. Slight offset in Y direction to compensate -->
-      <origin xyz="-0.00 ${-0.0215 + camera_baseline / 2} 0.09"
-              rpy="${-pi / 2} 0 ${-math.atan2((camera_baseline /2),camera_focal_depth)}"/>
+      <origin xyz="-0.00 0.02 0.11"
+              rpy="${pi / 2} 0 0"/>
     </joint>
     <joint name="camera_beam_lower_camera_lower_right_mount_joint" type="fixed">

Commit message: 1. Minor changes in filtering and transformations of aurmr_grasping, 2. Minor changes to offset distances in pick, 3. Function changeed in motion.py and tahoma.py, 4. Changes to fake_gripper_state, stand.xacro and tahoma.xacro as camera mount changed

File: tahoma_description/urdf/stand.xacro (robot description, xacro)
@@ -211,5 +211,5 @@
       <parent link="stand_upright"/>
       <child link="camera_beam_lower"/>
-      <origin rpy="0 0 0" xyz="-.1225 0 .465"/>
+      <origin rpy="0 0 0" xyz="-.1225 0 .193"/>
     </joint>
     <joint name="stand_upright_robot_control_box_mount_joint" type="fixed">

File: tahoma_description/urdf/tahoma.xacro (robot description, xacro)
@@ -76,6 +76,6 @@
       <child link="camera_lower_left_mount"/>
       <!-- Link is centered on the optical frames. Slight offset in Y direction to compensate -->
-      <origin xyz="-0.00 0.02 0.11"
-              rpy="${pi / 2} 0 0"/>
+      <origin xyz="-0.00 0.02 0.06"
+              rpy="0 0 0"/>
     </joint>
     <joint name="camera_beam_lower_camera_lower_right_mount_joint" type="fixed">

Commit message: Fix incorrect camera beam collision
Had accidentally swapped XYZ and RPY entries
Change all pose specs to declare XYZ first

File: tahoma_description/urdf/stand.xacro (robot description, xacro)
@@ -16,5 +16,5 @@
       </inertial>
       <visual>
-        <origin rpy="0 0 0" xyz="0 0 0"/>
+        <origin xyz="0 0 0" rpy="0 0 0"/>
         <geometry>
           <mesh filename="package://tahoma_description/meshes/stand/stand_base.stl"/>
@@ -24,5 +24,5 @@
       <collision>
         <!-- across -->
-        <origin rpy="0 0 0" xyz=".4050 0 .0281"/>
+        <origin xyz=".4050 0 .0281" rpy="0 0 0"/>
         <geometry>
           <box size=".09 1.53 .045"/>
@@ -31,5 +31,5 @@
       <collision>
         <!-- right -->
-        <origin rpy="0 0 0" xyz="0 -.72 -.0225"/>
+        <origin xyz="0 -.72 -.0225" rpy="0 0 0"/>
         <geometry>
           <box size=".9 .09 .0562"/>
@@ -38,5 +38,5 @@
       <collision>
         <!-- left -->
-        <origin rpy="0 0 0" xyz="0 .72 -.0225"/>
+        <origin xyz="0 .72 -.0225" rpy="0 0 0"/>
         <geometry>
           <box size=".9 .09 .0562"/>
@@ -50,5 +50,5 @@
       </inertial>
       <visual>
-        <origin rpy="0 0 0" xyz="0 0 0"/>
+        <origin xyz="0 0 0" rpy="0 0 0"/>
         <geometry>
           <mesh filename="package://tahoma_description/meshes/stand/stand_upright.stl"/>
@@ -58,5 +58,5 @@
       <collision>
         <!-- right upright -->
-        <origin rpy="0 0 0" xyz="-.1709 0.6975 0"/>
+        <origin xyz="-.1709 0.6975 0" rpy="0 0 0"/>
         <geometry>
           <box size=".2298 .0450 1.89"/>
@@ -65,5 +65,5 @@
       <collision>
         <!-- left upright -->
-        <origin rpy="0 0 0" xyz="-.1709 -0.6975 0"/>
+        <origin xyz="-.1709 -0.6975 0" rpy="0 0 0"/>
         <geometry>
           <box size=".2298 .0450 1.89"/>
@@ -72,5 +72,5 @@
       <collision>
         <!-- top beam -->
-        <origin rpy="0 0 0" xyz="-.1733 0 .9012"/>
+        <origin xyz="-.1733 0 .9012" rpy="0 0 0"/>
         <geometry>
           <box size=".2370 1.44 .0960"/>
@@ -84,5 +84,5 @@
       </inertial>
       <visual>
-        <origin rpy="0 0 0" xyz="0 0 0"/>
+        <origin xyz="0 0 0" rpy="0 0 0"/>
         <geometry>
           <mesh filename="package://tahoma_description/meshes/stand/stand_brace.stl"/>
@@ -91,5 +91,5 @@
       </visual>
       <collision>
-        <origin rpy="0 0 0" xyz="0 0 0"/>
+        <origin xyz="0 0 0" rpy="0 0 0"/>
         <geometry>
           <box size=".102 1.4390 .4934"/>
@@ -103,5 +103,5 @@
       </inertial>
       <visual>
-        <origin rpy="0 0 0" xyz="0 0 0"/>
+        <origin xyz="0 0 0" rpy="0 0 0"/>
         <geometry>
           <mesh filename="package://tahoma_description/meshes/stand/camera_beam.stl"/>
@@ -110,7 +110,7 @@
       </visual>
       <collision>
-        <origin rpy="0 0 .022" xyz="0 0 0"/>
-        <geometry>
-          <box size="0.045 1.25 0.045"/>
+        <origin xyz="0 0 0.022" rpy="0 0 0"/>
+        <geometry>
+          <box size="0.045 1.35 0.045"/>
         </geometry>
       </collision>
@@ -122,5 +122,5 @@
       </inertial>
       <visual>
-        <origin rpy="0 0 0" xyz="0 0 0"/>
+        <origin xyz="0 0 0" rpy="0 0 0"/>
         <geometry>
           <mesh filename="package://tahoma_description/meshes/stand/cantilever.stl"/>
@@ -141,5 +141,5 @@
       </inertial>
       <visual>
-        <origin rpy="0 0 0" xyz="0 0 0"/>
+        <origin xyz="0 0 0" rpy="0 0 0"/>
         <geometry>
           <mesh filename="package://tahoma_description/meshes/stand/control_box_mount.stl"/>
@@ -148,5 +148,5 @@
       </visual>
       <collision>
-        <origin rpy="0 0 0" xyz="0 0 0"/>
+        <origin xyz="0 0 0" rpy="0 0 0"/>
         <geometry>
           <box size=".585 .0602 .1790"/>
@@ -160,5 +160,5 @@
       </inertial>
       <visual>
-        <origin rpy="0 0 0" xyz="0 0 0"/>
+        <origin xyz="0 0 0" rpy="0 0 0"/>
         <geometry>
           <mesh filename="package://tahoma_description/meshes/stand/control_box.stl"/>
@@ -167,5 +167,5 @@
       </visual>
       <collision>
-        <origin rpy="0 0 0" xyz="0 0 0"/>
+        <origin xyz="0 0 0" rpy="0 0 0"/>
         <geometry>
           <box size=".46 .25 .44"/>
@@ -179,5 +179,5 @@
       </inertial>
       <visual>
-        <origin rpy="0 0 0" xyz="0 0 0"/>
+        <origin xyz="0 0 0" rpy="0 0 0"/>
         <geometry>
           <mesh filename="package://tahoma_description/meshes/stand/robot_plate.stl"/>
@@ -186,5 +186,5 @@
       </visual>
       <collision>
-        <origin rpy="0 0 0" xyz="0 0 0"/>
+        <origin xyz="0 0 0" rpy="0 0 0"/>
         <geometry>
           <box size=".225 .225 .0225"/>
@@ -201,20 +201,20 @@
       <parent link="stand"/>
       <child link="stand_upright"/>
-      <origin rpy="0 0 0" xyz="-.12 0 .95"/>
+      <origin xyz="-.12 0 .95" rpy="0 0 0"/>
     </joint>
     <joint name="stand_upright_stand_brace_joint" type="fixed">
       <parent link="stand_upright"/>
       <child link="stand_brace"/>
-      <origin rpy="0 0 0" xyz="-.24 0 -.59"/>
+      <origin xyz="-.24 0 -.59" rpy="0 0 0"/>
     </joint>
     <joint name="stand_upright_camera_beam_lower_joint" type="fixed">
       <parent link="stand_upright"/>
       <child link="camera_beam_lower"/>
-      <origin rpy="0 0 0" xyz="-.1225 0 .193"/>
+      <origin xyz="-.1225 0 .193" rpy="0 0 0"/>
     </joint>
     <joint name="stand_upright_robot_control_box_mount_joint" type="fixed">
       <parent link="stand_upright"/>
       <child link="control_box_mount"/>
-      <origin rpy="0 0 0" xyz="-.1725 .7475 .21"/>
+      <origin xyz="-.1725 .7475 .21" rpy="0 0 0"/>
     </joint>
     <joint name="control_box_mount_control_box_joint" type="fixed">
@@ -226,30 +226,30 @@
       <parent link="stand_upright"/>
       <child link="cantilever"/>
-      <origin rpy="0 0 0" xyz=".0775 0  0.9442"/>
+      <origin xyz=".0775 0  0.9442" rpy="0 0 0"/>
     </joint>
     <joint name="cantilever_robot_plate_joint" type="fixed">
       <parent link="cantilever"/>
       <child link="robot_plate"/>
-      <origin rpy="0 0 0" xyz="0.2505 0 -.015"/>
+      <origin xyz="0.2505 0 -.015" rpy="0 0 0"/>
     </joint>
     <joint name="stand_front_right_caster_joint" type="fixed">
       <parent link="stand"/>
       <child link="front_right_caster"/>
-      <origin rpy="0 0 0" xyz=".405 -.7375 -0.1"/>
+      <origin xyz=".405 -.7375 -0.1" rpy="0 0 0"/>
     </joint>
     <joint name="stand_front_left_caster_joint" type="fixed">
       <parent link="stand"/>
       <child link="front_left_caster"/>
-      <origin rpy="0 0 0" xyz=".405 .7025 -0.1"/>
+      <origin xyz=".405 .7025 -0.1" rpy="0 0 0"/>
     </joint>
     <joint name="stand_back_right_caster_joint" type="fixed">
       <parent link="stand"/>
       <child link="back_right_caster"/>
-      <origin rpy="0 0 0" xyz="-.405 -.7375 -0.1"/>
+      <origin xyz="-.405 -.7375 -0.1" rpy="0 0 0"/>
     </joint>
     <joint name="stand_back_left_caster_joint" type="fixed">
       <parent link="stand"/>
       <child link="back_left_caster"/>
-      <origin rpy="0 0 0" xyz="-.405 .7025 -0.1"/>
+      <origin xyz="-.405 .7025 -0.1" rpy="0 0 0"/>
     </joint>
     <joint name="stand_left_light_panel_joint" type="fixed">
