Commit message: Use our updated 2F-85 model
Point to our fork of the Robotiq packages, where we've updated the gripper model to reflect v4 hardware
The fork also disables many of the unused packages to make our use a little cleaner
Drop a copy of the coupling now that it's up to date in the model
Add coupling cable cover to model

File: tahoma_description/urdf/tahoma.xacro (robot description, xacro)
@@ -45,7 +45,16 @@
     <link name="coupling">
       <visual>
-        <origin xyz="0 0 0" rpy="0 0 ${pi}"/>
+        <origin xyz="0 0 0" rpy="0 0 0"/>
         <geometry>
-          <mesh filename="package://tahoma_description/meshes/robotiq_gripper_coupling.stl"/>
+          <mesh filename="package://robotiq_2f_85_gripper_visualization/meshes/visual/coupling.stl"/>
+        </geometry>
+        <material name="">
+          <color rgba="0.1 0.1 0.1 1"/>
+        </material>
+      </visual>
+     <visual>
+        <origin xyz="0.0335 0 0.006" rpy="0 0 0"/>
+        <geometry>
+          <mesh filename="package://robotiq_2f_85_gripper_visualization/meshes/visual/connector_cover.stl"/>
         </geometry>
         <material name="">
@@ -54,15 +63,25 @@
       </visual>
       <collision>
+        <!-- Primitives are centered, so offset -->
+        <origin xyz="${(0.029 / 2) + 0.0335} 0 -0.013" rpy="0 0 0"/>
         <geometry>
-          <cylinder radius=".0375" length=".0139"/>
+          <box size=".029 0.033 .056"/>
+        </geometry>
+      </collision>
+      <collision>
+        <!-- Primitives are centered, so offset -->
+        <origin xyz="0 0 ${.0169 / 2}" rpy="0 0 0"/>
+        <geometry>
+          <cylinder radius=".0375" length=".0169"/>
         </geometry>
       </collision>
     </link>
     <joint name="coupling_link_gripper_robotiq_arg2f_base_link_joint" type="fixed">
-      <origin xyz="0 0 0.012" rpy="0 0 ${pi/2}"/>
+      <origin xyz="0 0 0.0139" rpy="0 0 0"/>
       <parent link="coupling"/>
       <child link="gripper_base_link"/>
     </joint>
     <joint name="arm_tool0-coupling_joint" type="fixed">
+      <origin xyz="0 0 -0.003" rpy="0 0 ${1.5 * pi}"/>
       <parent link="arm_tool0"/>
       <child link="coupling"/>

Commit message: Fix and enhance many motion-related behaviors
Add servo states
Separate out and correctly implement "move to offset of current end effector pose" states. Previous implementation was only correct for base_link and wasn't clearly described by the name of its state
Add "robust" offset move sub state machine that rolls through movement options
Fix controller switching for real robot. Requires some elaboration of which controllers have resource conflicts so we can correctly disable whichever controller has what we need
Manually check goal tolerance for cartesian plan method so we ignore spurious aborts when they're harmless
Fix move_to_joint_angles tolerance check for named joint configurations
Turn up servo gains
Tweak home pose to level the gripper
Tweak controller configuration to make full-stop on switch happen faster. Trying to prevent drooping when switching controllers which I've observed both on the real robot and the simulator

File: tahoma_description/urdf/tahoma.xacro (robot description, xacro)
@@ -117,5 +117,5 @@
         <parent link="camera_beam_lower"/>
         <child link="camera_lower_right_mount"/>
-        <origin xyz="-0.00 ${-0.0215 + -camera_baseline / 2} 0.09"
+        <origin xyz="-0.00 ${-0.0215 + -camera_baseline / 2} 0.13"
                 rpy="${pi / 2} 0 ${math.atan2((camera_baseline /2),camera_focal_depth)}"/>
       </joint>

Commit message: Add and use a grasp frame
Add a frame to robot that expresses the theoretical center point between the fingers at which the robotiq 2f-85 would produce an equilibrium grasp (and not an enveloping grasp where the fingers bend around the object)
Specify grasping motions in this frame using MoveIt's end-effector APIs manually, for the moment
Make grasp service produce candidate grasps exactly, and make the caller responsible for creating the pregrasp target

File: tahoma_description/urdf/tahoma.xacro (robot description, xacro)
@@ -197,3 +197,10 @@
     </xacro:if>
   </xacro:macro>
+  <link name="gripper_equilibrium_grasp"/>
+  <joint name="gripper_base_link_gripper_equilibrium_grasp" type="fixed">
+    <parent link="gripper_base_link"/>
+      <child link="gripper_equilibrium_grasp"/>
+      <origin xyz="0 0 0.13"
+              rpy="0 0 0"/>
+  </joint>
 </robot>

Commit message: Update hardware bringup to match current robot configuration
Update camera mounts
Add second camera, disabled until interference is resolved
Update pod transform
Update some named joint configurations to keep them out of the way of the current camera mounts

File: tahoma_description/urdf/tahoma.xacro (robot description, xacro)
@@ -111,12 +111,12 @@
         <child link="camera_lower_left_mount"/>
         <!-- Link is centered on the optical frames. Slight offset in Y direction to compensate -->
-        <origin xyz="-0.00 0.02 0.06"
-                rpy="0 0 0"/>
+        <origin xyz="0.02 ${-0.0215 + (camera_baseline / 2)} 0.14"
+                rpy="${pi / 2} ${radians(15)} ${-math.atan2((camera_baseline /2),camera_focal_depth)}"/>
       </joint>
       <joint name="camera_beam_lower_camera_lower_right_mount_joint" type="fixed">
         <parent link="camera_beam_lower"/>
         <child link="camera_lower_right_mount"/>
-        <origin xyz="-0.00 ${-0.0215 + -camera_baseline / 2} 0.13"
-                rpy="${pi / 2} 0 ${math.atan2((camera_baseline /2),camera_focal_depth)}"/>
+        <origin xyz="0.02 ${0.0215 + (-camera_baseline / 2)} 0.14"
+                rpy="${pi / 2} ${radians(15)} ${math.atan2((camera_baseline /2),camera_focal_depth)}"/>
       </joint>
     </xacro:if>

Commit message: Add wirst camera to description

File: tahoma_description/urdf/tahoma.xacro (robot description, xacro)
@@ -178,4 +178,11 @@
               rpy="0 ${radians(15)} 0"/>
     </joint>
+    <!-- Wrist Camera -->
+    <link name="camera_wrist_mount"/>
+    <joint name="arm_wrist_3_link_camera_wrist_mount_joint" type="fixed">
+        <parent link="arm_wrist_3_link"/>
+        <child link="camera_wrist_mount"/>
+        <origin xyz="0.07 0.00 0.00" rpy="${pi} ${-pi / 2} 0"/>
+    </joint>
     <xacro:if value="${realsense}">
       <xacro:sensor_l515 name="camera_lower_right" parent="camera_lower_right_mount" use_nominal_extrinsics="${use_nominal_camera_extrinsics}">
@@ -195,4 +202,8 @@
         <origin xyz="0 0 0" rpy="0 0 0"/>
       </xacro:sensor_l515> -->
+      <!-- Wrist Camera -->
+      <xacro:sensor_l515 name="camera_wrist" parent="camera_wrist_mount" use_nominal_extrinsics="${use_nominal_camera_extrinsics}">
+        <origin xyz="0 0 0" rpy="0 0 0"/>
+      </xacro:sensor_l515>
     </xacro:if>
   </xacro:macro>

Commit message: Improve camera pose

File: tahoma_description/urdf/tahoma.xacro (robot description, xacro)
@@ -183,5 +183,5 @@
         <parent link="arm_wrist_3_link"/>
         <child link="camera_wrist_mount"/>
-        <origin xyz="0.07 0.00 0.00" rpy="${pi} ${-pi / 2} 0"/>
+        <origin xyz="0.00 -0.07 0.00" rpy="${pi/2} ${-pi / 2} 0"/>
     </joint>
     <xacro:if value="${realsense}">

Commit message: Update Tahoma model with new camera, camera mount URDFs
Add wrist camera
Use new back-mount parameter to simply attaching the cameras to the new mounts
Update collision matrix so MoveIt behaves well for the tweaked geometry
Update camera mount manual transform overrides to use the new frame names

File: tahoma_description/urdf/tahoma.xacro (robot description, xacro)
@@ -3,9 +3,12 @@
   <xacro:include filename="$(find ur_description)/urdf/inc/ur16e_macro.xacro"/>
   <xacro:include filename="$(find tahoma_description)/urdf/stand.xacro"/>
+  <xacro:include filename="$(find tahoma_description)/urdf/camera_mount_tilted.xacro"/>
   <xacro:include filename="$(find robotiq_2f_85_gripper_visualization)/urdf/robotiq_arg2f_85_macro.xacro"/>
-  <xacro:include filename="$(find realsense2_description)/urdf/_l515.urdf.xacro"/>
+  <xacro:include filename="$(find tahoma_description)/urdf/l515.xacro"/>
+  <xacro:include filename="$(find tahoma_description)/urdf/d405.xacro"/>
   <xacro:macro name="tahoma" params="
   realsense:=true
   use_nominal_camera_extrinsics:=false
+  wrist_camera:='true'
   camera_arrangement:='manual'
   camera_baseline:=.5
@@ -22,12 +25,12 @@
     <xacro:stand/>
     <xacro:ur16e_robot prefix="arm_"
-        joint_limits_parameters_file="${joint_limits_parameters_file}"
-        kinematics_parameters_file="${kinematics_parameters_file}"
-        physical_parameters_file="${physical_parameters_file}"
-        visual_parameters_file="${visual_parameters_file}"
-        transmission_hw_interface="${transmission_hw_interface}"
-        safety_limits="${safety_limits}"
-        safety_pos_margin="${safety_pos_margin}"
-        safety_k_position="${safety_k_position}"/>
+                       joint_limits_parameters_file="${joint_limits_parameters_file}"
+                       kinematics_parameters_file="${kinematics_parameters_file}"
+                       physical_parameters_file="${physical_parameters_file}"
+                       visual_parameters_file="${visual_parameters_file}"
+                       transmission_hw_interface="${transmission_hw_interface}"
+                       safety_limits="${safety_limits}"
+                       safety_pos_margin="${safety_pos_margin}"
+                       safety_k_position="${safety_k_position}"/>
     <xacro:robotiq_arg2f_85
             prefix="gripper_"
@@ -54,20 +57,4 @@
         </material>
       </visual>
-     <visual>
-        <origin xyz="0.0335 0 0.006" rpy="0 0 0"/>
-        <geometry>
-          <mesh filename="package://robotiq_2f_85_gripper_visualization/meshes/visual/connector_cover.stl"/>
-        </geometry>
-        <material name="">
-          <color rgba="0.1 0.1 0.1 1"/>
-        </material>
-      </visual>
-      <collision>
-        <!-- Primitives are centered, so offset -->
-        <origin xyz="${(0.029 / 2) + 0.0335} 0 -0.013" rpy="0 0 0"/>
-        <geometry>
-          <box size=".029 0.033 .056"/>
-        </geometry>
-      </collision>
       <collision>
         <!-- Primitives are centered, so offset -->
@@ -78,4 +65,45 @@
       </collision>
     </link>
+    <xacro:unless value="${wrist_camera}">
+      <!-- Assume we'll have the connector cover installed -->
+      <link name="coupling_connector_cover">
+        <visual>
+          <origin xyz="0.0335 0 0.006" rpy="0 0 0"/>
+          <geometry>
+            <mesh filename="package://robotiq_2f_85_gripper_visualization/meshes/visual/connector_cover.stl"/>
+          </geometry>
+          <material name="">
+            <color rgba="0.1 0.1 0.1 1"/>
+          </material>
+        </visual>
+        <collision>
+          <!-- Primitives are centered, so offset -->
+          <origin xyz="${(0.029 / 2) + 0.0335} 0 -0.013" rpy="0 0 0"/>
+          <geometry>
+            <box size=".029 0.033 .056"/>
+          </geometry>
+        </collision>
+      </link>
+      <joint name="coupling_coupling_connector_cover" type="fixed">
+        <origin xyz="0 0 0" rpy="0 0 0"/>
+        <parent link="coupling"/>
+        <child link="coupling_connector_cover"/>
+      </joint>
+    </xacro:unless>
+    <xacro:if value="${wrist_camera}">
+      <!-- We use the coupling connector cover mount points to attach our camera mount -->
+      <link name="gripper_camera_mount"/>
+      <link name="gripper_camera_mount_attach_point"/>
+      <joint name="coupling_wrist_camera_mount" type="fixed">
+        <origin xyz="0.0335 0 0.006" rpy="${pi / 2} -${pi / 2} ${pi / 2}"/>
+        <parent link="coupling"/>
+        <child link="gripper_camera_mount"/>
+      </joint>
+      <joint name="gripper_camera_mount-gripper_camera_mount_attach_point" type="fixed">
+        <origin xyz="-0.01 0 0.035" rpy="0 0 0"/>
+        <parent link="gripper_camera_mount"/>
+        <child link="gripper_camera_mount_attach_point"/>
+      </joint>
+    </xacro:if>
     <joint name="coupling_link_gripper_robotiq_arg2f_base_link_joint" type="fixed">
       <origin xyz="0 0 0.0139" rpy="0 0 0"/>
@@ -88,20 +116,6 @@
       <child link="coupling"/>
     </joint>
-    <link name="camera_lower_right_mount">
-      <collision>
-        <origin xyz="0 0 0" rpy="0 0 0"/>
-        <geometry>
-          <box size=".1 .15 .15"/>
-        </geometry>
-      </collision>
-    </link>
-    <link name="camera_lower_left_mount">
-      <collision>
-        <origin xyz="0 0 0" rpy="0 0 0"/>
-        <geometry>
-          <box size=".1 .15 .15"/>
-        </geometry>
-      </collision>
-    </link>
+      <xacro:camera_mount_tilted prefix="camera_lower_left_" side="left"/>
+      <xacro:camera_mount_tilted prefix="camera_lower_right_" side="right"/>
     <!-- These are the planned ("nominal") mount placements. On the real system, these should
      be overridden by calibrated transforms published separately -->
@@ -111,12 +125,12 @@
         <child link="camera_lower_left_mount"/>
         <!-- Link is centered on the optical frames. Slight offset in Y direction to compensate -->
-        <origin xyz="0.02 ${-0.0215 + (camera_baseline / 2)} 0.14"
-                rpy="${pi / 2} ${radians(15)} ${-math.atan2((camera_baseline /2),camera_focal_depth)}"/>
+        <origin xyz="0 ${-0.0215 + (camera_baseline / 2)} 0.042"
+                rpy="0 0 0"/>
       </joint>
       <joint name="camera_beam_lower_camera_lower_right_mount_joint" type="fixed">
         <parent link="camera_beam_lower"/>
         <child link="camera_lower_right_mount"/>
-        <origin xyz="0.02 ${0.0215 + (-camera_baseline / 2)} 0.14"
-                rpy="${pi / 2} ${radians(15)} ${math.atan2((camera_baseline /2),camera_focal_depth)}"/>
+        <origin xyz="0 ${0.0215 + (-camera_baseline / 2)} 0.042"
+                rpy="0 0 0"/>
       </joint>
     </xacro:if>
@@ -127,5 +141,5 @@
         <!-- Link is centered on the optical frames. Slight offset in Y direction to compensate -->
         <origin xyz="0 ${-0.0215 + -camera_baseline / 2} 0.09"
-                rpy="${pi / 2} 0 ${-math.atan2((camera_baseline /2),camera_focal_depth)}"/>
+                rpy="0 0 0"/>
       </joint>
       <joint name="camera_beam_lower_camera_lower_right_mount_joint" type="fixed">
@@ -133,5 +147,5 @@
         <child link="camera_lower_right_mount"/>
         <origin xyz="0 ${-0.0215 + -camera_baseline / 2} 0.09"
-                rpy="${pi / 2} 0 ${math.atan2((camera_baseline /2),camera_focal_depth)}"/>
+                rpy="0 0 0"/>
       </joint>
     </xacro:if>
@@ -179,13 +193,22 @@
     </joint>
     <xacro:if value="${realsense}">
-      <xacro:sensor_l515 name="camera_lower_right" parent="camera_lower_right_mount" use_nominal_extrinsics="${use_nominal_camera_extrinsics}">
-        <origin xyz="0 0 0" rpy="0 0 0"/>
-      </xacro:sensor_l515>
-      <xacro:sensor_l515 name="camera_lower_left" parent="camera_lower_left_mount" use_nominal_extrinsics="${use_nominal_camera_extrinsics}">
-        <origin xyz="0 0 0" rpy="0 0 0"/>
-      </xacro:sensor_l515>
-      <xacro:sensor_l515 name="camera_upper" parent="camera_upper_mount" use_nominal_extrinsics="${use_nominal_camera_extrinsics}">
-        <origin xyz="0 0 0" rpy="0 0 0"/>
-      </xacro:sensor_l515>
+      <xacro:sensor_l515 name="camera_lower_right" parent="camera_lower_right_mount_attach_point"
+                         use_nominal_extrinsics="${use_nominal_camera_extrinsics}" attach_at_bottom="false">
+        <origin xyz="0 0 0" rpy="0 0 0"/>
+      </xacro:sensor_l515>
+      <xacro:sensor_l515 name="camera_lower_left" parent="camera_lower_left_mount_attach_point"
+                         use_nominal_extrinsics="${use_nominal_camera_extrinsics}" attach_at_bottom="false">
+        <origin xyz="0 0 0" rpy="0 0 0"/>
+      </xacro:sensor_l515>
+      <xacro:sensor_l515 name="camera_upper" parent="camera_upper_mount"
+                         use_nominal_extrinsics="${use_nominal_camera_extrinsics}" attach_at_bottom="false">
+        <origin xyz="0 0 0" rpy="0 0 0"/>
+      </xacro:sensor_l515>
+      <xacro:if value="${wrist_camera}">
+        <xacro:sensor_d405 name="camera_wrist" parent="gripper_camera_mount_attach_point"
+                           use_nominal_extrinsics="${use_nominal_camera_extrinsics}" attach_at_bottom="false">
+          <origin xyz="0 0 0" rpy="0 0 0"/>
+        </xacro:sensor_d405>
+      </xacro:if>
       <!-- Upper cameras
       <xacro:sensor_l515 name="camera_upper_right" parent="camera_upper_right_mount" use_nominal_extrinsics="${use_nominal_camera_extrinsics}">
@@ -200,7 +223,7 @@
   <joint name="gripper_base_link_gripper_equilibrium_grasp" type="fixed">
     <parent link="gripper_base_link"/>
-      <child link="gripper_equilibrium_grasp"/>
-      <origin xyz="0 0 0.13"
-              rpy="0 0 0"/>
+    <child link="gripper_equilibrium_grasp"/>
+    <origin xyz="0 0 0.13"
+            rpy="0 0 0"/>
   </joint>
 </robot>

Commit message: pre-demo commit dump:

File: tahoma_description/urdf/tahoma.xacro (robot description, xacro)
@@ -3,5 +3,6 @@
   <xacro:include filename="$(find ur_description)/urdf/inc/ur16e_macro.xacro"/>
   <xacro:include filename="$(find tahoma_description)/urdf/stand.xacro"/>
-  <xacro:include filename="$(find robotiq_2f_85_gripper_visualization)/urdf/robotiq_arg2f_85_macro.xacro"/>
+  <!-- <xacro:include filename="$(find robotiq_2f_85_gripper_visualization)/urdf/robotiq_arg2f_85_macro.xacro"/> -->
+  <xacro:include filename="$(find robotiq_epick_visualization)/urdf/robotiq_epick_model_macro.xacro" />
   <!-- <xacro:include filename="$(find realsense2_description)/urdf/_l515.urdf.xacro"/> -->
   <xacro:macro name="tahoma" params="
@@ -31,7 +32,8 @@
         safety_pos_margin="${safety_pos_margin}"
         safety_k_position="${safety_k_position}"/>
-    <xacro:robotiq_arg2f_85
+    <!-- <xacro:robotiq_arg2f_85
             prefix="gripper_"
-            transmission_hw_interface="${gripper_transmission_hw_interface}"/>
+            transmission_hw_interface="${gripper_transmission_hw_interface}"/> -->
+    <xacro:epick_hand hand_link_name="gripper_base_link" robot_name="tahoma"/>
     <link name="base_link"/>
     <joint name="base_joint" type="fixed">
@@ -66,7 +68,7 @@
       <collision>
         <!-- Primitives are centered, so offset -->
-        <origin xyz="${(0.029 / 2) + 0.0335} 0 -0.013" rpy="0 0 0"/>
-        <geometry>
-          <box size=".029 0.033 .056"/>
+        <origin xyz="${(0.015 / 2) + 0.0335} 0 -0.013" rpy="0 0 0"/>
+        <geometry>
+          <box size=".015 0.033 .056"/>
         </geometry>
       </collision>
@@ -80,5 +82,5 @@
     </link>
     <joint name="coupling_link_gripper_robotiq_arg2f_base_link_joint" type="fixed">
-      <origin xyz="0 0 0.0139" rpy="0 0 0"/>
+      <origin xyz="0 0 0.017" rpy="0 0 0"/>
       <parent link="coupling"/>
       <child link="gripper_base_link"/>
@@ -182,9 +184,8 @@
       <xacro:include filename="$(find tahoma_description)/urdf/azure_kinect.urdf.xacro"/>
       <joint name="kinect_base_joint" type="fixed">
-        <parent link="camera_beam_lower"/>
+        <parent link="base_link"/>
         <child link="camera_base"/>
         <!-- Link is centered on the optical frames. Slight offset in Y direction to compensate -->
-        <origin xyz="0 0 .09"
-                rpy="0 0 0"/>
+        <origin xyz="-0.245645 ${0.000778815-.02} 1.41034" rpy="3.13764 3.12912 -3.12899" />
       </joint>
     </xacro:if>
@@ -210,7 +211,7 @@
   <link name="gripper_equilibrium_grasp"/>
   <joint name="gripper_base_link_gripper_equilibrium_grasp" type="fixed">
-    <parent link="gripper_base_link"/>
+    <parent link="epick_end_effector"/>
       <child link="gripper_equilibrium_grasp"/>
-      <origin xyz="0 0 0.13"
+      <origin xyz="0 0 0"
               rpy="0 0 0"/>
   </joint>

Commit message: Pre-Demo stable state

File: tahoma_description/urdf/tahoma.xacro (robot description, xacro)
@@ -187,5 +187,5 @@
         <child link="camera_base"/>
         <!-- Link is centered on the optical frames. Slight offset in Y direction to compensate -->
-        <origin xyz="-0.245645 ${0.000778815-.02} 1.41034" rpy="3.13764 3.12912 -3.12899" />
+        <origin xyz="-0.245645 ${0.000778815-.0125} 1.41034" rpy="3.13764 3.12912 -3.12899" />
       </joint>
     </xacro:if>
