Commit message: Revert "Update Tahoma model with new camera, camera mount URDFs"
This reverts commit 5cd8aabf1c2c4193a6128a671f30e45fd4c4c0f7.

File: tahoma_description/urdf/tahoma.xacro (robot description, xacro)
@@ -3,12 +3,9 @@
   <xacro:include filename="$(find ur_description)/urdf/inc/ur16e_macro.xacro"/>
   <xacro:include filename="$(find tahoma_description)/urdf/stand.xacro"/>
-  <xacro:include filename="$(find tahoma_description)/urdf/camera_mount_tilted.xacro"/>
   <xacro:include filename="$(find robotiq_2f_85_gripper_visualization)/urdf/robotiq_arg2f_85_macro.xacro"/>
-  <xacro:include filename="$(find tahoma_description)/urdf/l515.xacro"/>
-  <xacro:include filename="$(find tahoma_description)/urdf/d405.xacro"/>
+  <xacro:include filename="$(find realsense2_description)/urdf/_l515.urdf.xacro"/>
   <xacro:macro name="tahoma" params="
   realsense:=true
   use_nominal_camera_extrinsics:=false
-  wrist_camera:='true'
   camera_arrangement:='manual'
   camera_baseline:=.5
@@ -25,12 +22,12 @@
     <xacro:stand/>
     <xacro:ur16e_robot prefix="arm_"
-                       joint_limits_parameters_file="${joint_limits_parameters_file}"
-                       kinematics_parameters_file="${kinematics_parameters_file}"
-                       physical_parameters_file="${physical_parameters_file}"
-                       visual_parameters_file="${visual_parameters_file}"
-                       transmission_hw_interface="${transmission_hw_interface}"
-                       safety_limits="${safety_limits}"
-                       safety_pos_margin="${safety_pos_margin}"
-                       safety_k_position="${safety_k_position}"/>
+        joint_limits_parameters_file="${joint_limits_parameters_file}"
+        kinematics_parameters_file="${kinematics_parameters_file}"
+        physical_parameters_file="${physical_parameters_file}"
+        visual_parameters_file="${visual_parameters_file}"
+        transmission_hw_interface="${transmission_hw_interface}"
+        safety_limits="${safety_limits}"
+        safety_pos_margin="${safety_pos_margin}"
+        safety_k_position="${safety_k_position}"/>
     <xacro:robotiq_arg2f_85
             prefix="gripper_"
@@ -57,4 +54,20 @@
         </material>
       </visual>
+     <visual>
+        <origin xyz="0.0335 0 0.006" rpy="0 0 0"/>
+        <geometry>
+          <mesh filename="package://robotiq_2f_85_gripper_visualization/meshes/visual/connector_cover.stl"/>
+        </geometry>
+        <material name="">
+          <color rgba="0.1 0.1 0.1 1"/>
+        </material>
+      </visual>
+      <collision>
+        <!-- Primitives are centered, so offset -->
+        <origin xyz="${(0.029 / 2) + 0.0335} 0 -0.013" rpy="0 0 0"/>
+        <geometry>
+          <box size=".029 0.033 .056"/>
+        </geometry>
+      </collision>
       <collision>
         <!-- Primitives are centered, so offset -->
@@ -65,45 +78,4 @@
       </collision>
     </link>
-    <xacro:unless value="${wrist_camera}">
-      <!-- Assume we'll have the connector cover installed -->
-      <link name="coupling_connector_cover">
-        <visual>
-          <origin xyz="0.0335 0 0.006" rpy="0 0 0"/>
-          <geometry>
-            <mesh filename="package://robotiq_2f_85_gripper_visualization/meshes/visual/connector_cover.stl"/>
-          </geometry>
-          <material name="">
-            <color rgba="0.1 0.1 0.1 1"/>
-          </material>
-        </visual>
-        <collision>
-          <!-- Primitives are centered, so offset -->
-          <origin xyz="${(0.029 / 2) + 0.0335} 0 -0.013" rpy="0 0 0"/>
-          <geometry>
-            <box size=".029 0.033 .056"/>
-          </geometry>
-        </collision>
-      </link>
-      <joint name="coupling_coupling_connector_cover" type="fixed">
-        <origin xyz="0 0 0" rpy="0 0 0"/>
-        <parent link="coupling"/>
-        <child link="coupling_connector_cover"/>
-      </joint>
-    </xacro:unless>
-    <xacro:if value="${wrist_camera}">
-      <!-- We use the coupling connector cover mount points to attach our camera mount -->
-      <link name="gripper_camera_mount"/>
-      <link name="gripper_camera_mount_attach_point"/>
-      <joint name="coupling_wrist_camera_mount" type="fixed">
-        <origin xyz="0.0335 0 0.006" rpy="${pi / 2} -${pi / 2} ${pi / 2}"/>
-        <parent link="coupling"/>
-        <child link="gripper_camera_mount"/>
-      </joint>
-      <joint name="gripper_camera_mount-gripper_camera_mount_attach_point" type="fixed">
-        <origin xyz="-0.01 0 0.035" rpy="0 0 0"/>
-        <parent link="gripper_camera_mount"/>
-        <child link="gripper_camera_mount_attach_point"/>
-      </joint>
-    </xacro:if>
     <joint name="coupling_link_gripper_robotiq_arg2f_base_link_joint" type="fixed">
       <origin xyz="0 0 0.0139" rpy="0 0 0"/>
@@ -116,6 +88,20 @@
       <child link="coupling"/>
     </joint>
-      <xacro:camera_mount_tilted prefix="camera_lower_left_" side="left"/>
-      <xacro:camera_mount_tilted prefix="camera_lower_right_" side="right"/>
+    <link name="camera_lower_right_mount">
+      <collision>
+        <origin xyz="0 0 0" rpy="0 0 0"/>
+        <geometry>
+          <box size=".1 .15 .15"/>
+        </geometry>
+      </collision>
+    </link>
+    <link name="camera_lower_left_mount">
+      <collision>
+        <origin xyz="0 0 0" rpy="0 0 0"/>
+        <geometry>
+          <box size=".1 .15 .15"/>
+        </geometry>
+      </collision>
+    </link>
     <!-- These are the planned ("nominal") mount placements. On the real system, these should
      be overridden by calibrated transforms published separately -->
@@ -125,12 +111,12 @@
         <child link="camera_lower_left_mount"/>
         <!-- Link is centered on the optical frames. Slight offset in Y direction to compensate -->
-        <origin xyz="0 ${-0.0215 + (camera_baseline / 2)} 0.042"
-                rpy="0 0 0"/>
+        <origin xyz="0.02 ${-0.0215 + (camera_baseline / 2)} 0.14"
+                rpy="${pi / 2} ${radians(15)} ${-math.atan2((camera_baseline /2),camera_focal_depth)}"/>
       </joint>
       <joint name="camera_beam_lower_camera_lower_right_mount_joint" type="fixed">
         <parent link="camera_beam_lower"/>
         <child link="camera_lower_right_mount"/>
-        <origin xyz="0 ${0.0215 + (-camera_baseline / 2)} 0.042"
-                rpy="0 0 0"/>
+        <origin xyz="0.02 ${0.0215 + (-camera_baseline / 2)} 0.14"
+                rpy="${pi / 2} ${radians(15)} ${math.atan2((camera_baseline /2),camera_focal_depth)}"/>
       </joint>
     </xacro:if>
@@ -141,5 +127,5 @@
         <!-- Link is centered on the optical frames. Slight offset in Y direction to compensate -->
         <origin xyz="0 ${-0.0215 + -camera_baseline / 2} 0.09"
-                rpy="0 0 0"/>
+                rpy="${pi / 2} 0 ${-math.atan2((camera_baseline /2),camera_focal_depth)}"/>
       </joint>
       <joint name="camera_beam_lower_camera_lower_right_mount_joint" type="fixed">
@@ -147,5 +133,5 @@
         <child link="camera_lower_right_mount"/>
         <origin xyz="0 ${-0.0215 + -camera_baseline / 2} 0.09"
-                rpy="0 0 0"/>
+                rpy="${pi / 2} 0 ${math.atan2((camera_baseline /2),camera_focal_depth)}"/>
       </joint>
     </xacro:if>
@@ -193,22 +179,13 @@
     </joint>
     <xacro:if value="${realsense}">
-      <xacro:sensor_l515 name="camera_lower_right" parent="camera_lower_right_mount_attach_point"
-                         use_nominal_extrinsics="${use_nominal_camera_extrinsics}" attach_at_bottom="false">
-        <origin xyz="0 0 0" rpy="0 0 0"/>
-      </xacro:sensor_l515>
-      <xacro:sensor_l515 name="camera_lower_left" parent="camera_lower_left_mount_attach_point"
-                         use_nominal_extrinsics="${use_nominal_camera_extrinsics}" attach_at_bottom="false">
-        <origin xyz="0 0 0" rpy="0 0 0"/>
-      </xacro:sensor_l515>
-      <xacro:sensor_l515 name="camera_upper" parent="camera_upper_mount"
-                         use_nominal_extrinsics="${use_nominal_camera_extrinsics}" attach_at_bottom="false">
-        <origin xyz="0 0 0" rpy="0 0 0"/>
-      </xacro:sensor_l515>
-      <xacro:if value="${wrist_camera}">
-        <xacro:sensor_d405 name="camera_wrist" parent="gripper_camera_mount_attach_point"
-                           use_nominal_extrinsics="${use_nominal_camera_extrinsics}" attach_at_bottom="false">
-          <origin xyz="0 0 0" rpy="0 0 0"/>
-        </xacro:sensor_d405>
-      </xacro:if>
+      <xacro:sensor_l515 name="camera_lower_right" parent="camera_lower_right_mount" use_nominal_extrinsics="${use_nominal_camera_extrinsics}">
+        <origin xyz="0 0 0" rpy="0 0 0"/>
+      </xacro:sensor_l515>
+      <xacro:sensor_l515 name="camera_lower_left" parent="camera_lower_left_mount" use_nominal_extrinsics="${use_nominal_camera_extrinsics}">
+        <origin xyz="0 0 0" rpy="0 0 0"/>
+      </xacro:sensor_l515>
+      <xacro:sensor_l515 name="camera_upper" parent="camera_upper_mount" use_nominal_extrinsics="${use_nominal_camera_extrinsics}">
+        <origin xyz="0 0 0" rpy="0 0 0"/>
+      </xacro:sensor_l515>
       <!-- Upper cameras
       <xacro:sensor_l515 name="camera_upper_right" parent="camera_upper_right_mount" use_nominal_extrinsics="${use_nominal_camera_extrinsics}">
@@ -223,7 +200,7 @@
   <joint name="gripper_base_link_gripper_equilibrium_grasp" type="fixed">
     <parent link="gripper_base_link"/>
-    <child link="gripper_equilibrium_grasp"/>
-    <origin xyz="0 0 0.13"
-            rpy="0 0 0"/>
+      <child link="gripper_equilibrium_grasp"/>
+      <origin xyz="0 0 0.13"
+              rpy="0 0 0"/>
   </joint>
 </robot>

Commit message: Adding new calibrated data between camera-base and base_link and also increasing the offset so that arm goes inside the bin and attaches the object firmly

File: tahoma_description/urdf/tahoma.xacro (robot description, xacro)
@@ -187,5 +187,5 @@
         <child link="camera_base"/>
         <!-- Link is centered on the optical frames. Slight offset in Y direction to compensate -->
-        <origin xyz="-0.245645 ${0.000778815-.0125} 1.41034" rpy="3.13764 3.12912 -3.12899" />
+        <origin xyz="-0.246 0.001 1.410" rpy="3.13764 3.12912 -3.12899" />
       </joint>
     </xacro:if>

Commit message: new changes for camera

File: tahoma_description/urdf/tahoma.xacro (robot description, xacro)
@@ -58,5 +58,5 @@
       </visual>
      <visual>
-        <origin xyz="0.0335 0 0.006" rpy="0 0 0"/>
+        <origin xyz="0.0335 0 0.0" rpy="0 0 0"/>
         <geometry>
           <mesh filename="package://robotiq_2f_85_gripper_visualization/meshes/visual/connector_cover.stl"/>
@@ -82,10 +82,10 @@
     </link>
     <joint name="coupling_link_gripper_robotiq_arg2f_base_link_joint" type="fixed">
-      <origin xyz="0 0 0.017" rpy="0 0 0"/>
+      <origin xyz="0 0 0.055" rpy="0 0 0"/>
       <parent link="coupling"/>
       <child link="gripper_base_link"/>
     </joint>
     <joint name="arm_tool0-coupling_joint" type="fixed">
-      <origin xyz="0 0 -0.003" rpy="0 0 ${1.5 * pi}"/>
+      <origin xyz="0 0 0" rpy="0 0 ${1.5 * pi}"/>
       <parent link="arm_tool0"/>
       <child link="coupling"/>
@@ -174,8 +174,8 @@
     </joint>
     -->
-    <link name="camera_upper_mount"/>
+    <link name="cantilever_camera_upper_mount"/>
     <joint name="cantilever_camera_upper_mount_joint" type="fixed">
       <parent link="cantilever"/>
-      <child link="camera_upper_mount"/>
+      <child link="cantilever_camera_upper_mount"/>
       <origin xyz=".02 0 0.37"
               rpy="0 ${radians(15)} 0"/>
@@ -187,7 +187,55 @@
         <child link="camera_base"/>
         <!-- Link is centered on the optical frames. Slight offset in Y direction to compensate -->
-        <origin xyz="-0.246 0.001 1.410" rpy="3.13764 3.12912 -3.12899" />
-      </joint>
-    </xacro:if>
+        <origin xyz="-0.260 0 1.465" rpy="3.13764 3.12912 -3.12899" />
+      </joint>
+    </xacro:if>
+    <xacro:arg name="use_nominal_extrinsics" default="false"/>
+    <xacro:arg name="add_plug" default="false" />
+    <xacro:arg name="use_mesh" default="true" />
+    <xacro:include filename="$(find tahoma_description)/urdf/_l515.urdf.xacro" />
+    <!-- D435 Realsense Camera -->
+    <!-- <xacro:sensor_d435 parent="base_link" use_nominal_extrinsics="$(arg use_nominal_extrinsics)" add_plug="$(arg add_plug)" use_mesh="$(arg use_mesh)">
+      <origin xyz="-0.217 0.013 1.354" rpy="0 0 0"/>
+    </xacro:sensor_d435> -->
+    <!-- D455 Realsense Camera -->
+    <!-- <xacro:sensor_d455 parent="base_link" use_nominal_extrinsics="$(arg use_nominal_extrinsics)">
+      <origin xyz="-0.217 -0.025 1.364" rpy="0 0 0"/>
+    </xacro:sensor_d455> -->
+    <link name="realsense_back_gripper_mount">
+      <collision>
+        <origin xyz="0.010227 -0.005 0.035" rpy="0 0 0"/>
+        <geometry>
+          <box size="0.04 0.02 0.08"/>
+        </geometry>
+      </collision>
+      <visual>
+        <origin xyz="0 0 0" rpy="0 0 0"/>
+        <geometry>
+          <mesh filename="package://tahoma_description/meshes/realsense/couple_l515_mount.obj"/>
+        </geometry>
+      </visual>
+    </link>
+    <!-- L515 Realsense Camera -->
+    <xacro:sensor_l515 parent="coupling" use_nominal_extrinsics="$(arg use_nominal_extrinsics)" add_plug="$(arg add_plug)" use_mesh="$(arg use_mesh)">
+      <origin xyz="0.0 0.046 0.1165" rpy="${pi} -${0.5 * pi} ${0.5 * pi}"/>
+    </xacro:sensor_l515>
+    <!-- <link name="realsense_lower_mount">
+      <collision>
+        <origin xyz="0 0 0" rpy="0 0 0"/>
+        <geometry>
+          <box size="0.06 0.1 0.06"/>
+        </geometry>
+      </collision>
+    </link>
+    <joint name="realsense_mount_joint" type="fixed">
+        <parent link="camera_bottom_screw_frame"/>
+        <child link="realsense_lower_mount"/>
+        <origin xyz="0.03 0 -0.05" rpy="0 0 0" />
+    </joint> -->
+    <joint name="realsense_back_gripper_mount_joint" type="fixed">
+        <parent link="camera_link"/>
+        <child link="realsense_back_gripper_mount"/>
+        <origin xyz="-0.018 0.010227 -0.036" rpy="0 0 ${-0.5 * pi}" />
+    </joint>
     <xacro:if value="${realsense}">
       <xacro:sensor_l515 name="camera_lower_right" parent="camera_lower_right_mount" use_nominal_extrinsics="${use_nominal_camera_extrinsics}">
@@ -197,5 +245,5 @@
         <origin xyz="0 0 0" rpy="0 0 0"/>
       </xacro:sensor_l515>
-      <xacro:sensor_l515 name="camera_upper" parent="camera_upper_mount" use_nominal_extrinsics="${use_nominal_camera_extrinsics}">
+      <xacro:sensor_l515 name="camera_upper" parent="cantilever_camera_upper_mount" use_nominal_extrinsics="${use_nominal_camera_extrinsics}">
         <origin xyz="0 0 0" rpy="0 0 0"/>
       </xacro:sensor_l515>

Commit message: new changes for camera

File: tahoma_description/urdf/tahoma.xacro (robot description, xacro)
@@ -92,4 +92,94 @@
       <child link="coupling"/>
     </joint>
+    <link name="camera_lower_right_mount">
+      <collision>
+        <origin xyz="0 0 0" rpy="0 0 0"/>
+        <geometry>
+          <box size=".1 .15 .15"/>
+        </geometry>
+      </collision>
+    </link>
+    <link name="camera_lower_left_mount">
+      <collision>
+        <origin xyz="0 0 0" rpy="0 0 0"/>
+        <geometry>
+          <box size=".1 .15 .15"/>
+        </geometry>
+      </collision>
+    </link>
+    <!-- These are the planned ("nominal") mount placements. On the real system, these should
+     be overridden by calibrated transforms published separately -->
+    <xacro:if value="${camera_arrangement == 'manual' }">
+      <joint name="camera_beam_lower_camera_lower_left_mount_joint" type="fixed">
+        <parent link="camera_beam_lower"/>
+        <child link="camera_lower_left_mount"/>
+        <!-- Link is centered on the optical frames. Slight offset in Y direction to compensate -->
+        <origin xyz="0.02 ${-0.0215 + (camera_baseline / 2)} 0.14"
+                rpy="${pi / 2} ${radians(15)} ${-atan2((camera_baseline /2),camera_focal_depth)}"/>
+      </joint>
+      <joint name="camera_beam_lower_camera_lower_right_mount_joint" type="fixed">
+        <parent link="camera_beam_lower"/>
+        <child link="camera_lower_right_mount"/>
+        <origin xyz="0.02 ${0.0215 + (-camera_baseline / 2)} 0.14"
+                rpy="${pi / 2} ${radians(15)} ${atan2((camera_baseline /2),camera_focal_depth)}"/>
+      </joint>
+    </xacro:if>
+    <xacro:if value="${camera_arrangement == 'convergent' }">
+      <joint name="camera_beam_lower_camera_lower_left_mount_joint" type="fixed">
+        <parent link="camera_beam_lower"/>
+        <child link="camera_lower_left_mount"/>
+        <!-- Link is centered on the optical frames. Slight offset in Y direction to compensate -->
+        <origin xyz="0 ${-0.0215 + -camera_baseline / 2} 0.09"
+                rpy="${pi / 2} 0 ${-atan2((camera_baseline /2),camera_focal_depth)}"/>
+      </joint>
+      <joint name="camera_beam_lower_camera_lower_right_mount_joint" type="fixed">
+        <parent link="camera_beam_lower"/>
+        <child link="camera_lower_right_mount"/>
+        <origin xyz="0 ${-0.0215 + -camera_baseline / 2} 0.09"
+                rpy="${pi / 2} 0 ${atan2((camera_baseline /2),camera_focal_depth)}"/>
+      </joint>
+    </xacro:if>
+    <xacro:if value="${camera_arrangement == 'convergent_tilted' }">
+      <joint name="camera_beam_lower_camera_lower_left_mount_joint" type="fixed">
+        <parent link="camera_beam_lower"/>
+        <child link="camera_lower_left_mount"/>
+        <!-- Link is centered on the optical frames. Slight offset in Y direction to compensate -->
+        <origin xyz="-0.00 ${-0.0215 + (camera_baseline / 2)} 0.09"
+                rpy="${pi / 2} ${radians(15)} ${-atan2((camera_baseline /2),camera_focal_depth)}"/>
+      </joint>
+      <joint name="camera_beam_lower_camera_lower_right_mount_joint" type="fixed">
+        <parent link="camera_beam_lower"/>
+        <child link="camera_lower_right_mount"/>
+        <origin xyz="-0.00 ${0.0215 + (-camera_baseline / 2)} 0.09"
+                rpy="${pi / 2} ${radians(15)} ${atan2((camera_baseline /2),camera_focal_depth)}"/>
+      </joint>
+    </xacro:if>
+    <!-- Upper cameras -->
+    <!-- Link is centered on the optical frames. Slight offset in Y direction to compensate -->
+    <!-- Z=1.10 for on top of the top beam -->
+    <!-- Z=0.80 for underneath the top beam -->
+    <!-- Disabled until we know about manipulability in upper bins
+    <link name="camera_upper_right_mount"/>
+    <link name="camera_upper_left_mount"/>
+    <joint name="stand_upright_camera_upper_left_mount_joint" type="fixed">
+      <parent link="stand_upright"/>
+      <child link="camera_upper_left_mount"/>
+      <origin xyz="-.1 ${-0.0215 + (camera_baseline / 2)} 0.80"
+              rpy="${pi / 2} ${radians(15)} ${-atan2((camera_baseline /2),camera_focal_depth)}"/>
+    </joint>
+    <joint name="stand_upright_camera_upper_right_mount_joint" type="fixed">
+      <parent link="stand_upright"/>
+      <child link="camera_upper_right_mount"/>
+      <origin xyz="-.1 ${0.0215 + (-camera_baseline / 2)} 0.80"
+              rpy="${pi / 2} ${radians(15)} ${atan2((camera_baseline /2),camera_focal_depth)}"/>
+    </joint>
+    -->
+    <link name="cantilever_camera_upper_mount"/>
+    <joint name="cantilever_camera_upper_mount_joint" type="fixed">
+      <parent link="cantilever"/>
+      <child link="cantilever_camera_upper_mount"/>
+      <origin xyz=".02 0 0.37"
+              rpy="0 ${radians(15)} 0"/>
+    </joint>
     <xacro:if value="${azure_kinect}">
       <xacro:include filename="$(find tahoma_description)/urdf/azure_kinect.urdf.xacro"/>
@@ -98,8 +188,19 @@
         <child link="camera_base"/>
         <!-- Link is centered on the optical frames. Slight offset in Y direction to compensate -->
-        <origin xyz="-0.256 -0.0277 1.4245" rpy="3.14 3.14 -3.14" />
-        <!-- <origin xyz="-0.2426 -0.0277 1.4078" rpy="3.14 3.14 -3.14" /> -->
-      </joint>
-    </xacro:if>
+        <origin xyz="-0.260 0 1.465" rpy="3.13764 3.12912 -3.12899" />
+      </joint>
+    </xacro:if>
+    <xacro:arg name="use_nominal_extrinsics" default="false"/>
+    <xacro:arg name="add_plug" default="false" />
+    <xacro:arg name="use_mesh" default="true" />
+    <xacro:include filename="$(find tahoma_description)/urdf/_l515.urdf.xacro" />
+    <!-- D435 Realsense Camera -->
+    <!-- <xacro:sensor_d435 parent="base_link" use_nominal_extrinsics="$(arg use_nominal_extrinsics)" add_plug="$(arg add_plug)" use_mesh="$(arg use_mesh)">
+      <origin xyz="-0.217 0.013 1.354" rpy="0 0 0"/>
+    </xacro:sensor_d435> -->
+    <!-- D455 Realsense Camera -->
+    <!-- <xacro:sensor_d455 parent="base_link" use_nominal_extrinsics="$(arg use_nominal_extrinsics)">
+      <origin xyz="-0.217 -0.025 1.364" rpy="0 0 0"/>
+    </xacro:sensor_d455> -->
     <link name="realsense_back_gripper_mount">
       <collision>
@@ -116,4 +217,47 @@
       </visual>
     </link>
+    <!-- L515 Realsense Camera -->
+    <xacro:sensor_l515 parent="coupling" use_nominal_extrinsics="$(arg use_nominal_extrinsics)" add_plug="$(arg add_plug)" use_mesh="$(arg use_mesh)">
+      <origin xyz="0.0 0.046 0.1165" rpy="${pi} -${0.5 * pi} ${0.5 * pi}"/>
+    </xacro:sensor_l515>
+    <!-- <link name="realsense_lower_mount">
+      <collision>
+        <origin xyz="0 0 0" rpy="0 0 0"/>
+        <geometry>
+          <box size="0.06 0.1 0.06"/>
+        </geometry>
+      </collision>
+    </link>
+    <joint name="realsense_mount_joint" type="fixed">
+        <parent link="camera_bottom_screw_frame"/>
+        <child link="realsense_lower_mount"/>
+        <origin xyz="0.03 0 -0.05" rpy="0 0 0" />
+    </joint> -->
+    <joint name="realsense_back_gripper_mount_joint" type="fixed">
+        <parent link="camera_link"/>
+        <child link="realsense_back_gripper_mount"/>
+        <origin xyz="-0.018 0.010227 -0.036" rpy="0 0 ${-0.5 * pi}" />
+    </joint>
+    <xacro:if value="${realsense}">
+      <xacro:sensor_l515 name="camera_lower_right" parent="camera_lower_right_mount" use_nominal_extrinsics="${use_nominal_camera_extrinsics}">
+        <origin xyz="0 0 0" rpy="0 0 0"/>
+      </xacro:sensor_l515>
+    <link name="realsense_back_gripper_mount">
+      <collision>
+        <origin xyz="0.010227 -0.005 0.035" rpy="0 0 0"/>
+        <geometry>
+          <box size="0.04 0.02 0.08"/>
+        </geometry>
+      </collision>
+      <visual>
+        <origin xyz="0 0 0" rpy="0 0 0"/>
+        <geometry>
+          <mesh filename="package://tahoma_description/meshes/realsense/couple_l515_mount.obj"/>
+        </geometry>
+      </visual>
+    </link>
+      <xacro:sensor_l515 name="camera_upper" parent="cantilever_camera_upper_mount" use_nominal_extrinsics="${use_nominal_camera_extrinsics}">
+        <origin xyz="0 0 0" rpy="0 0 0"/>
+      </xacro:sensor_l515>
     <!-- L515 Realsense Camera -->
     <xacro:sensor_l515 parent="realsense_back_gripper_mount" use_nominal_extrinsics="${use_nominal_camera_extrinsics}" add_plug="false" use_mesh="true">
