Commit message: new changes for camera

File: tahoma_description/urdf/tahoma.xacro (robot description, xacro)
@@ -187,6 +187,5 @@
         <child link="camera_base"/>
         <!-- Link is centered on the optical frames. Slight offset in Y direction to compensate -->
-        <origin xyz="-0.20750794 -0.01749962  1.40753882" rpy="3.14 3.14 -3.14" />
-        <!-- <origin xyz="-0.2426 -0.0277 1.4078" rpy="3.14 3.14 -3.14" /> -->
+        <origin xyz="-0.260 0 1.465" rpy="3.13764 3.12912 -3.12899" />
       </joint>
     </xacro:if>
@@ -203,5 +202,4 @@
       <origin xyz="-0.217 -0.025 1.364" rpy="0 0 0"/>
     </xacro:sensor_d455> -->
-    <!-- ##################################################################3 -->
     <link name="realsense_back_gripper_mount">
       <collision>
@@ -218,11 +216,8 @@
       </visual>
     </link>
+    <!-- L515 Realsense Camera -->
     <xacro:sensor_l515 parent="coupling" use_nominal_extrinsics="$(arg use_nominal_extrinsics)" add_plug="$(arg add_plug)" use_mesh="$(arg use_mesh)">
-      <origin xyz="0.0 0.046 0.06" rpy="${pi} -${0.5 * pi} ${0.5 * pi}"/>
+      <origin xyz="0.0 0.046 0.1165" rpy="${pi} -${0.5 * pi} ${0.5 * pi}"/>
     </xacro:sensor_l515>
-    <!-- ####################################################################### -->
-    <!-- <xacro:sensor_l515 parent="coupling" use_nominal_extrinsics="$(arg use_nominal_extrinsics)" add_plug="$(arg add_plug)" use_mesh="$(arg use_mesh)">
-      <origin xyz="0.0 0.046 0.0765" rpy="${pi} -${0.5 * pi} ${0.5 * pi}"/>
-    </xacro:sensor_l515> -->
     <!-- <link name="realsense_lower_mount">
       <collision>
@@ -238,5 +233,4 @@
         <origin xyz="0.03 0 -0.05" rpy="0 0 0" />
     </joint> -->
-    <!-- #######################################################################3 -->
     <joint name="realsense_back_gripper_mount_joint" type="fixed">
         <parent link="camera_link"/>

Commit message: collin committing for soofiyan

File: tahoma_description/urdf/tahoma.xacro (robot description, xacro)
@@ -187,5 +187,5 @@
         <child link="camera_base"/>
         <!-- Link is centered on the optical frames. Slight offset in Y direction to compensate -->
-        <origin xyz="-0.260 0 1.465" rpy="3.13764 3.12912 -3.12899" />
+        <origin xyz="-0.260 -0.012 1.465" rpy="3.13764 3.12912 -3.12899" />
       </joint>
     </xacro:if>

Commit message: adjusting camera transform and od transform

File: tahoma_description/urdf/tahoma.xacro (robot description, xacro)
@@ -187,5 +187,5 @@
         <child link="camera_base"/>
         <!-- Link is centered on the optical frames. Slight offset in Y direction to compensate -->
-        <origin xyz="-0.260 -0.012 1.465" rpy="3.13764 3.12912 -3.12899" />
+        <origin xyz="-0.260 -0.015 1.465" rpy="3.13764 3.12912 -3.12899" />
       </joint>
     </xacro:if>
@@ -217,6 +217,9 @@
     </link>
     <!-- L515 Realsense Camera -->
+    <!-- <xacro:sensor_l515 parent="coupling" use_nominal_extrinsics="$(arg use_nominal_extrinsics)" add_plug="$(arg add_plug)" use_mesh="$(arg use_mesh)">
+      <origin xyz="0.0 0.046 0.1165" rpy="${pi} -${0.5 * pi} ${0.5 * pi}"/>
+    </xacro:sensor_l515> -->
     <xacro:sensor_l515 parent="coupling" use_nominal_extrinsics="$(arg use_nominal_extrinsics)" add_plug="$(arg add_plug)" use_mesh="$(arg use_mesh)">
-      <origin xyz="0.0 0.046 0.1165" rpy="${pi} -${0.5 * pi} ${0.5 * pi}"/>
+      <origin xyz="0.0 0.046 0.0765" rpy="${pi} -${0.5 * pi} ${0.5 * pi}"/>
     </xacro:sensor_l515>
     <!-- <link name="realsense_lower_mount">

Commit message: collin committing leftover changes from py39 workspace

File: tahoma_description/urdf/tahoma.xacro (robot description, xacro)
@@ -221,4 +221,11 @@
       <origin xyz="0.0 0.046 0.06" rpy="${pi} -${0.5 * pi} ${0.5 * pi}"/>
     </xacro:sensor_l515>
+    <!-- <xacro:sensor_l515 parent="coupling" use_nominal_extrinsics="$(arg use_nominal_extrinsics)" add_plug="$(arg add_plug)" use_mesh="$(arg use_mesh)">
+      <origin xyz="0.0 0.046 0.1165" rpy="${pi} -${0.5 * pi} ${0.5 * pi}"/>
+    </xacro:sensor_l515> -->
+    <!-- ####################################################################### -->
+    <!-- <xacro:sensor_l515 parent="coupling" use_nominal_extrinsics="$(arg use_nominal_extrinsics)" add_plug="$(arg add_plug)" use_mesh="$(arg use_mesh)">
+      <origin xyz="0.0 0.046 0.0765" rpy="${pi} -${0.5 * pi} ${0.5 * pi}"/>
+    </xacro:sensor_l515> -->
     <!-- <link name="realsense_lower_mount">
       <collision>
@@ -236,8 +243,10 @@
     <!-- #######################################################################3 -->
     <joint name="realsense_back_gripper_mount_joint" type="fixed">
+    <!-- #######################################################################3 -->
+    <!-- <joint name="realsense_back_gripper_mount_joint" type="fixed">
         <parent link="camera_link"/>
         <child link="realsense_back_gripper_mount"/>
         <origin xyz="-0.018 0.010227 -0.036" rpy="0 0 ${-0.5 * pi}" />
-    </joint>
+    </joint> -->
     <xacro:if value="${realsense}">
       <xacro:sensor_l515 name="camera_lower_right" parent="camera_lower_right_mount" use_nominal_extrinsics="${use_nominal_camera_extrinsics}">

Commit message: collin committing leftover changes from py39 workspace

File: tahoma_description/urdf/tahoma.xacro (robot description, xacro)
@@ -202,5 +202,6 @@
       <origin xyz="-0.217 -0.025 1.364" rpy="0 0 0"/>
     </xacro:sensor_d455> -->
-    <link name="realsense_back_gripper_mount">
+    <!-- ##################################################################3 -->
+    <!-- <link name="realsense_back_gripper_mount">
       <collision>
         <origin xyz="0.010227 -0.005 0.035" rpy="0 0 0"/>
@@ -215,12 +216,13 @@
         </geometry>
       </visual>
-    </link>
+    </link> -->
     <!-- L515 Realsense Camera -->
     <!-- <xacro:sensor_l515 parent="coupling" use_nominal_extrinsics="$(arg use_nominal_extrinsics)" add_plug="$(arg add_plug)" use_mesh="$(arg use_mesh)">
       <origin xyz="0.0 0.046 0.1165" rpy="${pi} -${0.5 * pi} ${0.5 * pi}"/>
     </xacro:sensor_l515> -->
-    <xacro:sensor_l515 parent="coupling" use_nominal_extrinsics="$(arg use_nominal_extrinsics)" add_plug="$(arg add_plug)" use_mesh="$(arg use_mesh)">
+    <!-- ####################################################################### -->
+    <!-- <xacro:sensor_l515 parent="coupling" use_nominal_extrinsics="$(arg use_nominal_extrinsics)" add_plug="$(arg add_plug)" use_mesh="$(arg use_mesh)">
       <origin xyz="0.0 0.046 0.0765" rpy="${pi} -${0.5 * pi} ${0.5 * pi}"/>
-    </xacro:sensor_l515>
+    </xacro:sensor_l515> -->
     <!-- <link name="realsense_lower_mount">
       <collision>
@@ -236,9 +238,10 @@
         <origin xyz="0.03 0 -0.05" rpy="0 0 0" />
     </joint> -->
-    <joint name="realsense_back_gripper_mount_joint" type="fixed">
+    <!-- #######################################################################3 -->
+    <!-- <joint name="realsense_back_gripper_mount_joint" type="fixed">
         <parent link="camera_link"/>
         <child link="realsense_back_gripper_mount"/>
         <origin xyz="-0.018 0.010227 -0.036" rpy="0 0 ${-0.5 * pi}" />
-    </joint>
+    </joint> -->
     <xacro:if value="${realsense}">
       <xacro:sensor_l515 name="camera_lower_right" parent="camera_lower_right_mount" use_nominal_extrinsics="${use_nominal_camera_extrinsics}">

Commit message: collin committing leftover changes from py39 workspace

File: tahoma_description/urdf/tahoma.xacro (robot description, xacro)
@@ -187,5 +187,5 @@
         <child link="camera_base"/>
         <!-- Link is centered on the optical frames. Slight offset in Y direction to compensate -->
-        <origin xyz="-0.260 0.0 1.465" rpy="3.13764 3.12912 -3.12899" />
+        <origin xyz="-0.260 -0.015 1.465" rpy="3.13764 3.12912 -3.12899" />
       </joint>
     </xacro:if>
@@ -203,5 +203,5 @@
     </xacro:sensor_d455> -->
     <!-- ##################################################################3 -->
-    <link name="realsense_back_gripper_mount">
+    <!-- <link name="realsense_back_gripper_mount">
       <collision>
         <origin xyz="0.010227 -0.005 0.035" rpy="0 0 0"/>
@@ -216,8 +216,13 @@
         </geometry>
       </visual>
-    </link>
-    <xacro:sensor_l515 parent="coupling" use_nominal_extrinsics="$(arg use_nominal_extrinsics)" add_plug="$(arg add_plug)" use_mesh="$(arg use_mesh)">
-      <origin xyz="0.0 0.046 0.06" rpy="${pi} -${0.5 * pi} ${0.5 * pi}"/>
-    </xacro:sensor_l515>
+    </link> -->
+    <!-- L515 Realsense Camera -->
+    <!-- <xacro:sensor_l515 parent="coupling" use_nominal_extrinsics="$(arg use_nominal_extrinsics)" add_plug="$(arg add_plug)" use_mesh="$(arg use_mesh)">
+      <origin xyz="0.0 0.046 0.1165" rpy="${pi} -${0.5 * pi} ${0.5 * pi}"/>
+    </xacro:sensor_l515> -->
+    <!-- ####################################################################### -->
+    <!-- <xacro:sensor_l515 parent="coupling" use_nominal_extrinsics="$(arg use_nominal_extrinsics)" add_plug="$(arg add_plug)" use_mesh="$(arg use_mesh)">
+      <origin xyz="0.0 0.046 0.0765" rpy="${pi} -${0.5 * pi} ${0.5 * pi}"/>
+    </xacro:sensor_l515> -->
     <!-- <link name="realsense_lower_mount">
       <collision>
@@ -234,9 +239,9 @@
     </joint> -->
     <!-- #######################################################################3 -->
-    <joint name="realsense_back_gripper_mount_joint" type="fixed">
+    <!-- <joint name="realsense_back_gripper_mount_joint" type="fixed">
         <parent link="camera_link"/>
         <child link="realsense_back_gripper_mount"/>
         <origin xyz="-0.018 0.010227 -0.036" rpy="0 0 ${-0.5 * pi}" />
-    </joint>
+    </joint> -->
     <xacro:if value="${realsense}">
       <xacro:sensor_l515 name="camera_lower_right" parent="camera_lower_right_mount" use_nominal_extrinsics="${use_nominal_camera_extrinsics}">

Commit message: working on impedance control

File: tahoma_description/urdf/tahoma.xacro (robot description, xacro)
@@ -182,5 +182,5 @@
         </geometry>
       </visual>
-    </link>
+    </link> -->
     <xacro:if value="${realsense}">
       <xacro:sensor_l515 name="camera_lower_right" parent="camera_lower_right_mount" use_nominal_extrinsics="${use_nominal_camera_extrinsics}">

Commit message: working on impedance control

File: tahoma_description/urdf/tahoma.xacro (robot description, xacro)
@@ -203,5 +203,6 @@
       <origin xyz="-0.217 -0.025 1.364" rpy="0 0 0"/>
     </xacro:sensor_d455> -->
-    <link name="realsense_back_gripper_mount">
+    <!-- ##################################################################3 -->
+    <!-- <link name="realsense_back_gripper_mount">
       <collision>
         <origin xyz="0.010227 -0.005 0.035" rpy="0 0 0"/>
@@ -216,9 +217,13 @@
         </geometry>
       </visual>
-    </link>
+    </link> -->
     <!-- L515 Realsense Camera -->
-    <xacro:sensor_l515 parent="coupling" use_nominal_extrinsics="$(arg use_nominal_extrinsics)" add_plug="$(arg add_plug)" use_mesh="$(arg use_mesh)">
+    <!-- <xacro:sensor_l515 parent="coupling" use_nominal_extrinsics="$(arg use_nominal_extrinsics)" add_plug="$(arg add_plug)" use_mesh="$(arg use_mesh)">
       <origin xyz="0.0 0.046 0.1165" rpy="${pi} -${0.5 * pi} ${0.5 * pi}"/>
-    </xacro:sensor_l515>
+    </xacro:sensor_l515> -->
+    <!-- ####################################################################### -->
+    <!-- <xacro:sensor_l515 parent="coupling" use_nominal_extrinsics="$(arg use_nominal_extrinsics)" add_plug="$(arg add_plug)" use_mesh="$(arg use_mesh)">
+      <origin xyz="0.0 0.046 0.0765" rpy="${pi} -${0.5 * pi} ${0.5 * pi}"/>
+    </xacro:sensor_l515> -->
     <!-- <link name="realsense_lower_mount">
       <collision>
@@ -234,9 +239,10 @@
         <origin xyz="0.03 0 -0.05" rpy="0 0 0" />
     </joint> -->
-    <joint name="realsense_back_gripper_mount_joint" type="fixed">
+    <!-- #######################################################################3 -->
+    <!-- <joint name="realsense_back_gripper_mount_joint" type="fixed">
         <parent link="camera_link"/>
         <child link="realsense_back_gripper_mount"/>
         <origin xyz="-0.018 0.010227 -0.036" rpy="0 0 ${-0.5 * pi}" />
-    </joint>
+    </joint> -->
     <xacro:if value="${realsense}">
       <xacro:sensor_l515 name="camera_lower_right" parent="camera_lower_right_mount" use_nominal_extrinsics="${use_nominal_camera_extrinsics}">

Commit message: working on impedance control

File: tahoma_description/urdf/tahoma.xacro (robot description, xacro)
@@ -182,5 +182,5 @@
         </geometry>
       </visual>
-    </link>
+    </link> -->
     <xacro:if value="${realsense}">
       <xacro:sensor_l515 name="camera_lower_right" parent="camera_lower_right_mount" use_nominal_extrinsics="${use_nominal_camera_extrinsics}">
@@ -210,5 +210,5 @@
         <child link="realsense_back_gripper_mount"/>
         <origin xyz="-0.018 0.010227 -0.036" rpy="0 0 ${-0.5 * pi}" />
-    </joint>
+    </joint> -->
   <link name="gripper_equilibrium_grasp"/>
   <joint name="gripper_base_link_gripper_equilibrium_grasp" type="fixed">

Commit message: got picks with impedance control. cleaned up code. tuned impedance control parameters
Co-authored-by: Collin Dang <collindang88@gmail.com>
Co-authored-by: Soofiyan Atar
Co-authored-by: Markus Grotz

File: tahoma_description/urdf/tahoma.xacro (robot description, xacro)
@@ -188,5 +188,5 @@
         <child link="camera_base"/>
         <!-- Link is centered on the optical frames. Slight offset in Y direction to compensate -->
-        <origin xyz="-0.260 0 1.465" rpy="3.13764 3.12912 -3.12899" />
+        <origin xyz="-0.260 -0.01 1.465" rpy="3.13764 3.12912 -3.12899" />
       </joint>
     </xacro:if>

Commit message: got picks with impedance control. cleaned up code. tuned impedance control parameters
Co-authored-by: Collin Dang <collindang88@gmail.com>
Co-authored-by: Soofiyan Atar
Co-authored-by: Markus Grotz

File: tahoma_description/urdf/tahoma.xacro (robot description, xacro)
@@ -187,5 +187,5 @@
         <child link="camera_base"/>
         <!-- Link is centered on the optical frames. Slight offset in Y direction to compensate -->
-        <origin xyz="-0.260 -0.015 1.465" rpy="3.13764 3.12912 -3.12899" />
+        <origin xyz="-0.260 -0.01 1.465" rpy="3.13764 3.12912 -3.12899" />
       </joint>
     </xacro:if>

Commit message: first commit

File: tahoma_description/urdf/tahoma.xacro (robot description, xacro)
@@ -187,5 +187,5 @@
         <child link="camera_base"/>
         <!-- Link is centered on the optical frames. Slight offset in Y direction to compensate -->
-        <origin xyz="-0.260 -0.015 1.465" rpy="3.13764 3.12912 -3.12899" />
+        <origin xyz="-0.260 0.0 1.465" rpy="3.13764 3.12912 -3.12899" />
       </joint>
     </xacro:if>
@@ -202,4 +202,5 @@
       <origin xyz="-0.217 -0.025 1.364" rpy="0 0 0"/>
     </xacro:sensor_d455> -->
+    <!-- ##################################################################3 -->
     <link name="realsense_back_gripper_mount">
       <collision>
@@ -216,10 +217,6 @@
       </visual>
     </link>
-    <!-- L515 Realsense Camera -->
-    <!-- <xacro:sensor_l515 parent="coupling" use_nominal_extrinsics="$(arg use_nominal_extrinsics)" add_plug="$(arg add_plug)" use_mesh="$(arg use_mesh)">
-      <origin xyz="0.0 0.046 0.1165" rpy="${pi} -${0.5 * pi} ${0.5 * pi}"/>
-    </xacro:sensor_l515> -->
     <xacro:sensor_l515 parent="coupling" use_nominal_extrinsics="$(arg use_nominal_extrinsics)" add_plug="$(arg add_plug)" use_mesh="$(arg use_mesh)">
-      <origin xyz="0.0 0.046 0.0765" rpy="${pi} -${0.5 * pi} ${0.5 * pi}"/>
+      <origin xyz="0.0 0.046 0.06" rpy="${pi} -${0.5 * pi} ${0.5 * pi}"/>
     </xacro:sensor_l515>
     <!-- <link name="realsense_lower_mount">
@@ -236,4 +233,5 @@
         <origin xyz="0.03 0 -0.05" rpy="0 0 0" />
     </joint> -->
+    <!-- #######################################################################3 -->
     <joint name="realsense_back_gripper_mount_joint" type="fixed">
         <parent link="camera_link"/>

Commit message: first commit

File: tahoma_description/urdf/tahoma.xacro (robot description, xacro)
@@ -188,5 +188,5 @@
         <child link="camera_base"/>
         <!-- Link is centered on the optical frames. Slight offset in Y direction to compensate -->
-        <origin xyz="-0.260 0 1.465" rpy="3.13764 3.12912 -3.12899" />
+        <origin xyz="-0.260 0.0 1.465" rpy="3.13764 3.12912 -3.12899" />
       </joint>
     </xacro:if>
@@ -203,4 +203,5 @@
       <origin xyz="-0.217 -0.025 1.364" rpy="0 0 0"/>
     </xacro:sensor_d455> -->
+    <!-- ##################################################################3 -->
     <link name="realsense_back_gripper_mount">
       <collision>
@@ -234,4 +235,5 @@
         <origin xyz="0.03 0 -0.05" rpy="0 0 0" />
     </joint> -->
+    <!-- #######################################################################3 -->
     <joint name="realsense_back_gripper_mount_joint" type="fixed">
         <parent link="camera_link"/>

Commit message: Adding changes doenfor increasing the speed of the arm adn also adding new retry mechanism with human input

File: tahoma_description/urdf/tahoma.xacro (robot description, xacro)
@@ -187,5 +187,5 @@
         <child link="camera_base"/>
         <!-- Link is centered on the optical frames. Slight offset in Y direction to compensate -->
-        <origin xyz="-0.260 0 1.465" rpy="3.13764 3.12912 -3.12899" />
+        <origin xyz="-0.260 0.0 1.465" rpy="3.13764 3.12912 -3.12899" />
       </joint>
     </xacro:if>
@@ -202,4 +202,5 @@
       <origin xyz="-0.217 -0.025 1.364" rpy="0 0 0"/>
     </xacro:sensor_d455> -->
+    <!-- ##################################################################3 -->
     <link name="realsense_back_gripper_mount">
       <collision>
@@ -218,5 +219,5 @@
     <!-- L515 Realsense Camera -->
     <xacro:sensor_l515 parent="coupling" use_nominal_extrinsics="$(arg use_nominal_extrinsics)" add_plug="$(arg add_plug)" use_mesh="$(arg use_mesh)">
-      <origin xyz="0.0 0.046 0.1165" rpy="${pi} -${0.5 * pi} ${0.5 * pi}"/>
+      <origin xyz="0.0 0.046 0.06" rpy="${pi} -${0.5 * pi} ${0.5 * pi}"/>
     </xacro:sensor_l515>
     <!-- <link name="realsense_lower_mount">
@@ -233,4 +234,5 @@
         <origin xyz="0.03 0 -0.05" rpy="0 0 0" />
     </joint> -->
+    <!-- #######################################################################3 -->
     <joint name="realsense_back_gripper_mount_joint" type="fixed">
         <parent link="camera_link"/>

Commit message: Soofiyan updates from other workspace

File: tahoma_description/urdf/tahoma.xacro (robot description, xacro)
@@ -187,5 +187,5 @@
         <child link="camera_base"/>
         <!-- Link is centered on the optical frames. Slight offset in Y direction to compensate -->
-        <origin xyz="-0.260 0.0 1.465" rpy="3.13764 3.12912 -3.12899" />
+        <origin xyz="-0.2426 -0.0264 1.4078" rpy="3.14 3.14 -3.14" />
       </joint>
     </xacro:if>

Commit message: Soofiyan updates from other workspace

File: tahoma_description/urdf/tahoma.xacro (robot description, xacro)
@@ -188,5 +188,5 @@
         <child link="camera_base"/>
         <!-- Link is centered on the optical frames. Slight offset in Y direction to compensate -->
-        <origin xyz="-0.260 0.0 1.465" rpy="3.13764 3.12912 -3.12899" />
+        <origin xyz="-0.2426 -0.0264 1.4078" rpy="3.14 3.14 -3.14" />
       </joint>
     </xacro:if>

Commit message: Integrating calibration method for the bins in pixel coordinate system and adding changes for the manipulation contraints for better manipulability

File: tahoma_description/urdf/tahoma.xacro (robot description, xacro)
@@ -187,5 +187,6 @@
         <child link="camera_base"/>
         <!-- Link is centered on the optical frames. Slight offset in Y direction to compensate -->
-        <origin xyz="-0.260 0.0 1.465" rpy="3.13764 3.12912 -3.12899" />
+        <origin xyz="-0.256 -0.0277 1.4245" rpy="3.14 3.14 -3.14" />
+        <!-- <origin xyz="-0.2426 -0.0277 1.4078" rpy="3.14 3.14 -3.14" /> -->
       </joint>
     </xacro:if>

Commit message: Integrating calibration method for the bins in pixel coordinate system and adding changes for the manipulation contraints for better manipulability

File: tahoma_description/urdf/tahoma.xacro (robot description, xacro)
@@ -187,5 +187,6 @@
         <child link="camera_base"/>
         <!-- Link is centered on the optical frames. Slight offset in Y direction to compensate -->
-        <origin xyz="-0.260 -0.015 1.465" rpy="3.13764 3.12912 -3.12899" />
+        <origin xyz="-0.256 -0.0277 1.4245" rpy="3.14 3.14 -3.14" />
+        <!-- <origin xyz="-0.2426 -0.0277 1.4078" rpy="3.14 3.14 -3.14" /> -->
       </joint>
     </xacro:if>
@@ -203,5 +204,5 @@
     </xacro:sensor_d455> -->
     <!-- ##################################################################3 -->
-    <!-- <link name="realsense_back_gripper_mount">
+    <link name="realsense_back_gripper_mount">
       <collision>
         <origin xyz="0.010227 -0.005 0.035" rpy="0 0 0"/>
@@ -216,9 +217,8 @@
         </geometry>
       </visual>
-    </link> -->
-    <!-- L515 Realsense Camera -->
-    <!-- <xacro:sensor_l515 parent="coupling" use_nominal_extrinsics="$(arg use_nominal_extrinsics)" add_plug="$(arg add_plug)" use_mesh="$(arg use_mesh)">
-      <origin xyz="0.0 0.046 0.1165" rpy="${pi} -${0.5 * pi} ${0.5 * pi}"/>
-    </xacro:sensor_l515> -->
+    </link>
+    <xacro:sensor_l515 parent="coupling" use_nominal_extrinsics="$(arg use_nominal_extrinsics)" add_plug="$(arg add_plug)" use_mesh="$(arg use_mesh)">
+      <origin xyz="0.0 0.046 0.06" rpy="${pi} -${0.5 * pi} ${0.5 * pi}"/>
+    </xacro:sensor_l515>
     <!-- ####################################################################### -->
     <!-- <xacro:sensor_l515 parent="coupling" use_nominal_extrinsics="$(arg use_nominal_extrinsics)" add_plug="$(arg add_plug)" use_mesh="$(arg use_mesh)">
@@ -239,9 +239,9 @@
     </joint> -->
     <!-- #######################################################################3 -->
-    <!-- <joint name="realsense_back_gripper_mount_joint" type="fixed">
+    <joint name="realsense_back_gripper_mount_joint" type="fixed">
         <parent link="camera_link"/>
         <child link="realsense_back_gripper_mount"/>
         <origin xyz="-0.018 0.010227 -0.036" rpy="0 0 ${-0.5 * pi}" />
-    </joint> -->
+    </joint>
     <xacro:if value="${realsense}">
       <xacro:sensor_l515 name="camera_lower_right" parent="camera_lower_right_mount" use_nominal_extrinsics="${use_nominal_camera_extrinsics}">
