Commit message: Adding changes to the urdf of the pod to accomodate different pod faces and different bin depths. Also incorporating changes for the manual calibration for different pods.

File: tahoma_description/urdf/tahoma.xacro (robot description, xacro)
@@ -187,5 +187,5 @@
         <child link="camera_base"/>
         <!-- Link is centered on the optical frames. Slight offset in Y direction to compensate -->
-        <origin xyz="-0.256 -0.0277 1.4245" rpy="3.14 3.14 -3.14" />
+        <origin xyz="-0.20750794 -0.01749962  1.40753882" rpy="3.14 3.14 -3.14" />
         <!-- <origin xyz="-0.2426 -0.0277 1.4078" rpy="3.14 3.14 -3.14" /> -->
       </joint>

Commit message: Added files to open/close gripper independently. Calibrated vacuum sensor setting. 450 seems to be a happy medium.

File: tahoma_description/urdf/tahoma.xacro (robot description, xacro)
@@ -187,5 +187,5 @@
         <child link="camera_base"/>
         <!-- Link is centered on the optical frames. Slight offset in Y direction to compensate -->
-        <origin xyz="-0.2426 -0.0264 1.4078" rpy="3.14 3.14 -3.14" />
+        <origin xyz="-0.25676 -0.02 1.4078" rpy="3.14 3.14 -3.14" />
       </joint>
     </xacro:if>

Commit message: Added files to open/close gripper independently. Calibrated vacuum sensor setting. 450 seems to be a happy medium.

File: tahoma_description/urdf/tahoma.xacro (robot description, xacro)
@@ -188,5 +188,5 @@
         <child link="camera_base"/>
         <!-- Link is centered on the optical frames. Slight offset in Y direction to compensate -->
-        <origin xyz="-0.2426 -0.0264 1.4078" rpy="3.14 3.14 -3.14" />
+        <origin xyz="-0.25676 -0.02 1.4078" rpy="3.14 3.14 -3.14" />
       </joint>
     </xacro:if>

Commit message: Fix xacro bug introduced in rebase

File: tahoma_description/urdf/tahoma.xacro (robot description, xacro)
@@ -244,29 +244,8 @@
     <!-- #######################################################################3 -->
     <joint name="realsense_back_gripper_mount_joint" type="fixed">
-    <!-- #######################################################################3 -->
-    <!-- <joint name="realsense_back_gripper_mount_joint" type="fixed">
         <parent link="camera_link"/>
         <child link="realsense_back_gripper_mount"/>
         <origin xyz="-0.018 0.010227 -0.036" rpy="0 0 ${-0.5 * pi}" />
-    </joint> -->
-    <xacro:if value="${realsense}">
-      <xacro:sensor_l515 name="camera_lower_right" parent="camera_lower_right_mount" use_nominal_extrinsics="${use_nominal_camera_extrinsics}">
-        <origin xyz="0 0 0" rpy="0 0 0"/>
-      </xacro:sensor_l515>
-      <xacro:sensor_l515 name="camera_lower_left" parent="camera_lower_left_mount" use_nominal_extrinsics="${use_nominal_camera_extrinsics}">
-        <origin xyz="0 0 0" rpy="0 0 0"/>
-      </xacro:sensor_l515>
-      <xacro:sensor_l515 name="camera_upper" parent="cantilever_camera_upper_mount" use_nominal_extrinsics="${use_nominal_camera_extrinsics}">
-        <origin xyz="0 0 0" rpy="0 0 0"/>
-      </xacro:sensor_l515>
-       <!-- Upper cameras -->
-      <xacro:sensor_l515 name="camera_upper_right" parent="camera_upper_right_mount" use_nominal_extrinsics="${use_nominal_camera_extrinsics}">
-        <origin xyz="0 0 0" rpy="0 0 0"/>
-      </xacro:sensor_l515>
-      <xacro:sensor_l515 name="camera_upper_left" parent="camera_upper_left_mount" use_nominal_extrinsics="${use_nominal_camera_extrinsics}">
-        <origin xyz="0 0 0" rpy="0 0 0"/>
-      </xacro:sensor_l515>
-    </xacro:if>
-  </xacro:macro>
+    </joint>
   <link name="gripper_equilibrium_grasp"/>
   <joint name="gripper_base_link_gripper_equilibrium_grasp" type="fixed">

Commit message: Basic fixes and dead code removal from robot xacro
Motion planning not working with this new model yet due to out of date SRDF

File: tahoma_description/urdf/tahoma.xacro (robot description, xacro)
@@ -5,4 +5,5 @@
   <!-- <xacro:include filename="$(find robotiq_2f_85_gripper_visualization)/urdf/robotiq_arg2f_85_macro.xacro"/> -->
   <xacro:include filename="$(find robotiq_epick_visualization)/urdf/robotiq_epick_model_macro.xacro" />
+  <xacro:include filename="$(find tahoma_description)/urdf/_l515.urdf.xacro" />
   <!-- <xacro:include filename="$(find realsense2_description)/urdf/_l515.urdf.xacro"/> -->
   <xacro:macro name="tahoma" params="
@@ -91,94 +92,4 @@
       <child link="coupling"/>
     </joint>
-    <link name="camera_lower_right_mount">
-      <collision>
-        <origin xyz="0 0 0" rpy="0 0 0"/>
-        <geometry>
-          <box size=".1 .15 .15"/>
-        </geometry>
-      </collision>
-    </link>
-    <link name="camera_lower_left_mount">
-      <collision>
-        <origin xyz="0 0 0" rpy="0 0 0"/>
-        <geometry>
-          <box size=".1 .15 .15"/>
-        </geometry>
-      </collision>
-    </link>
-    <!-- These are the planned ("nominal") mount placements. On the real system, these should
-     be overridden by calibrated transforms published separately -->
-    <xacro:if value="${camera_arrangement == 'manual' }">
-      <joint name="camera_beam_lower_camera_lower_left_mount_joint" type="fixed">
-        <parent link="camera_beam_lower"/>
-        <child link="camera_lower_left_mount"/>
-        <!-- Link is centered on the optical frames. Slight offset in Y direction to compensate -->
-        <origin xyz="0.02 ${-0.0215 + (camera_baseline / 2)} 0.14"
-                rpy="${pi / 2} ${radians(15)} ${-atan2((camera_baseline /2),camera_focal_depth)}"/>
-      </joint>
-      <joint name="camera_beam_lower_camera_lower_right_mount_joint" type="fixed">
-        <parent link="camera_beam_lower"/>
-        <child link="camera_lower_right_mount"/>
-        <origin xyz="0.02 ${0.0215 + (-camera_baseline / 2)} 0.14"
-                rpy="${pi / 2} ${radians(15)} ${atan2((camera_baseline /2),camera_focal_depth)}"/>
-      </joint>
-    </xacro:if>
-    <xacro:if value="${camera_arrangement == 'convergent' }">
-      <joint name="camera_beam_lower_camera_lower_left_mount_joint" type="fixed">
-        <parent link="camera_beam_lower"/>
-        <child link="camera_lower_left_mount"/>
-        <!-- Link is centered on the optical frames. Slight offset in Y direction to compensate -->
-        <origin xyz="0 ${-0.0215 + -camera_baseline / 2} 0.09"
-                rpy="${pi / 2} 0 ${-atan2((camera_baseline /2),camera_focal_depth)}"/>
-      </joint>
-      <joint name="camera_beam_lower_camera_lower_right_mount_joint" type="fixed">
-        <parent link="camera_beam_lower"/>
-        <child link="camera_lower_right_mount"/>
-        <origin xyz="0 ${-0.0215 + -camera_baseline / 2} 0.09"
-                rpy="${pi / 2} 0 ${atan2((camera_baseline /2),camera_focal_depth)}"/>
-      </joint>
-    </xacro:if>
-    <xacro:if value="${camera_arrangement == 'convergent_tilted' }">
-      <joint name="camera_beam_lower_camera_lower_left_mount_joint" type="fixed">
-        <parent link="camera_beam_lower"/>
-        <child link="camera_lower_left_mount"/>
-        <!-- Link is centered on the optical frames. Slight offset in Y direction to compensate -->
-        <origin xyz="-0.00 ${-0.0215 + (camera_baseline / 2)} 0.09"
-                rpy="${pi / 2} ${radians(15)} ${-atan2((camera_baseline /2),camera_focal_depth)}"/>
-      </joint>
-      <joint name="camera_beam_lower_camera_lower_right_mount_joint" type="fixed">
-        <parent link="camera_beam_lower"/>
-        <child link="camera_lower_right_mount"/>
-        <origin xyz="-0.00 ${0.0215 + (-camera_baseline / 2)} 0.09"
-                rpy="${pi / 2} ${radians(15)} ${atan2((camera_baseline /2),camera_focal_depth)}"/>
-      </joint>
-    </xacro:if>
-    <!-- Upper cameras -->
-    <!-- Link is centered on the optical frames. Slight offset in Y direction to compensate -->
-    <!-- Z=1.10 for on top of the top beam -->
-    <!-- Z=0.80 for underneath the top beam -->
-    <!-- Disabled until we know about manipulability in upper bins
-    <link name="camera_upper_right_mount"/>
-    <link name="camera_upper_left_mount"/>
-    <joint name="stand_upright_camera_upper_left_mount_joint" type="fixed">
-      <parent link="stand_upright"/>
-      <child link="camera_upper_left_mount"/>
-      <origin xyz="-.1 ${-0.0215 + (camera_baseline / 2)} 0.80"
-              rpy="${pi / 2} ${radians(15)} ${-atan2((camera_baseline /2),camera_focal_depth)}"/>
-    </joint>
-    <joint name="stand_upright_camera_upper_right_mount_joint" type="fixed">
-      <parent link="stand_upright"/>
-      <child link="camera_upper_right_mount"/>
-      <origin xyz="-.1 ${0.0215 + (-camera_baseline / 2)} 0.80"
-              rpy="${pi / 2} ${radians(15)} ${atan2((camera_baseline /2),camera_focal_depth)}"/>
-    </joint>
-    -->
-    <link name="cantilever_camera_upper_mount"/>
-    <joint name="cantilever_camera_upper_mount_joint" type="fixed">
-      <parent link="cantilever"/>
-      <child link="cantilever_camera_upper_mount"/>
-      <origin xyz=".02 0 0.37"
-              rpy="0 ${radians(15)} 0"/>
-    </joint>
     <xacro:if value="${azure_kinect}">
       <xacro:include filename="$(find tahoma_description)/urdf/azure_kinect.urdf.xacro"/>
@@ -191,17 +102,4 @@
       </joint>
     </xacro:if>
-    <xacro:arg name="use_nominal_extrinsics" default="false"/>
-    <xacro:arg name="add_plug" default="false" />
-    <xacro:arg name="use_mesh" default="true" />
-    <xacro:include filename="$(find tahoma_description)/urdf/_l515.urdf.xacro" />
-    <!-- D435 Realsense Camera -->
-    <!-- <xacro:sensor_d435 parent="base_link" use_nominal_extrinsics="$(arg use_nominal_extrinsics)" add_plug="$(arg add_plug)" use_mesh="$(arg use_mesh)">
-      <origin xyz="-0.217 0.013 1.354" rpy="0 0 0"/>
-    </xacro:sensor_d435> -->
-    <!-- D455 Realsense Camera -->
-    <!-- <xacro:sensor_d455 parent="base_link" use_nominal_extrinsics="$(arg use_nominal_extrinsics)">
-      <origin xyz="-0.217 -0.025 1.364" rpy="0 0 0"/>
-    </xacro:sensor_d455> -->
-    <!-- ##################################################################3 -->
     <link name="realsense_back_gripper_mount">
       <collision>
@@ -219,30 +117,9 @@
     </link>
     <!-- L515 Realsense Camera -->
-    <xacro:sensor_l515 parent="coupling" use_nominal_extrinsics="$(arg use_nominal_extrinsics)" add_plug="$(arg add_plug)" use_mesh="$(arg use_mesh)">
+    <xacro:sensor_l515 parent="realsense_back_gripper_mount" use_nominal_extrinsics="${use_nominal_camera_extrinsics}" add_plug="false" use_mesh="true">
       <origin xyz="0.0 0.046 0.06" rpy="${pi} -${0.5 * pi} ${0.5 * pi}"/>
     </xacro:sensor_l515>
-    <!-- <xacro:sensor_l515 parent="coupling" use_nominal_extrinsics="$(arg use_nominal_extrinsics)" add_plug="$(arg add_plug)" use_mesh="$(arg use_mesh)">
-      <origin xyz="0.0 0.046 0.1165" rpy="${pi} -${0.5 * pi} ${0.5 * pi}"/>
-    </xacro:sensor_l515> -->
-    <!-- ####################################################################### -->
-    <!-- <xacro:sensor_l515 parent="coupling" use_nominal_extrinsics="$(arg use_nominal_extrinsics)" add_plug="$(arg add_plug)" use_mesh="$(arg use_mesh)">
-      <origin xyz="0.0 0.046 0.0765" rpy="${pi} -${0.5 * pi} ${0.5 * pi}"/>
-    </xacro:sensor_l515> -->
-    <!-- <link name="realsense_lower_mount">
-      <collision>
-        <origin xyz="0 0 0" rpy="0 0 0"/>
-        <geometry>
-          <box size="0.06 0.1 0.06"/>
-        </geometry>
-      </collision>
-    </link>
-    <joint name="realsense_mount_joint" type="fixed">
-        <parent link="camera_bottom_screw_frame"/>
-        <child link="realsense_lower_mount"/>
-        <origin xyz="0.03 0 -0.05" rpy="0 0 0" />
-    </joint> -->
-    <!-- #######################################################################3 -->
     <joint name="realsense_back_gripper_mount_joint" type="fixed">
-        <parent link="camera_link"/>
+        <parent link="coupling"/>
         <child link="realsense_back_gripper_mount"/>
         <origin xyz="-0.018 0.010227 -0.036" rpy="0 0 ${-0.5 * pi}" />
@@ -255,3 +132,4 @@
               rpy="0 0 0"/>
   </joint>
+</xacro:macro>
 </robot>

Commit message: 1. Added changes for multiple suction outlets for vaccum gripper 2. Added pod models which were created by sanjar. 3. Added pod calibration script for both the pods. 4. Added modified version of reachability code originally implemented by hitesh. 4. Modified collision scene for arm by adding a constraint space instead of only pod model. 5. Modified the 3d point calibration for multiple files Co-authored-by: Nindroz <mantha.hitesh@gmail.com> Co-authored-by: Paolo Torrado <paolo.a.torrado@gmail.com> Co-authored-by: Sanjar Normuradov <snnormuradov@gmail.com>

File: tahoma_description/urdf/tahoma.xacro (robot description, xacro)
@@ -188,5 +188,6 @@
         <child link="camera_base"/>
         <!-- Link is centered on the optical frames. Slight offset in Y direction to compensate -->
-        <origin xyz="-0.25676 -0.02 1.4078" rpy="3.14 3.14 -3.14" />
+        <origin xyz="-0.20750794 -0.01815336  1.40753882" rpy="3.14 3.14 -3.14" />
+        <!-- <origin xyz="-0.2426 -0.0277 1.4078" rpy="3.14 3.14 -3.14" /> -->
       </joint>
     </xacro:if>

Commit message: Add camera and increase pod collision box

File: tahoma_description/urdf/tahoma.xacro (robot description, xacro)
@@ -5,4 +5,5 @@
   <!-- <xacro:include filename="$(find robotiq_2f_85_gripper_visualization)/urdf/robotiq_arg2f_85_macro.xacro"/> -->
   <xacro:include filename="$(find robotiq_epick_visualization)/urdf/robotiq_epick_model_macro.xacro" />
+  <xacro:include filename="$(find tahoma_description)/urdf/_l515.urdf.xacro" />
   <!-- <xacro:include filename="$(find realsense2_description)/urdf/_l515.urdf.xacro"/> -->
   <xacro:macro name="tahoma" params="
@@ -58,5 +59,5 @@
       </visual>
      <visual>
-        <origin xyz="0.0335 0 0.006" rpy="0 0 0"/>
+        <origin xyz="0.0335 0 0.0" rpy="0 0 0"/>
         <geometry>
           <mesh filename="package://robotiq_2f_85_gripper_visualization/meshes/visual/connector_cover.stl"/>
@@ -82,10 +83,10 @@
     </link>
     <joint name="coupling_link_gripper_robotiq_arg2f_base_link_joint" type="fixed">
-      <origin xyz="0 0 0.017" rpy="0 0 0"/>
+      <origin xyz="0 0 0.055" rpy="0 0 0"/>
       <parent link="coupling"/>
       <child link="gripper_base_link"/>
     </joint>
     <joint name="arm_tool0-coupling_joint" type="fixed">
-      <origin xyz="0 0 -0.003" rpy="0 0 ${1.5 * pi}"/>
+      <origin xyz="0 0 0" rpy="0 0 ${1.5 * pi}"/>
       <parent link="arm_tool0"/>
       <child link="coupling"/>
@@ -154,31 +155,4 @@
       </joint>
     </xacro:if>
-    <!-- Upper cameras -->
-    <!-- Link is centered on the optical frames. Slight offset in Y direction to compensate -->
-    <!-- Z=1.10 for on top of the top beam -->
-    <!-- Z=0.80 for underneath the top beam -->
-    <!-- Disabled until we know about manipulability in upper bins
-    <link name="camera_upper_right_mount"/>
-    <link name="camera_upper_left_mount"/>
-    <joint name="stand_upright_camera_upper_left_mount_joint" type="fixed">
-      <parent link="stand_upright"/>
-      <child link="camera_upper_left_mount"/>
-      <origin xyz="-.1 ${-0.0215 + (camera_baseline / 2)} 0.80"
-              rpy="${pi / 2} ${radians(15)} ${-atan2((camera_baseline /2),camera_focal_depth)}"/>
-    </joint>
-    <joint name="stand_upright_camera_upper_right_mount_joint" type="fixed">
-      <parent link="stand_upright"/>
-      <child link="camera_upper_right_mount"/>
-      <origin xyz="-.1 ${0.0215 + (-camera_baseline / 2)} 0.80"
-              rpy="${pi / 2} ${radians(15)} ${atan2((camera_baseline /2),camera_focal_depth)}"/>
-    </joint>
-    -->
-    <link name="camera_upper_mount"/>
-    <joint name="cantilever_camera_upper_mount_joint" type="fixed">
-      <parent link="cantilever"/>
-      <child link="camera_upper_mount"/>
-      <origin xyz=".02 0 0.37"
-              rpy="0 ${radians(15)} 0"/>
-    </joint>
     <xacro:if value="${azure_kinect}">
       <xacro:include filename="$(find tahoma_description)/urdf/azure_kinect.urdf.xacro"/>
@@ -187,26 +161,54 @@
         <child link="camera_base"/>
         <!-- Link is centered on the optical frames. Slight offset in Y direction to compensate -->
-        <origin xyz="-0.245645 ${0.000778815-.0125} 1.41034" rpy="3.13764 3.12912 -3.12899" />
-      </joint>
-    </xacro:if>
+        <origin xyz="-0.20750794 -0.01815336  1.40753882" rpy="3.14 3.14 -3.14" />
+        <!-- <origin xyz="-0.2426 -0.0277 1.4078" rpy="3.14 3.14 -3.14" /> -->
+      </joint>
+    </xacro:if>
+    <xacro:arg name="use_nominal_extrinsics" default="false"/>
+    <xacro:arg name="add_plug" default="false" />
+    <xacro:arg name="use_mesh" default="true" />
+    <xacro:include filename="$(find tahoma_description)/urdf/_l515.urdf.xacro" />
+    <link name="realsense_back_gripper_mount">
+      <collision>
+        <origin xyz="0.010227 -0.005 0.035" rpy="0 0 0"/>
+        <geometry>
+          <box size="0.04 0.02 0.08"/>
+        </geometry>
+      </collision>
+      <visual>
+        <origin xyz="0 0 0" rpy="0 0 0"/>
+        <geometry>
+          <mesh filename="package://tahoma_description/meshes/realsense/couple_l515_mount.obj"/>
+        </geometry>
+      </visual>
+    </link>
     <xacro:if value="${realsense}">
       <xacro:sensor_l515 name="camera_lower_right" parent="camera_lower_right_mount" use_nominal_extrinsics="${use_nominal_camera_extrinsics}">
         <origin xyz="0 0 0" rpy="0 0 0"/>
       </xacro:sensor_l515>
-      <xacro:sensor_l515 name="camera_lower_left" parent="camera_lower_left_mount" use_nominal_extrinsics="${use_nominal_camera_extrinsics}">
-        <origin xyz="0 0 0" rpy="0 0 0"/>
-      </xacro:sensor_l515>
-      <xacro:sensor_l515 name="camera_upper" parent="camera_upper_mount" use_nominal_extrinsics="${use_nominal_camera_extrinsics}">
-        <origin xyz="0 0 0" rpy="0 0 0"/>
-      </xacro:sensor_l515>
-       <!-- Upper cameras -->
-      <xacro:sensor_l515 name="camera_upper_right" parent="camera_upper_right_mount" use_nominal_extrinsics="${use_nominal_camera_extrinsics}">
-        <origin xyz="0 0 0" rpy="0 0 0"/>
-      </xacro:sensor_l515>
-      <xacro:sensor_l515 name="camera_upper_left" parent="camera_upper_left_mount" use_nominal_extrinsics="${use_nominal_camera_extrinsics}">
-        <origin xyz="0 0 0" rpy="0 0 0"/>
-      </xacro:sensor_l515>
-    </xacro:if>
-  </xacro:macro>
+    <link name="realsense_back_gripper_mount">
+      <collision>
+        <origin xyz="0.010227 -0.005 0.035" rpy="0 0 0"/>
+        <geometry>
+          <box size="0.04 0.02 0.08"/>
+        </geometry>
+      </collision>
+      <visual>
+        <origin xyz="0 0 0" rpy="0 0 0"/>
+        <geometry>
+          <mesh filename="package://tahoma_description/meshes/realsense/couple_l515_mount.obj"/>
+        </geometry>
+      </visual>
+    </link>
+    </xacro:if>
+    <!-- L515 Realsense Camera -->
+    <xacro:sensor_l515 parent="realsense_back_gripper_mount" use_nominal_extrinsics="${use_nominal_camera_extrinsics}" add_plug="false" use_mesh="true">
+      <origin xyz="0.0 0.046 0.06" rpy="${pi} -${0.5 * pi} ${0.5 * pi}"/>
+    </xacro:sensor_l515>
+    <joint name="realsense_back_gripper_mount_joint" type="fixed">
+        <parent link="coupling"/>
+        <child link="realsense_back_gripper_mount"/>
+        <origin xyz="-0.018 0.010227 -0.036" rpy="0 0 ${-0.5 * pi}" />
+    </joint>
   <link name="gripper_equilibrium_grasp"/>
   <joint name="gripper_base_link_gripper_equilibrium_grasp" type="fixed">
@@ -216,3 +218,4 @@
               rpy="0 0 0"/>
   </joint>
+</xacro:macro>
 </robot>

Commit message: Calibrated camera pose and gripper camera orientation with mount

File: tahoma_description/urdf/tahoma.xacro (robot description, xacro)
@@ -5,5 +5,4 @@
   <!-- <xacro:include filename="$(find robotiq_2f_85_gripper_visualization)/urdf/robotiq_arg2f_85_macro.xacro"/> -->
   <xacro:include filename="$(find robotiq_epick_visualization)/urdf/robotiq_epick_model_macro.xacro" />
-  <xacro:include filename="$(find tahoma_description)/urdf/_l515.urdf.xacro" />
   <!-- <xacro:include filename="$(find realsense2_description)/urdf/_l515.urdf.xacro"/> -->
   <xacro:macro name="tahoma" params="
@@ -161,5 +160,5 @@
         <child link="camera_base"/>
         <!-- Link is centered on the optical frames. Slight offset in Y direction to compensate -->
-        <origin xyz="-0.20750794 -0.01815336  1.40753882" rpy="3.14 3.14 -3.14" />
+        <origin xyz="-0.21 -0.01  1.375" rpy="0.0 -0.08 0.0" />
         <!-- <origin xyz="-0.2426 -0.0277 1.4078" rpy="3.14 3.14 -3.14" /> -->
       </joint>
@@ -183,33 +182,17 @@
       </visual>
     </link>
+    <xacro:sensor_l515 parent="coupling" use_nominal_extrinsics="$(arg use_nominal_extrinsics)" add_plug="$(arg add_plug)" use_mesh="$(arg use_mesh)">
+      <origin xyz="0.0 0.046 0.06" rpy="${pi} -${0.5 * pi} ${0.5 * pi}"/>
+    </xacro:sensor_l515>
+    <joint name="realsense_back_gripper_mount_joint" type="fixed">
+        <parent link="camera_link"/>
+        <child link="realsense_back_gripper_mount"/>
+        <origin xyz="-0.018 0.010227 -0.036" rpy="0 0 ${-0.5 * pi}" />
+    </joint>
     <xacro:if value="${realsense}">
       <xacro:sensor_l515 name="camera_lower_right" parent="camera_lower_right_mount" use_nominal_extrinsics="${use_nominal_camera_extrinsics}">
         <origin xyz="0 0 0" rpy="0 0 0"/>
       </xacro:sensor_l515>
-    <link name="realsense_back_gripper_mount">
-      <collision>
-        <origin xyz="0.010227 -0.005 0.035" rpy="0 0 0"/>
-        <geometry>
-          <box size="0.04 0.02 0.08"/>
-        </geometry>
-      </collision>
-      <visual>
-        <origin xyz="0 0 0" rpy="0 0 0"/>
-        <geometry>
-          <mesh filename="package://tahoma_description/meshes/realsense/couple_l515_mount.obj"/>
-        </geometry>
-      </visual>
-    </link>
-    </xacro:if>
-    <!-- L515 Realsense Camera -->
-    <xacro:sensor_l515 parent="realsense_back_gripper_mount" use_nominal_extrinsics="${use_nominal_camera_extrinsics}" add_plug="false" use_mesh="true">
-      <origin xyz="0.0 0.046 0.06" rpy="${pi} -${0.5 * pi} ${0.5 * pi}"/>
-    </xacro:sensor_l515>
-    <!-- #######################################################################3 -->
-    <joint name="realsense_back_gripper_mount_joint" type="fixed">
-        <parent link="coupling"/>
-        <child link="realsense_back_gripper_mount"/>
-        <origin xyz="-0.018 0.010227 -0.036" rpy="0 0 ${-0.5 * pi}" />
-    </joint>
+    </xacro:if>
   <link name="gripper_equilibrium_grasp"/>
   <joint name="gripper_base_link_gripper_equilibrium_grasp" type="fixed">
