Commit message: Calibrated camera pose and gripper camera orientation with mount

File: tahoma_description/urdf/tahoma.xacro (robot description, xacro)
@@ -5,5 +5,4 @@
   <!-- <xacro:include filename="$(find robotiq_2f_85_gripper_visualization)/urdf/robotiq_arg2f_85_macro.xacro"/> -->
   <xacro:include filename="$(find robotiq_epick_visualization)/urdf/robotiq_epick_model_macro.xacro" />
-  <xacro:include filename="$(find tahoma_description)/urdf/_l515.urdf.xacro" />
   <!-- <xacro:include filename="$(find realsense2_description)/urdf/_l515.urdf.xacro"/> -->
   <xacro:macro name="tahoma" params="
@@ -161,5 +160,5 @@
         <child link="camera_base"/>
         <!-- Link is centered on the optical frames. Slight offset in Y direction to compensate -->
-        <origin xyz="-0.20750794 -0.01815336  1.40753882" rpy="3.14 3.14 -3.14" />
+        <origin xyz="-0.21 -0.01  1.375" rpy="0.0 -0.08 0.0" />
         <!-- <origin xyz="-0.2426 -0.0277 1.4078" rpy="3.14 3.14 -3.14" /> -->
       </joint>
@@ -183,32 +182,17 @@
       </visual>
     </link>
-    <xacro:if value="${realsense}">
-      <xacro:sensor_l515 name="camera_lower_right" parent="camera_lower_right_mount" use_nominal_extrinsics="${use_nominal_camera_extrinsics}">
-        <origin xyz="0 0 0" rpy="0 0 0"/>
-      </xacro:sensor_l515>
-    <link name="realsense_back_gripper_mount">
-      <collision>
-        <origin xyz="0.010227 -0.005 0.035" rpy="0 0 0"/>
-        <geometry>
-          <box size="0.04 0.02 0.08"/>
-        </geometry>
-      </collision>
-      <visual>
-        <origin xyz="0 0 0" rpy="0 0 0"/>
-        <geometry>
-          <mesh filename="package://tahoma_description/meshes/realsense/couple_l515_mount.obj"/>
-        </geometry>
-      </visual>
-    </link>
-    </xacro:if>
-    <!-- L515 Realsense Camera -->
-    <xacro:sensor_l515 parent="realsense_back_gripper_mount" use_nominal_extrinsics="${use_nominal_camera_extrinsics}" add_plug="false" use_mesh="true">
+    <xacro:sensor_l515 parent="coupling" use_nominal_extrinsics="$(arg use_nominal_extrinsics)" add_plug="$(arg add_plug)" use_mesh="$(arg use_mesh)">
       <origin xyz="0.0 0.046 0.06" rpy="${pi} -${0.5 * pi} ${0.5 * pi}"/>
     </xacro:sensor_l515>
     <joint name="realsense_back_gripper_mount_joint" type="fixed">
-        <parent link="coupling"/>
+        <parent link="camera_link"/>
         <child link="realsense_back_gripper_mount"/>
         <origin xyz="-0.018 0.010227 -0.036" rpy="0 0 ${-0.5 * pi}" />
     </joint>
+    <xacro:if value="${realsense}">
+      <xacro:sensor_l515 name="camera_lower_right" parent="camera_lower_right_mount" use_nominal_extrinsics="${use_nominal_camera_extrinsics}">
+        <origin xyz="0 0 0" rpy="0 0 0"/>
+      </xacro:sensor_l515>
+    </xacro:if>
   <link name="gripper_equilibrium_grasp"/>
   <joint name="gripper_base_link_gripper_equilibrium_grasp" type="fixed">

Commit message: Tweak gripper camera collision geometry
Remove old realsense joints/links/frames

File: tahoma_description/urdf/tahoma.xacro (robot description, xacro)
@@ -5,7 +5,5 @@
   <!-- <xacro:include filename="$(find robotiq_2f_85_gripper_visualization)/urdf/robotiq_arg2f_85_macro.xacro"/> -->
   <xacro:include filename="$(find robotiq_epick_visualization)/urdf/robotiq_epick_model_macro.xacro" />
-  <!-- <xacro:include filename="$(find realsense2_description)/urdf/_l515.urdf.xacro"/> -->
   <xacro:macro name="tahoma" params="
-  realsense:=false
   azure_kinect:=true
   use_nominal_camera_extrinsics:=false
@@ -91,67 +89,4 @@
       <child link="coupling"/>
     </joint>
-    <link name="camera_lower_right_mount">
-      <collision>
-        <origin xyz="0 0 0" rpy="0 0 0"/>
-        <geometry>
-          <box size=".1 .15 .15"/>
-        </geometry>
-      </collision>
-    </link>
-    <link name="camera_lower_left_mount">
-      <collision>
-        <origin xyz="0 0 0" rpy="0 0 0"/>
-        <geometry>
-          <box size=".1 .15 .15"/>
-        </geometry>
-      </collision>
-    </link>
-    <!-- These are the planned ("nominal") mount placements. On the real system, these should
-     be overridden by calibrated transforms published separately -->
-    <xacro:if value="${camera_arrangement == 'manual' }">
-      <joint name="camera_beam_lower_camera_lower_left_mount_joint" type="fixed">
-        <parent link="camera_beam_lower"/>
-        <child link="camera_lower_left_mount"/>
-        <!-- Link is centered on the optical frames. Slight offset in Y direction to compensate -->
-        <origin xyz="0.02 ${-0.0215 + (camera_baseline / 2)} 0.14"
-                rpy="${pi / 2} ${radians(15)} ${-atan2((camera_baseline /2),camera_focal_depth)}"/>
-      </joint>
-      <joint name="camera_beam_lower_camera_lower_right_mount_joint" type="fixed">
-        <parent link="camera_beam_lower"/>
-        <child link="camera_lower_right_mount"/>
-        <origin xyz="0.02 ${0.0215 + (-camera_baseline / 2)} 0.14"
-                rpy="${pi / 2} ${radians(15)} ${atan2((camera_baseline /2),camera_focal_depth)}"/>
-      </joint>
-    </xacro:if>
-    <xacro:if value="${camera_arrangement == 'convergent' }">
-      <joint name="camera_beam_lower_camera_lower_left_mount_joint" type="fixed">
-        <parent link="camera_beam_lower"/>
-        <child link="camera_lower_left_mount"/>
-        <!-- Link is centered on the optical frames. Slight offset in Y direction to compensate -->
-        <origin xyz="0 ${-0.0215 + -camera_baseline / 2} 0.09"
-                rpy="${pi / 2} 0 ${-atan2((camera_baseline /2),camera_focal_depth)}"/>
-      </joint>
-      <joint name="camera_beam_lower_camera_lower_right_mount_joint" type="fixed">
-        <parent link="camera_beam_lower"/>
-        <child link="camera_lower_right_mount"/>
-        <origin xyz="0 ${-0.0215 + -camera_baseline / 2} 0.09"
-                rpy="${pi / 2} 0 ${atan2((camera_baseline /2),camera_focal_depth)}"/>
-      </joint>
-    </xacro:if>
-    <xacro:if value="${camera_arrangement == 'convergent_tilted' }">
-      <joint name="camera_beam_lower_camera_lower_left_mount_joint" type="fixed">
-        <parent link="camera_beam_lower"/>
-        <child link="camera_lower_left_mount"/>
-        <!-- Link is centered on the optical frames. Slight offset in Y direction to compensate -->
-        <origin xyz="-0.00 ${-0.0215 + (camera_baseline / 2)} 0.09"
-                rpy="${pi / 2} ${radians(15)} ${-atan2((camera_baseline /2),camera_focal_depth)}"/>
-      </joint>
-      <joint name="camera_beam_lower_camera_lower_right_mount_joint" type="fixed">
-        <parent link="camera_beam_lower"/>
-        <child link="camera_lower_right_mount"/>
-        <origin xyz="-0.00 ${0.0215 + (-camera_baseline / 2)} 0.09"
-                rpy="${pi / 2} ${radians(15)} ${atan2((camera_baseline /2),camera_focal_depth)}"/>
-      </joint>
-    </xacro:if>
     <xacro:if value="${azure_kinect}">
       <xacro:include filename="$(find tahoma_description)/urdf/azure_kinect.urdf.xacro"/>
@@ -168,38 +103,36 @@
     <xacro:arg name="use_mesh" default="true" />
     <xacro:include filename="$(find tahoma_description)/urdf/_l515.urdf.xacro" />
-    <link name="realsense_back_gripper_mount">
+    <link name="gripper_camera_mount">
       <collision>
         <origin xyz="0.010227 -0.005 0.035" rpy="0 0 0"/>
         <geometry>
-          <box size="0.04 0.02 0.08"/>
+          <box size="0.04 0.03 0.08"/>
         </geometry>
       </collision>
       <visual>
-        <origin xyz="0 0 0" rpy="0 0 0"/>
+        <origin xyz="0.010227 -0.005 0.035" rpy="0 0 0"/>
         <geometry>
-          <mesh filename="package://tahoma_description/meshes/realsense/couple_l515_mount.obj"/>
+          <box size="0.04 0.03 0.08"/>
         </geometry>
       </visual>
     </link>
-    <xacro:sensor_l515 parent="coupling" use_nominal_extrinsics="$(arg use_nominal_extrinsics)" add_plug="$(arg add_plug)" use_mesh="$(arg use_mesh)">
-      <origin xyz="0.0 0.046 0.06" rpy="${pi} -${0.5 * pi} ${0.5 * pi}"/>
-    </xacro:sensor_l515>
-    <joint name="realsense_back_gripper_mount_joint" type="fixed">
-        <parent link="camera_link"/>
-        <child link="realsense_back_gripper_mount"/>
-        <origin xyz="-0.018 0.010227 -0.036" rpy="0 0 ${-0.5 * pi}" />
+    <link name="gripper_camera" />
+    <joint name="gripper_camera_mount_gripper_camera_joint" type="fixed">
+        <parent link="gripper_camera_mount"/>
+        <child link="gripper_camera"/>
+        <origin xyz="-0.018 0.010227 -0.036" rpy="0 0 0" />
     </joint>
-    <xacro:if value="${realsense}">
-      <xacro:sensor_l515 name="camera_lower_right" parent="camera_lower_right_mount" use_nominal_extrinsics="${use_nominal_camera_extrinsics}">
-        <origin xyz="0 0 0" rpy="0 0 0"/>
-      </xacro:sensor_l515>
-    </xacro:if>
-  <link name="gripper_equilibrium_grasp"/>
-  <joint name="gripper_base_link_gripper_equilibrium_grasp" type="fixed">
-    <parent link="epick_end_effector"/>
-      <child link="gripper_equilibrium_grasp"/>
-      <origin xyz="0 0 0"
-              rpy="0 0 0"/>
-  </joint>
+    <joint name="gripprer_base_link_gripper_camera_mount_joint" type="fixed">
+        <parent link="gripper_base_link"/>
+        <child link="gripper_camera_mount"/>
+        <origin xyz="0.0 0.0 -0.036" rpy="${-0.5 * pi} 0 0" />
+    </joint>
+    <link name="gripper_equilibrium_grasp"/>
+    <joint name="gripper_base_link_gripper_equilibrium_grasp" type="fixed">
+      <parent link="epick_end_effector"/>
+        <child link="gripper_equilibrium_grasp"/>
+        <origin xyz="0 0 0"
+                rpy="0 0 0"/>
+    </joint>
 </xacro:macro>
 </robot>
