Commit message: Added begripa code

File: tahoma_description/urdf/tahoma.xacro (robot description, xacro)
@@ -42,4 +42,26 @@
       <child link="stand"/>
     </joint>
+    <link name="table">
+      <visual>
+        <origin xyz="0 0 0" rpy="0 0 0"/>
+        <geometry>
+          <box size="1.0 0.8 0.05"/>
+        </geometry>
+        <material name="table_color">
+          <color rgba="0.8 0.6 0.4 0.5"/>
+        </material>
+      </visual>
+      <collision>
+        <origin xyz="0 0 0" rpy="0 0 0"/>
+        <geometry>
+          <box size="1.0 0.8 0.05"/>
+        </geometry>
+      </collision>
+    </link>
+    <joint name="base_link_table_joint" type="fixed">
+      <parent link="base_link"/>
+      <child link="table"/>
+      <origin xyz="1.0 0.0 0.75" rpy="0 0 0"/>
+    </joint>
     <joint name="robot_plate_arm_base_link_joint" type="fixed">
       <parent link="robot_plate"/>
@@ -187,5 +209,5 @@
         <child link="camera_base"/>
         <!-- Link is centered on the optical frames. Slight offset in Y direction to compensate -->
-        <origin xyz="-0.20750794 -0.01749962  1.40753882" rpy="3.14 3.14 -3.14" />
+        <origin xyz="-0.20750794 -0.03749962  1.40753882" rpy="3.14 3.14 -3.14" />
         <!-- <origin xyz="-0.2426 -0.0277 1.4078" rpy="3.14 3.14 -3.14" /> -->
       </joint>
@@ -258,11 +280,11 @@
       </xacro:sensor_l515>
     </xacro:if>
+    <link name="gripper_equilibrium_grasp"/>
+    <joint name="gripper_base_link_gripper_equilibrium_grasp" type="fixed">
+      <parent link="epick_end_effector"/>
+        <child link="gripper_equilibrium_grasp"/>
+        <origin xyz="0 0 0"
+                rpy="0 0 0"/>
+    </joint>
   </xacro:macro>
-  <link name="gripper_equilibrium_grasp"/>
-  <joint name="gripper_base_link_gripper_equilibrium_grasp" type="fixed">
-    <parent link="epick_end_effector"/>
-      <child link="gripper_equilibrium_grasp"/>
-      <origin xyz="0 0 0"
-              rpy="0 0 0"/>
-  </joint>
 </robot>

Commit message: Phase 0 archive: inter:/home/aurmr/workspaces/aurmr_demo_integration_03/src/aurmr_tahoma
Branch: soofiyan-new-grasp-with-normals
Base HEAD: 65f824e6ed6374ade11f945c6df2f190abe5b3b9
Includes uncommitted tracked changes and untracked code/config.
Excluded untracked files (noise/data/>5MB): 0

File: tahoma_description/urdf/tahoma.xacro (robot description, xacro)
@@ -187,5 +187,5 @@
         <child link="camera_base"/>
         <!-- Link is centered on the optical frames. Slight offset in Y direction to compensate -->
-        <origin xyz="-0.20750794 -0.01749962  1.40753882" rpy="3.14 3.14 -3.14" />
+        <origin xyz="-0.20750794 -0.03749962  1.40753882" rpy="3.14 3.14 -3.14" />
         <!-- <origin xyz="-0.2426 -0.0277 1.4078" rpy="3.14 3.14 -3.14" /> -->
       </joint>

Commit message: Phase 0 archive: inter:/home/aurmr/workspaces/calib/src/aurmr_tahoma
Branch: calib
Base HEAD: 5735170d3f481b19fa151b2059ed2e1eb1ab75bb
Includes uncommitted tracked changes and untracked code/config.
Excluded untracked files (noise/data/>5MB): 0

File: tahoma_description/urdf/tahoma.xacro (robot description, xacro)
@@ -217,4 +217,5 @@
     <xacro:arg name="use_mesh" default="true" />
     <xacro:include filename="$(find tahoma_description)/urdf/_l515.urdf.xacro" />
+    <xacro:include filename="$(find tahoma_description)/urdf/_arducam.urdf.xacro" />
     <!-- D435 Realsense Camera -->
     <!-- <xacro:sensor_d435 parent="base_link" use_nominal_extrinsics="$(arg use_nominal_extrinsics)" add_plug="$(arg add_plug)" use_mesh="$(arg use_mesh)">
@@ -243,4 +244,11 @@
       <origin xyz="0.0 0.046 0.06" rpy="${pi} -${0.5 * pi} ${0.5 * pi}"/>
     </xacro:sensor_l515>
+    <!-- Wrist-mounted arducam (eye-in-hand). NOMINAL placement only, measured
+         by hand — not calibrated. Do not trust for precision until
+         calib_with_april_tag_eye_in_hand.py has been run and this origin is
+         replaced with the solved transform (see the arducam integration plan). -->
+    <xacro:sensor_arducam parent="coupling" name="arducam">
+      <origin xyz="0.03 -0.04 0.05" rpy="0 0 0"/>
+    </xacro:sensor_arducam>
     <!-- <link name="realsense_lower_mount">
       <collision>

Commit message: Phase 0 archive: emmons:/home/aurmr/workspaces/aurmr_demo_staging_clone/src/aurmr_tahoma
Branch: motion_planning
Base HEAD: ebbdd7ecf244d0584951ca651e7a10241e619708
Includes uncommitted tracked changes and untracked code/config.
Excluded untracked files (noise/data/>5MB): 0

File: tahoma_description/urdf/tahoma.xacro (robot description, xacro)
@@ -42,4 +42,26 @@
       <child link="stand"/>
     </joint>
+    <link name="table">
+      <visual>
+        <origin xyz="0 0 0" rpy="0 0 0"/>
+        <geometry>
+          <box size="0.8 1.5 0.05"/>
+        </geometry>
+        <material name="table_color">
+          <color rgba="0.8 0.6 0.4 0.5"/>
+        </material>
+      </visual>
+      <collision>
+        <origin xyz="0 0 0" rpy="0 0 0"/>
+        <geometry>
+          <box size="0.8 1.5 0.05"/>
+        </geometry>
+      </collision>
+    </link>
+    <joint name="base_link_table_joint" type="fixed">
+      <parent link="base_link"/>
+      <child link="table"/>
+      <origin xyz="0.0 0.0 0.75" rpy="0 0 0"/>
+    </joint>
     <joint name="robot_plate_arm_base_link_joint" type="fixed">
       <parent link="robot_plate"/>

Commit message: Phase 0 archive: emmons:/home/aurmr/workspaces/markus_test/src/aurmr_tahoma
Branch: motion_planning
Base HEAD: ebbdd7ecf244d0584951ca651e7a10241e619708
Includes uncommitted tracked changes and untracked code/config.
Excluded untracked files (noise/data/>5MB): 0

File: tahoma_description/urdf/tahoma.xacro (robot description, xacro)
@@ -35,5 +35,5 @@
             prefix="gripper_"
             transmission_hw_interface="${gripper_transmission_hw_interface}"/> -->
-    <xacro:epick_hand hand_link_name="gripper_base_link" robot_name="tahoma"/>
+    <!-- <xacro:epick_hand hand_link_name="gripper_base_link" robot_name="tahoma"/> -->
     <link name="base_link"/>
     <joint name="base_joint" type="fixed">
@@ -42,4 +42,26 @@
       <child link="stand"/>
     </joint>
+    <link name="table">
+      <visual>
+        <origin xyz="0 0 0" rpy="0 0 0"/>
+        <geometry>
+          <box size="1.0 1.5 0.05"/>
+        </geometry>
+        <material name="table_color">
+          <color rgba="0.8 0.6 0.4 0.5"/>
+        </material>
+      </visual>
+      <collision>
+        <origin xyz="0 0 0" rpy="0 0 0"/>
+        <geometry>
+          <box size="1.0 1.5 0.05"/>
+        </geometry>
+      </collision>
+    </link>
+    <joint name="base_link_table_joint" type="fixed">
+      <parent link="base_link"/>
+      <child link="table"/>
+      <origin xyz="0.0 0.0 0.76" rpy="0 0 0"/>
+    </joint>
     <joint name="robot_plate_arm_base_link_joint" type="fixed">
       <parent link="robot_plate"/>
@@ -81,9 +103,41 @@
       </collision>
     </link>
-    <joint name="coupling_link_gripper_robotiq_arg2f_base_link_joint" type="fixed">
+    <joint name="gripper_base" type="fixed">
+      <parent link="coupling"/>
+      <child link="capacitive_cup"/>
+      <origin rpy="0 0 0" xyz="0 0.0 .0169"/>
+    </joint>
+    <link name="capacitive_cup">
+      <!-- <visual>
+        <origin xyz="0 0 0" rpy="0 0 0"/>
+        <geometry>
+          <mesh filename="package://robotiq_2f_85_gripper_visualization/meshes/visual/coupling.stl"/>
+        </geometry>
+        <material name="">
+          <color rgba="0.1 0.1 0.1 1"/>
+        </material>
+      </visual>
+     <visual>
+        <origin xyz="0.0335 0 0.0" rpy="0 0 0"/>
+        <geometry>
+          <mesh filename="package://robotiq_2f_85_gripper_visualization/meshes/visual/connector_cover.stl"/>
+        </geometry>
+        <material name="">
+          <color rgba="0.1 0.1 0.1 1"/>
+        </material>
+      </visual> -->
+      <collision>
+        <!-- Primitives are centered, so offset -->
+        <origin xyz="0 0 ${.177 / 2}" rpy="0 0 0"/>
+        <geometry>
+          <cylinder radius=".0375" length=".177"/>
+        </geometry>
+      </collision>
+    </link>
+    <!-- <joint name="coupling_link_gripper_robotiq_arg2f_base_link_joint" type="fixed">
       <origin xyz="0 0 0.055" rpy="0 0 0"/>
       <parent link="coupling"/>
       <child link="gripper_base_link"/>
-    </joint>
+    </joint> -->
     <joint name="arm_tool0-coupling_joint" type="fixed">
       <origin xyz="0 0 0" rpy="0 0 ${1.5 * pi}"/>
@@ -168,5 +222,5 @@
     <xacro:arg name="use_mesh" default="true" />
     <xacro:include filename="$(find tahoma_description)/urdf/_l515.urdf.xacro" />
-    <link name="realsense_back_gripper_mount">
+    <!-- <link name="realsense_back_gripper_mount">
       <collision>
         <origin xyz="0.010227 -0.005 0.035" rpy="0 0 0"/>
@@ -181,23 +235,25 @@
         </geometry>
       </visual>
-    </link>
-    <xacro:sensor_l515 parent="coupling" use_nominal_extrinsics="$(arg use_nominal_extrinsics)" add_plug="$(arg add_plug)" use_mesh="$(arg use_mesh)">
+    </link> -->
+    <!-- <xacro:sensor_l515 parent="coupling" use_nominal_extrinsics="$(arg use_nominal_extrinsics)" add_plug="$(arg add_plug)" use_mesh="$(arg use_mesh)">
       <origin xyz="0.0 0.046 0.06" rpy="${pi} -${0.5 * pi} ${0.5 * pi}"/>
-    </xacro:sensor_l515>
-    <joint name="realsense_back_gripper_mount_joint" type="fixed">
+    </xacro:sensor_l515> -->
+    <!-- <joint name="realsense_back_gripper_mount_joint" type="fixed">
         <parent link="camera_link"/>
         <child link="realsense_back_gripper_mount"/>
         <origin xyz="-0.018 0.010227 -0.036" rpy="0 0 ${-0.5 * pi}" />
-    </joint>
-    <xacro:if value="${realsense}">
+    </joint> -->
+    <!-- <xacro:if value="${realsense}">
       <xacro:sensor_l515 name="camera_lower_right" parent="camera_lower_right_mount" use_nominal_extrinsics="${use_nominal_camera_extrinsics}">
         <origin xyz="0 0 0" rpy="0 0 0"/>
       </xacro:sensor_l515>
-    </xacro:if>
-  <link name="gripper_equilibrium_grasp"/>
+    </xacro:if> -->
+  <link name="gripper_equilibrium_grasp">
+        <!-- <collisioncommon -->
+  </link>
   <joint name="gripper_base_link_gripper_equilibrium_grasp" type="fixed">
-    <parent link="epick_end_effector"/>
+    <parent link="capacitive_cup"/>
       <child link="gripper_equilibrium_grasp"/>
-      <origin xyz="0 0 0"
+      <origin xyz="0 0 0.177"
               rpy="0 0 0"/>
   </joint>

Commit message: Phase 0 archive: emmons:/home/aurmr/workspaces/soofiyan_ws_old_gripper/src/aurmr_tahoma
Branch: vacuum_gripper
Base HEAD: ed34fcca842606779e05623a2d49110041c11977
Includes uncommitted tracked changes and untracked code/config.
Excluded untracked files (noise/data/>5MB): 0

File: tahoma_description/urdf/tahoma.xacro (robot description, xacro)
@@ -91,87 +91,4 @@
       <child link="coupling"/>
     </joint>
-    <link name="camera_lower_right_mount">
-      <collision>
-        <origin xyz="0 0 0" rpy="0 0 0"/>
-        <geometry>
-          <box size=".1 .15 .15"/>
-        </geometry>
-      </collision>
-    </link>
-    <link name="camera_lower_left_mount">
-      <collision>
-        <origin xyz="0 0 0" rpy="0 0 0"/>
-        <geometry>
-          <box size=".1 .15 .15"/>
-        </geometry>
-      </collision>
-    </link>
-    <!-- These are the planned ("nominal") mount placements. On the real system, these should
-     be overridden by calibrated transforms published separately -->
-    <xacro:if value="${camera_arrangement == 'manual' }">
-      <joint name="camera_beam_lower_camera_lower_left_mount_joint" type="fixed">
-        <parent link="camera_beam_lower"/>
-        <child link="camera_lower_left_mount"/>
-        <!-- Link is centered on the optical frames. Slight offset in Y direction to compensate -->
-        <origin xyz="0.02 ${-0.0215 + (camera_baseline / 2)} 0.14"
-                rpy="${pi / 2} ${radians(15)} ${-atan2((camera_baseline /2),camera_focal_depth)}"/>
-      </joint>
-      <joint name="camera_beam_lower_camera_lower_right_mount_joint" type="fixed">
-        <parent link="camera_beam_lower"/>
-        <child link="camera_lower_right_mount"/>
-        <origin xyz="0.02 ${0.0215 + (-camera_baseline / 2)} 0.14"
-                rpy="${pi / 2} ${radians(15)} ${atan2((camera_baseline /2),camera_focal_depth)}"/>
-      </joint>
-    </xacro:if>
-    <xacro:if value="${camera_arrangement == 'convergent' }">
-      <joint name="camera_beam_lower_camera_lower_left_mount_joint" type="fixed">
-        <parent link="camera_beam_lower"/>
-        <child link="camera_lower_left_mount"/>
-        <!-- Link is centered on the optical frames. Slight offset in Y direction to compensate -->
-        <origin xyz="0 ${-0.0215 + -camera_baseline / 2} 0.09"
-                rpy="${pi / 2} 0 ${-atan2((camera_baseline /2),camera_focal_depth)}"/>
-      </joint>
-      <joint name="camera_beam_lower_camera_lower_right_mount_joint" type="fixed">
-        <parent link="camera_beam_lower"/>
-        <child link="camera_lower_right_mount"/>
-        <origin xyz="0 ${-0.0215 + -camera_baseline / 2} 0.09"
-                rpy="${pi / 2} 0 ${atan2((camera_baseline /2),camera_focal_depth)}"/>
-      </joint>
-    </xacro:if>
-    <xacro:if value="${camera_arrangement == 'convergent_tilted' }">
-      <joint name="camera_beam_lower_camera_lower_left_mount_joint" type="fixed">
-        <parent link="camera_beam_lower"/>
-        <child link="camera_lower_left_mount"/>
-        <!-- Link is centered on the optical frames. Slight offset in Y direction to compensate -->
-        <origin xyz="-0.00 ${-0.0215 + (camera_baseline / 2)} 0.09"
-                rpy="${pi / 2} ${radians(15)} ${-atan2((camera_baseline /2),camera_focal_depth)}"/>
-      </joint>
-      <joint name="camera_beam_lower_camera_lower_right_mount_joint" type="fixed">
-        <parent link="camera_beam_lower"/>
-        <child link="camera_lower_right_mount"/>
-        <origin xyz="-0.00 ${0.0215 + (-camera_baseline / 2)} 0.09"
-                rpy="${pi / 2} ${radians(15)} ${atan2((camera_baseline /2),camera_focal_depth)}"/>
-      </joint>
-    </xacro:if>
-    <!-- Upper cameras -->
-    <!-- Link is centered on the optical frames. Slight offset in Y direction to compensate -->
-    <!-- Z=1.10 for on top of the top beam -->
-    <!-- Z=0.80 for underneath the top beam -->
-    <!-- Disabled until we know about manipulability in upper bins
-    <link name="camera_upper_right_mount"/>
-    <link name="camera_upper_left_mount"/>
-    <joint name="stand_upright_camera_upper_left_mount_joint" type="fixed">
-      <parent link="stand_upright"/>
-      <child link="camera_upper_left_mount"/>
-      <origin xyz="-.1 ${-0.0215 + (camera_baseline / 2)} 0.80"
-              rpy="${pi / 2} ${radians(15)} ${-atan2((camera_baseline /2),camera_focal_depth)}"/>
-    </joint>
-    <joint name="stand_upright_camera_upper_right_mount_joint" type="fixed">
-      <parent link="stand_upright"/>
-      <child link="camera_upper_right_mount"/>
-      <origin xyz="-.1 ${0.0215 + (-camera_baseline / 2)} 0.80"
-              rpy="${pi / 2} ${radians(15)} ${atan2((camera_baseline /2),camera_focal_depth)}"/>
-    </joint>
-    -->
     <link name="cantilever_camera_upper_mount"/>
     <joint name="cantilever_camera_upper_mount_joint" type="fixed">

Commit message: Phase 0 archive: winthrop:/home/aurmr/workspaces/dynamo_grasp_ws/src/aurmr_tahoma
Branch: soofiyan-new-grasp-with-normals
Base HEAD: 6c847f6577eccfde2e31307d9b738e9eb4568d58
Includes uncommitted tracked changes and untracked code/config.
Excluded untracked files (noise/data/>5MB): 0

File: tahoma_description/urdf/tahoma.xacro (robot description, xacro)
@@ -187,5 +187,5 @@
         <child link="camera_base"/>
         <!-- Link is centered on the optical frames. Slight offset in Y direction to compensate -->
-        <origin xyz="-0.260 0.0 1.465" rpy="3.13764 3.12912 -3.12899" />
+        <origin xyz="-0.260 -0.005 1.465" rpy="3.13764 3.12912 -3.12899" />
       </joint>
     </xacro:if>
