Commit message: new changes for camera

File: tahoma_description/urdf/_l515.urdf.xacro (robot description, xacro)
@@ -21,6 +21,5 @@
 <robot name="sensor_l515" xmlns:xacro="http://ros.org/wiki/xacro">
   <!-- Includes -->
-  <!-- FIXME(nickswalker,9-29-23): Somehow aluminum is ending up duplicated in our full xacros. Debug if you need to fix the colors-->
-  <!--xacro:include filename="$(find tahoma_description)/urdf/_materials.urdf.xacro" /> -->
+  <xacro:include filename="$(find tahoma_description)/urdf/_materials.urdf.xacro" />
   <xacro:include filename="$(find tahoma_description)/urdf/_usb_plug.urdf.xacro" /> <!-- this specific plug does not apply to L515 -->
   <xacro:macro name="sensor_l515" params="parent *origin name:=camera use_nominal_extrinsics:=false add_plug:=false use_mesh:=true">

File: tahoma_description/urdf/tahoma.xacro (robot description, xacro)
@@ -155,4 +155,31 @@
       </joint>
     </xacro:if>
+    <!-- Upper cameras -->
+    <!-- Link is centered on the optical frames. Slight offset in Y direction to compensate -->
+    <!-- Z=1.10 for on top of the top beam -->
+    <!-- Z=0.80 for underneath the top beam -->
+    <!-- Disabled until we know about manipulability in upper bins
+    <link name="camera_upper_right_mount"/>
+    <link name="camera_upper_left_mount"/>
+    <joint name="stand_upright_camera_upper_left_mount_joint" type="fixed">
+      <parent link="stand_upright"/>
+      <child link="camera_upper_left_mount"/>
+      <origin xyz="-.1 ${-0.0215 + (camera_baseline / 2)} 0.80"
+              rpy="${pi / 2} ${radians(15)} ${-atan2((camera_baseline /2),camera_focal_depth)}"/>
+    </joint>
+    <joint name="stand_upright_camera_upper_right_mount_joint" type="fixed">
+      <parent link="stand_upright"/>
+      <child link="camera_upper_right_mount"/>
+      <origin xyz="-.1 ${0.0215 + (-camera_baseline / 2)} 0.80"
+              rpy="${pi / 2} ${radians(15)} ${atan2((camera_baseline /2),camera_focal_depth)}"/>
+    </joint>
+    -->
+    <link name="cantilever_camera_upper_mount"/>
+    <joint name="cantilever_camera_upper_mount_joint" type="fixed">
+      <parent link="cantilever"/>
+      <child link="cantilever_camera_upper_mount"/>
+      <origin xyz=".02 0 0.37"
+              rpy="0 ${radians(15)} 0"/>
+    </joint>
     <xacro:if value="${azure_kinect}">
       <xacro:include filename="$(find tahoma_description)/urdf/azure_kinect.urdf.xacro"/>
@@ -161,6 +188,5 @@
         <child link="camera_base"/>
         <!-- Link is centered on the optical frames. Slight offset in Y direction to compensate -->
-        <origin xyz="-0.20750794 -0.01815336  1.40753882" rpy="3.14 3.14 -3.14" />
-        <!-- <origin xyz="-0.2426 -0.0277 1.4078" rpy="3.14 3.14 -3.14" /> -->
+        <origin xyz="-0.260 0 1.465" rpy="3.13764 3.12912 -3.12899" />
       </joint>
     </xacro:if>
@@ -169,4 +195,12 @@
     <xacro:arg name="use_mesh" default="true" />
     <xacro:include filename="$(find tahoma_description)/urdf/_l515.urdf.xacro" />
+    <!-- D435 Realsense Camera -->
+    <!-- <xacro:sensor_d435 parent="base_link" use_nominal_extrinsics="$(arg use_nominal_extrinsics)" add_plug="$(arg add_plug)" use_mesh="$(arg use_mesh)">
+      <origin xyz="-0.217 0.013 1.354" rpy="0 0 0"/>
+    </xacro:sensor_d435> -->
+    <!-- D455 Realsense Camera -->
+    <!-- <xacro:sensor_d455 parent="base_link" use_nominal_extrinsics="$(arg use_nominal_extrinsics)">
+      <origin xyz="-0.217 -0.025 1.364" rpy="0 0 0"/>
+    </xacro:sensor_d455> -->
     <link name="realsense_back_gripper_mount">
       <collision>
@@ -183,4 +217,26 @@
       </visual>
     </link>
+    <!-- L515 Realsense Camera -->
+    <xacro:sensor_l515 parent="coupling" use_nominal_extrinsics="$(arg use_nominal_extrinsics)" add_plug="$(arg add_plug)" use_mesh="$(arg use_mesh)">
+      <origin xyz="0.0 0.046 0.1165" rpy="${pi} -${0.5 * pi} ${0.5 * pi}"/>
+    </xacro:sensor_l515>
+    <!-- <link name="realsense_lower_mount">
+      <collision>
+        <origin xyz="0 0 0" rpy="0 0 0"/>
+        <geometry>
+          <box size="0.06 0.1 0.06"/>
+        </geometry>
+      </collision>
+    </link>
+    <joint name="realsense_mount_joint" type="fixed">
+        <parent link="camera_bottom_screw_frame"/>
+        <child link="realsense_lower_mount"/>
+        <origin xyz="0.03 0 -0.05" rpy="0 0 0" />
+    </joint> -->
+    <joint name="realsense_back_gripper_mount_joint" type="fixed">
+        <parent link="camera_link"/>
+        <child link="realsense_back_gripper_mount"/>
+        <origin xyz="-0.018 0.010227 -0.036" rpy="0 0 ${-0.5 * pi}" />
+    </joint>
     <xacro:if value="${realsense}">
       <xacro:sensor_l515 name="camera_lower_right" parent="camera_lower_right_mount" use_nominal_extrinsics="${use_nominal_camera_extrinsics}">
@@ -202,4 +258,7 @@
     </link>
     </xacro:if>
+      <xacro:sensor_l515 name="camera_upper" parent="cantilever_camera_upper_mount" use_nominal_extrinsics="${use_nominal_camera_extrinsics}">
+        <origin xyz="0 0 0" rpy="0 0 0"/>
+      </xacro:sensor_l515>
     <!-- L515 Realsense Camera -->
     <xacro:sensor_l515 parent="realsense_back_gripper_mount" use_nominal_extrinsics="${use_nominal_camera_extrinsics}" add_plug="false" use_mesh="true">

Commit message: Fix errors in robot, pod xacros
Fix a missing </if>
Remove duplicated camera mount
Drop old realsenses
Rename a material to avoid conflicts with realsense material names

File: tahoma_description/urdf/_l515.urdf.xacro (robot description, xacro)
@@ -21,5 +21,6 @@
 <robot name="sensor_l515" xmlns:xacro="http://ros.org/wiki/xacro">
   <!-- Includes -->
-  <xacro:include filename="$(find tahoma_description)/urdf/_materials.urdf.xacro" />
+  <!-- FIXME(nickswalker,9-29-23): Somehow aluminum is ending up duplicated in our full xacros. Debug if you need to fix the colors-->
+  <!--xacro:include filename="$(find tahoma_description)/urdf/_materials.urdf.xacro" /> -->
   <xacro:include filename="$(find tahoma_description)/urdf/_usb_plug.urdf.xacro" /> <!-- this specific plug does not apply to L515 -->
   <xacro:macro name="sensor_l515" params="parent *origin name:=camera use_nominal_extrinsics:=false add_plug:=false use_mesh:=true">

File: tahoma_description/urdf/pod.xacro (robot description, xacro)
@@ -65,5 +65,5 @@
       <color rgba="1 .91 .2 1"/>
     </material>
-    <material name="aluminum">
+    <material name="steel">
       <color rgba=".6 .6 .6 1"/>
     </material>
@@ -78,5 +78,5 @@
           <mesh filename="package://tahoma_description/meshes/pod/pod_frame.stl"/>
         </geometry>
-        <material name="aluminum"/>
+        <material name="steel"/>
       </visual>
       <collision>

File: tahoma_description/urdf/pod1.xacro (robot description, xacro)
@@ -18,5 +18,5 @@
       <color rgba="1 .91 .2 1"/>
     </material>
-    <material name="aluminum">
+    <material name="steel">
       <color rgba=".6 .6 .6 1"/>
     </material>

File: tahoma_description/urdf/pod2.xacro (robot description, xacro)
@@ -18,5 +18,5 @@
       <color rgba="1 .91 .2 1"/>
     </material>
-    <material name="aluminum">
+    <material name="steel">
       <color rgba=".6 .6 .6 1"/>
     </material>

File: tahoma_description/urdf/tahoma.xacro (robot description, xacro)
@@ -155,31 +155,4 @@
       </joint>
     </xacro:if>
-    <!-- Upper cameras -->
-    <!-- Link is centered on the optical frames. Slight offset in Y direction to compensate -->
-    <!-- Z=1.10 for on top of the top beam -->
-    <!-- Z=0.80 for underneath the top beam -->
-    <!-- Disabled until we know about manipulability in upper bins
-    <link name="camera_upper_right_mount"/>
-    <link name="camera_upper_left_mount"/>
-    <joint name="stand_upright_camera_upper_left_mount_joint" type="fixed">
-      <parent link="stand_upright"/>
-      <child link="camera_upper_left_mount"/>
-      <origin xyz="-.1 ${-0.0215 + (camera_baseline / 2)} 0.80"
-              rpy="${pi / 2} ${radians(15)} ${-atan2((camera_baseline /2),camera_focal_depth)}"/>
-    </joint>
-    <joint name="stand_upright_camera_upper_right_mount_joint" type="fixed">
-      <parent link="stand_upright"/>
-      <child link="camera_upper_right_mount"/>
-      <origin xyz="-.1 ${0.0215 + (-camera_baseline / 2)} 0.80"
-              rpy="${pi / 2} ${radians(15)} ${atan2((camera_baseline /2),camera_focal_depth)}"/>
-    </joint>
-    -->
-    <link name="cantilever_camera_upper_mount"/>
-    <joint name="cantilever_camera_upper_mount_joint" type="fixed">
-      <parent link="cantilever"/>
-      <child link="cantilever_camera_upper_mount"/>
-      <origin xyz=".02 0 0.37"
-              rpy="0 ${radians(15)} 0"/>
-    </joint>
     <xacro:if value="${azure_kinect}">
       <xacro:include filename="$(find tahoma_description)/urdf/azure_kinect.urdf.xacro"/>
@@ -196,13 +169,4 @@
     <xacro:arg name="use_mesh" default="true" />
     <xacro:include filename="$(find tahoma_description)/urdf/_l515.urdf.xacro" />
-    <!-- D435 Realsense Camera -->
-    <!-- <xacro:sensor_d435 parent="base_link" use_nominal_extrinsics="$(arg use_nominal_extrinsics)" add_plug="$(arg add_plug)" use_mesh="$(arg use_mesh)">
-      <origin xyz="-0.217 0.013 1.354" rpy="0 0 0"/>
-    </xacro:sensor_d435> -->
-    <!-- D455 Realsense Camera -->
-    <!-- <xacro:sensor_d455 parent="base_link" use_nominal_extrinsics="$(arg use_nominal_extrinsics)">
-      <origin xyz="-0.217 -0.025 1.364" rpy="0 0 0"/>
-    </xacro:sensor_d455> -->
-    <!-- ##################################################################3 -->
     <link name="realsense_back_gripper_mount">
       <collision>
@@ -219,27 +183,4 @@
       </visual>
     </link>
-    <!-- L515 Realsense Camera -->
-    <xacro:sensor_l515 parent="coupling" use_nominal_extrinsics="$(arg use_nominal_extrinsics)" add_plug="$(arg add_plug)" use_mesh="$(arg use_mesh)">
-      <origin xyz="0.0 0.046 0.1165" rpy="${pi} -${0.5 * pi} ${0.5 * pi}"/>
-    </xacro:sensor_l515>
-    <!-- <link name="realsense_lower_mount">
-      <collision>
-        <origin xyz="0 0 0" rpy="0 0 0"/>
-        <geometry>
-          <box size="0.06 0.1 0.06"/>
-        </geometry>
-      </collision>
-    </link>
-    <joint name="realsense_mount_joint" type="fixed">
-        <parent link="camera_bottom_screw_frame"/>
-        <child link="realsense_lower_mount"/>
-        <origin xyz="0.03 0 -0.05" rpy="0 0 0" />
-    </joint> -->
-    <!-- #######################################################################3 -->
-    <joint name="realsense_back_gripper_mount_joint" type="fixed">
-        <parent link="camera_link"/>
-        <child link="realsense_back_gripper_mount"/>
-        <origin xyz="-0.018 0.010227 -0.036" rpy="0 0 ${-0.5 * pi}" />
-    </joint>
     <xacro:if value="${realsense}">
       <xacro:sensor_l515 name="camera_lower_right" parent="camera_lower_right_mount" use_nominal_extrinsics="${use_nominal_camera_extrinsics}">
@@ -260,7 +201,5 @@
       </visual>
     </link>
-      <xacro:sensor_l515 name="camera_upper" parent="cantilever_camera_upper_mount" use_nominal_extrinsics="${use_nominal_camera_extrinsics}">
-        <origin xyz="0 0 0" rpy="0 0 0"/>
-      </xacro:sensor_l515>
+    </xacro:if>
     <!-- L515 Realsense Camera -->
     <xacro:sensor_l515 parent="realsense_back_gripper_mount" use_nominal_extrinsics="${use_nominal_camera_extrinsics}" add_plug="false" use_mesh="true">

Commit message: Integrated vacuum array gripper to state machine

File: tahoma_description/urdf/_l515.urdf.xacro (robot description, xacro)
@@ -88,10 +88,10 @@
         </xacro:unless>
       </visual>
-      <collision>
+      <!-- <collision>
         <origin xyz="${-l515_cam_depth_px+l515_cam_mount_from_glass_offset-l515_cam_depth/2} 0 ${-l515_cam_center_to_depth_pz}" rpy="${M_PI/2} 0 ${M_PI/2}"/>
         <geometry>
           <cylinder radius="${l515_cam_width/2.0}" length="${l515_cam_depth}"/>
         </geometry>
-      </collision>
+      </collision> -->
       <inertial>
         <!-- The following are not reliable values, and should not be used for modeling -->

File: tahoma_description/urdf/tahoma.xacro (robot description, xacro)
@@ -83,5 +83,6 @@
     </link>
     <joint name="coupling_link_gripper_robotiq_arg2f_base_link_joint" type="fixed">
-      <origin xyz="0 0 0.055" rpy="0 0 0"/>
+    <!-- xyz use to be 0 0 0.055 before new multifingered vacuum gripper-->
+      <origin xyz="0 0 0.0" rpy="0 0 0"/>
       <parent link="coupling"/>
       <child link="gripper_base_link"/>
